File: Boards/baseVariant/schematic.sch (EAGLE design)
At the start: 114 parts

Commit message: Development in supply section, ongoing...
Parts:
- removed $$U$7: JST-2MM, BaseApp:JST-2MM
- removed 5V: TPSB2,54, testpad:TPSB2,54
- removed C18, C27: 4.7u, BaseApp:CAPACITOR
- removed D3, D4: ss14, SparkFun:DIODE-SCHOTTKY_
- removed MCP73831: (no value), BaseApp:MCP73831
- removed R24: 10k, rcl:R-EU_R0603
- removed R25: 1K, resistor:R-EU_R0603
- added BAT: (no value), SparkFun-Connectors:M03PTH
- added C3, C4: 0.1uF, SparkFun-Capacitors:CAP0402-CAP
- added C8: 10uF, SparkFun-Capacitors:CAP0402-CAP
- added IC1: BQ24120, texas:BQ24120
- added L3: 10uH, SparkFun-Passives:INDUCTOR-B82462G
- added LED3, LED4, LED6: (no value), led:LEDCHIP-LED0603
- added R11, R12, R20, R7: 7.5k, SparkFun-Passives:RESISTOR0402-RES
- added R2, R3, R6: 1.5k, SparkFun-Passives:RESISTOR0402-RES
- added RSNS: 0.1, SparkFun-Passives:RESISTOR0402-RES
- C29: device BaseApp:CAPACITOR -> SparkFun-Capacitors:CAP0402-CAP
Connections:
- removed net +5V: 5V.PP, C27.1, C29.1, D4.A, JP4.VBUS, MCP73831.VDD, R25.2
- removed net N$20 (its old number): D3.C, D4.C, JP5.2
- removed net N$41: MCP73831.PROG, R24.1
- new net N$14: C3.1, IC1G$1.TTC
- new net N$2: IC1G$1.OUT@1, IC1G$1.OUT@2, L3.1
- new net N$28: LED6.A, R6.1
- new net N$29: LED4.A, R3.1
- new net N$30: LED3.A, R2.1
- new net N$33: R20.2
- new net N$36: IC1G$1.ISET2, R11.2
- new net N$40: IC1G$1.ISET1, R7.2
- new net N$46: BAT.1, IC1G$1.BAT, RSNS.1
- new net N$5: IC1G$1.STAT2, LED4.C
- new net N$6: IC1G$1.!PG, LED6.C
- new net N$7: IC1G$1.STAT1, LED3.C
- new net NTC: BAT.2, IC1G$1.TS, R12.2, R20.1
- new net VBUS: C29.1, IC1G$1.IN1, IC1G$1.IN2, IC1G$1.VCC, JP4.VBUS, R2.2, R3.2, R6.2
- new net VTSB: C4.1, IC1G$1.VTSB, R12.1
- net GND: now also BAT.3, C3.2, C4.2, C8.2, IC1G$1.!CE, IC1G$1.PGND@1, IC1G$1.PGND@2, IC1G$1.VSS, R11.1, R7.1; no longer $$U$7.-, C18.2, C27.2, MCP73831.VSS, R24.2
- net STAT: no longer MCP73831.STAT, R25.1
- net VBAT: now also C8.1, IC1G$1.SNS, L3.2, RSNS.2; no longer $$U$7.+, C18.1, D3.A, MCP73831.VBAT
- net VDD: no longer JP5.1, MCP1826G$1.VIN
Other:
- moved on the sheet: 3V3, C1, C10, C11, C12, C13, C14, C15, C16, C17, C2, C28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

Commit message: Schematic Reframed.
Parts:
- removed C2: 100u, rcl:CPOL-USD
- removed D8: ss14, SparkFun:DIODE-SCHOTTKY_
- removed JP5: (no value), jumper:JP1E
- removed L1: 22uH, SparkFun:INDUCTORCR54
- removed NCP1: (no value), SparkFun:V_REG_NCP1400SOT23-5
- removed R31: 10K, resistor:R-EU_R0603
Connections:
- removed net N$1: D8.A, L1.1, NCP1.LX
- removed net N$33: R20.2
- removed net RC6: NCP1.EN
- removed net VUSB: C2.+, D8.C, NCP1.OUT
- new net N$31: MCP1826G$1.VIN
- new net SHDN: MCP1826G$1.!SHDN
- net !SHDN: no longer MCP1826G$1.!SHDN, R31.2
- net +3V3: no longer C13.1, C7.+, MCP1826G$1.VOUT, R22.1, R31.1
- net GND: now also R20.2; no longer C2.-, NCP1.GND
- net VDD: now also C13.1, C7.+, MCP1826G$1.VOUT, R22.1; no longer L1.2
Other:
- moved on the sheet: 3V3, C1, C10, C11, C12, C13, C14, C15, C16, C17, C28, C29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

Commit message: Normal Push
Parts:
- removed U$31: PINHEAD-1X3, BaseApp:PINHEAD-1X3
- added SKW71_UART: (no value), SparkFun-Connectors:M03SMD_RA_MALE
Connections:
- net +3V3: no longer C62.2, C89.2, R59.1, R64.1, U$19.VDD_3.3V, U$19.VDD_3.3V@1, U$19.VDD_3.3V@2, V-.2
- net GND: now also SKW71_UART.3; no longer U$31.3
- net SKW71_RX: now also SKW71_UART.1; no longer U$31.1
- net SKW71_TX: now also SKW71_UART.2; no longer U$31.2
- net VDD: now also C62.2, C89.2, R59.1, R64.1, U$19.VDD_3.3V, U$19.VDD_3.3V@1, U$19.VDD_3.3V@2, V-.2
Other:
- moved on the sheet: R65, V-

Commit message: normal Push.
Parts:
- removed 3V3: TPSB2,54, testpad:TPSB2,54
- removed BAT: (no value), SparkFun-Connectors:M03PTH
- removed C63, C64: 220uf, adafruit:CPOL-USD
- removed D5, D7: SMA, SparkFun:DIODE-SCHOTTKY_
- removed D6: 5320, SparkFun:DIODE-SCHOTTKY_
- removed L3: 10uH, SparkFun-Passives:INDUCTOR-B82462G
- removed L4: 47uh, BaseApp:INDUCTOR
- removed LED4, LED6: (no value), led:LEDCHIP-LED0603
- removed LM2596: (no value), BaseApp:LM25XX-2596
- removed R11, R12, R20, R7: 7.5k, SparkFun-Passives:RESISTOR0402-RES
- removed R13, R52: 3.1K, BaseApp:RESISTOR
- removed R3, R6: 1.5k, SparkFun-Passives:RESISTOR0402-RES
- removed R58: 1K, BaseApp:RESISTOR
- removed RSNS: 0.1, SparkFun-Passives:RESISTOR0402-RES
- removed RST_BRD: (no value), SparkFun-Connectors:M02POLAR
- added C18, C19: 4.7uF, rcl:C-EUC0603
- added C2: 200uF, schematic:CPOL-USE
- added CN1: (no value), adafruit:DCBARRELPTH
- added CN2: (no value), adafruit:JST_2PIN-THM
- added D3: DIODE-SCHOTTKY_, schematic:DIODE-SCHOTTKY_
- added GND, VCC: TPSB2,54, testpad:TPSB2,54
- added J1: MAX9850ETI+, schematic:MAX9850ETI+
- added L1: 33uH 3A, schematic:INDUCTOR
- added Q1, Q2, Q3, Q4, Q5: BSS84, transistor-small-signal:BSS84
- added U$1: (no value), schematic:MCP73831
- C15: value 150pf/50V -> 3.3nF
- C16: value 3.3nf/50v -> 150pF
- C3: value 0.1uF -> 680uF; device SparkFun-Capacitors:CAP0402-CAP -> schematic:CPOL-USE
- C4: value 0.1uF -> 220uF; device SparkFun-Capacitors:CAP0402-CAP -> schematic:CPOL-USE
- C7: device adafruit:CPOL-USE2.5-6 -> adafruit:CPOL-USF
- C8: value 10uF -> 4.7uF; device SparkFun-Capacitors:CAP0402-CAP -> rcl:C-EUC0603
- IC1: value BQ24120 -> LM2596S; device texas:BQ24120 -> national-semiconductor:LM2596S
- ICSP: value PIC-ICSPPOLAR_LOCK -> PIC-ICSPPTH; device SparkFun-Connectors:PIC-ICSPPOLAR_LOCK -> SparkFun-Connectors:PIC-ICSPPTH
- LED3: device led:LEDCHIP-LED0603 -> schematic:LEDCHIP-LED0603
- R1: value 1K -> (none); device BaseApp:RESISTOR -> SparkFun-Passives:RESISTOR0402-RES
- R15: value 51R -> 45.3
- R19: value 20K -> 49.9k
- R2: value 1.5k -> 2k
Connections:
- net +48V renamed +57
- removed net 22.2V: D5.A
- removed net N$17: C16.2, C17.2, U$4.VSSA
- removed net N$28: LED6.A, R6.1
- removed net N$29: LED4.A, R3.1
- removed net N$31: MCP1826G$1.VIN
- removed net N$34: C15.2, C16.1, R21.1
- removed net N$40: IC1G$1.ISET1, R7.2
- removed net N$44: D6.C, L4.2, LM2596.OUTPUT
- removed net N$46: BAT.1, IC1G$1.BAT, RSNS.1
- removed net N$61: LM2596.FEEDBACK, R1.2, R13.1
- removed net N$90: R52.1, R58.2, RST_BRD.2
- removed net NTC: BAT.2, IC1G$1.TS, R12.2, R20.1
- removed net VIN: C63.+, D5.C, D7.C, LM2596.VIN, R52.2
- removed net VTSB: C4.1, IC1G$1.VTSB, R12.1
- new net CRGH_STAT: R1.2, U$1.STAT
- new net N$27: R2.1, U$1.PROG
- new net PD_VDC: Q1.D
- new net PVDC: C4.+, IC1.FB, L1.2, Q2.D
- new net VCC: C2.+, LED3.A, Q1.S, Q2.S, Q3.S, Q5.D, U$1.VDD, VCC.PP
- new net VSOURCE: C18.1, MCP1826G$1.VIN, Q4.S, Q5.S
- net +3V3: no longer 3V3.PP, C64.+, L4.1, R13.2, R14.1, R4.1, R5.1
- net 25V: no longer D7.A
- net GND: now also C18.2, C19.2, C2.-, C3.-, C4.-, CN2.1, D3.A, GND.PP, IC1.!ON!/OFF, IC1.GND, Q1.G, Q2.G, Q3.G, Q4.G, Q5.G, R2.2, U$1.VSS; no longer BAT.3, C3.2, C4.2, C63.-, C64.-, D6.A, IC1G$1.!CE, IC1G$1.PGND@1, IC1G$1.PGND@2, IC1G$1.VSS, LM2596.!ON/!OFF, LM2596.GND, LM2596.TAB, R1.1, R11.1, R20.2, R58.1, R7.1, RST_BRD.1
- net N$13: no longer R21.2
- net N$14: now also CN1.GND; no longer C3.1, IC1G$1.TTC
- net N$2: now also D3.C, IC1.OUT, L1.1; no longer IC1G$1.OUT@1, IC1G$1.OUT@2, L3.1
- net N$30: now also C3.+, CN1.PWR, IC1.VIN; no longer LED3.A, R2.1
- net N$36: now also LED3.C, R1.1; no longer IC1G$1.ISET2, R11.2
- net N$5: now also CN1.GNDBREAK; no longer IC1G$1.STAT2, LED4.C
- net N$6: now also C16.2, C17.2, R21.1, U$4.VSSA; no longer IC1G$1.!PG, LED6.C
- net N$7: now also C15.2, C16.1, R21.2; no longer IC1G$1.STAT1, LED3.C
- net VBAT: now also C19.1, CN2.2, Q4.D, U$1.VBAT; no longer IC1G$1.SNS, L3.2, RSNS.2
- net VBUS: now also Q3.D; no longer IC1G$1.IN1, IC1G$1.IN2, IC1G$1.VCC, R2.2, R3.2, R6.2
- net VDD: now also R14.1, R4.1, R5.1
Other:
- note added: "5VDC - 40VDC"
- note added: "5VDC and Battery Power Switching"
- note added: "Battery JST"
- note added: "Charger IC"
- note added: "DC 5V"
- note added: "DC Power IN"
- note added: "On"
- note added: "PD 5V"
- note added: "Power Supply"
- note added: "Power Switching"
- note added: "USB Power"
- note added: "VDD Regulation from Battery or from 5VDC"
- moved on the sheet: C1, C10, C11, C12, C13, C14, C15, C16, C17, C28, C29, C32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
