File: Boards/baseVariant/schematic.sch (EAGLE design)
At the start: 109 parts, among them IC1 LM2596S, J1 MAX9850ETI+, Q1 BSS84, Q2 BSS84, Q3 BSS84, Q4 BSS84, Q5 BSS84

Commit message: Normal Push
Parts:
- removed Q1, Q3: BSS84, transistor-small-signal:BSS84
- added B1: DBLS201G, rectifier:DBLS201G
- added D4, D5: BA340A, SparkFun-DiscreteSemi:B340A
Connections:
- removed net N$14: CN1.GND
- removed net N$30: C3.+, CN1.PWR, IC1.VIN
- removed net N$5: CN1.GNDBREAK
- new net N$17: B1.AC1, CN1.PWR
- new net N$31: B1.+, C3.+, IC1.VIN
- new net OR_VDC: C2.+, D4.C, D5.C
- net GND: now also B1.-, B1.AC2, CN1.GND, CN1.GNDBREAK; no longer Q1.G, Q2.G, Q3.G
- net PD_VDC: now also D4.A; no longer Q1.D
- net PVDC: now also D5.A; no longer Q2.D
- net VBUS: no longer Q3.D
- net VCC: no longer C2.+, Q1.S, Q2.S, Q3.S
Other:
- note added: "DC 5V - 35V"
- note added: "PD 25V"
- note added: "VBUS"
- note removed: "DC 5V"
- note removed: "On"
- note removed: "PD 5V"
- moved on the sheet: C2, C3, C4, CN1, D3, IC1, L1, Q2

Commit message: normal Push.
Parts:
- removed C91, C92: 0.1uf, BaseApp:CAPACITOR
- removed C93: 1uf, BaseApp:CAPACITOR
- removed C94: 0.1uf/100V, BaseApp:CAPACITOR
- removed LED5: (no value), adafruit:LEDCHIP-LED0603
- removed Q2, Q4, Q5: BSS84, transistor-small-signal:BSS84
- removed R49: 330R, BaseApp:RESISTOR
- removed R50: 7.15K, BaseApp:RESISTOR
- removed SMAJ58A: (no value), BaseApp:SCHOTTKY-DIODESMA2
- removed U$14: LTC4263, BaseApp:LTC4263
- added C20, C21: 0.1uf, rcl:C-EUC0603
- added D6, D7: BA340A, SparkFun-DiscreteSemi:B340A
- added LED4: (no value), led:LEDCHIP-LED0603
- added Q1: BSS84, transistor-small-signal:BSS84
- added R11, R12, R6, R7: 57.6k, resistor:R-EU_R0402
- added R13: 10k, resistor:R-EU_R0402
- added R20: 71.5, resistor:R-EU_R0402
- added R3: (no value), SparkFun-Passives:RESISTOR0402-RES
- C18, C8: value 4.7uF -> 0.1uf
- LED3: device schematic:LEDCHIP-LED0603 -> led:LEDCHIP-LED0603
- R1: value (none) -> 57.6k; device SparkFun-Passives:RESISTOR0402-RES -> resistor:R-EU_R0402
- R2: value 2k -> (none)
- U$1: value (none) -> AAT3672-1/-2; device schematic:MCP73831 -> schematic:AAT3672-1/-2
Connections:
- removed net 25V: C28.+, R17.1, R18.2, U$28.2
- removed net CRGH_STAT: R1.2, U$1.STAT
- removed net N$27: R2.1, U$1.PROG
- removed net N$31: B1.+, C3.+, IC1.VIN
- removed net N$92: LED5.C, R49.1
- removed net N$93: R49.2, U$14.LED
- removed net N$94: C93.2, R50.1, U$14.PWRMGT
- removed net OR_VDC: C2.+, D4.C, D5.C
- removed net PVDC: C4.+, D5.A, IC1.FB, L1.2
- new net CHRADP: R11.2, R12.1, U$1.CHRADP
- new net N$14: C20.2, U$1.OUT
- new net N$28: R7.1, U$1.STAT2N
- new net N$42: C21.2, U$1.CT
- new net N$47: LED4.C, R7.2
- new net N$48: LED3.C, R6.2
- new net N$49: LED3.A
- new net N$5: R1.2, U$1.ADPSET
- new net N$50: LED4.A
- new net PAS_VDC: D5.A, U$6.VDC+@0, U$6.VDC+@1
- new net TS: R13.1, U$1.TS
- new net VIN: C2.+, C3.+, D4.C, D5.C, D6.C, IC1.VIN, R3.2
- new net VJACK: B1.+, D6.A
- new net VOUT: C4.+, D7.A, IC1.FB, L1.2, Q1.G, R2.1
- net +57: no longer C92.2, C94.2, LED5.A, SMAJ58A.C, U$14.VDD48, U$6.VDC+@0, U$6.VDC+@1
- net AGND: no longer C91.1, C92.1, C93.1, C94.1, R50.2, SMAJ58A.A, U$14.LEGACY, U$14.OSC, U$14.OUT@0, U$14.OUT@1, U$14.VSS@0, U$14.VSS@1, U$6.VDC-@0, U$6.VDC-@1
- net GND: now also C20.1, C21.1, R1.1, R12.2, R20.1, R3.1, U$1.EP, U$1.GND, U$6.VDC-@0, U$6.VDC-@1; no longer Q4.G, Q5.G, U$1.VSS
- net N$22: now also R6.1, U$1.STAT1N; no longer C91.2, U$14.!SD, U$14.ENFCLS, U$14.MIDSPAN, U$14.VDD5
- net N$36: now also R20.2, U$1.TERM; no longer LED3.C, R1.1
- net PD_VDC: now also C28.+, R17.1, R18.2, U$28.2
- net VBAT: now also U$1.BAT, U$1.ENBAT; no longer C8.1, Q4.D, U$1.VBAT
- net VBUS: now also Q1.D
- net VCC: no longer LED3.A, Q5.D, U$1.VDD
- net VSOURCE: now also C8.1, D7.C, Q1.S, R11.1, R13.2, U$1.ADP, U$1.EN, U$1.EN0; no longer Q4.S, Q5.S
Other:
- note added: "DC 3V3"
- note added: "DC 5V-6V"
- note added: "DC 6V - 40V"
- note added: "P Channel MOSFET"
- note added: "PD 8V - 12V"
- note added: "Passive VDc 8V- 12V"
- note added: "Power ORing"
- note removed: "5VDC and Battery Power Switching"
- note removed: "Charger IC"
- note removed: "DC 5V - 35V"
- note removed: "PD 25V"
- note removed: "VBUS"
- moved on the sheet: B1, C1, C10, C11, C12, C15, C16, C17, C18, C19, C2, C28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

Commit message: normal Push
Parts:
- removed C14: 0.47u, BaseApp:CAPACITOR
- removed C5, C6, C9: (no value), BaseApp:CAPACITOR
- removed C65, C66, C96, C97: 0.1uf, BaseApp:CAPACITOR
- removed D2: BAT54, diode:BAT54
- removed DUO-LED2: (no value), BaseApp:DUOLED-1X2
- removed FID1, FID2, FID3, FID4: FIDUCIAL1X2.5, SparkFun-Aesthetics:FIDUCIAL1X2.5
- removed FX1, FX2: TG110-E055N5, halo-electronics:TG110-E055N5
- removed GND, VCC, VDD: TPSB2,54, testpad:TPSB2,54
- removed ICSP: PIC-ICSPPTH, SparkFun-Connectors:PIC-ICSPPTH
- removed J1: MAX9850ETI+, schematic:MAX9850ETI+
- removed JP1: (no value), SparkFun-Passives:JUMPER-2SMD-NC
- removed P-RESET: SPST_TACT-EVQQ2, adafruit:SPST_TACT-EVQQ2
- removed PIC25K50: PIC18F25K50, BaseApp:PIC18F25K50
- removed POWER: (no value), switch-omron:31-XX
- removed R10: ~200R, BaseApp:RESISTOR
- removed R14: 300K, rcl:R-EU_R0603
- removed R28, R9: 10K, BaseApp:RESISTOR
- removed R4, R5: 330R, rcl:R-EU_R0603
- removed R42, R43, R56, R57: 75R, BaseApp:RESISTOR
- removed U$15, U$6: RJ45, BaseApp:RJ45
- removed U$18: LIGHT_PIPE, BaseApp:LIGHT_PIPE
- added LED5, LED6: (no value), led:LED3MM
- added U$2: ATMEGA32U4QFN, SparkFun-DigitalIC:ATMEGA32U4QFN
- added U1, U2: MAGJACK-POE, SparkFun-Connectors:MAGJACK-POE
- added USB1: USB_SHIELDUSB_A_VERTICAL, schematic:USB_SHIELDUSB_A_VERTICAL
- LED1, LED2: device adafruit:LEDCHIP-LED0603 -> led:LED3MM
Connections:
- removed net !SHDN: PIC25K50.RB5/IOCB5/T3CKI/T1G/AN13
- removed net +3V3: R48.2
- removed net AGND: C1.1, R15.2, U$4.PAD, U$4.VNEG
- removed net LED1: LED1.C, PIC25K50.RB3/CTED2/CCP2/SDO/C12IN2-/AN9
- removed net LED2: LED2.C, PIC25K50.RB2/INT2/CTED1/P1B/AN8
- removed net MCLR: ICSP.VPP, P-RESET.P, P-RESET.P1, PIC25K50.MCLR/VPP/RE3, R10.1
- removed net N$19: FX1.16, U$6.TX+
- removed net N$21: FX1.14, U$6.TX-
- removed net N$32: C96.2, R56.2
- removed net N$35: C6.2, JP1.1
- removed net N$37: JP1.2, R10.2, R9.1
- removed net N$38: C14.2, PIC25K50.VUSB3V3
- removed net N$49: LED3.A
- removed net N$50: LED4.A
- removed net N$69: C65.2, R42.2
- removed net N$70: C66.2, R43.2
- removed net N$73: FX2.15, R43.1
- removed net N$74: FX2.10, R42.1
- removed net N$75: FX1.11, U$6.RX+
- removed net N$77: FX1.9, U$6.RX-
- removed net N$78: R47.1, U$6.Y-
- removed net N$79: R48.1, U$6.G+
- removed net N$80: FX2.16, U$15.TX+
- removed net N$87: FX2.14, U$15.TX-
- removed net N$88: FX2.11, U$15.RX+
- removed net N$89: FX2.9, U$15.RX-
- removed net N$91: R53.1, U$15.Y-
- removed net P-RX: PIC25K50.RC7/SDO/IOCC7/RX/DT/AN19
- removed net P-TX: D2.A, R14.2
- removed net P-TX*: D2.C, PIC25K50.RC6/IOCC6/TX/CK/AN18
- removed net PGC: ICSP.PGC, PIC25K50.RB6/IOCB6/PGC
- removed net PGD: ICSP.PGD, PIC25K50.RB7/IOCB7/PGD
- removed net RA0: PIC25K50.RA0/C12IN0-/AN0
- removed net RA1: PIC25K50.RA1/C12IN1-/AN1
- removed net RB0: PIC25K50.RB0/INT0/FLT0/SRI/SDI/SDA/AN12, POWER.S, R28.1
- removed net STAT: PIC25K50.RB4/IOCB4/P1D/AN11
- removed net VCC: VCC.PP
- new net N$17: USB1.3
- new net N$27: USB1.4
- new net N$29: USB1.5
- new net N$31: R47.1, U2.YLED-
- net +2V: now also U1.RCT, U1.TCT, U2.RCT, U2.TCT; no longer FX1.2, FX1.7, FX2.2, FX2.7
- net ETH0_GRN-: now also U1.GLED-; no longer U$15.G-
- net GND: now also C1.1, R15.2, U$4.PAD, U$4.VNEG, U1.SHIELD@0, U1.SHIELD@1, U2.GLED-, U2.SHIELD@0, U2.SHIELD@1, U2.V-; no longer C14.1, C5.2, C6.1, C65.1, C66.1, C9.2, C96.1, C97.1, GND.PP, ICSP.GND, P-RESET.S, P-RESET.S1, PIC25K50.VSS, PIC25K50.VSS_2, POWER.P, U$15.S1, U$15.S2, U$6.G-, U$6.S1, U$6.S2, U$6.VDC-@0, U$6.VDC-@1
- net LAN_TX+: now also U1.TD+; no longer FX2.1
- net LAN_TX-: now also U1.TD-; no longer FX2.3
- net LAN_YLW: now also U1.YLED+; no longer U$15.Y+
- net N$23: now also U2.YLED+; no longer FX1.15, R57.1
- net N$24: now also R53.1, U1.YLED-; no longer FX1.10, R56.1
- net N$25: now also R48.1, U2.GLED+; no longer C97.2, R57.2
- net N$3: now also USB1.1; no longer LED1.A, R4.2
- net N$4: now also USB1.2; no longer LED2.A, R5.2
- net N$95: now also U1.GLED+; no longer U$15.G+
- net PAS_VDC: now also U2.V+; no longer U$6.VDC+@0, U$6.VDC+@1
- net SP1: now also U1.V-; no longer U$15.VDC-@0, U$15.VDC-@1
- net SP2: now also U1.V+; no longer U$15.VDC+@0, U$15.VDC+@1
- net USB_D_N: no longer PIC25K50.D-/IOCC4
- net USB_D_P: no longer PIC25K50.D+/IOCC5
- net VDD: now also R48.2; no longer C5.1, C9.1, ICSP.VCC, PIC25K50.VDD, R14.1, R28.2, R4.1, R5.1, R9.2, VDD.PP
- net VSOURCE: now also LED3.A, LED4.A
- net WAN_RX+: now also U1.RD+, U2.RD+; no longer FX1.6, FX2.6
- net WAN_RX-: now also U1.RD-, U2.RD-; no longer FX1.8, FX2.8
- net WAN_TX+: now also U2.TD+; no longer FX1.1
- net WAN_TX-: now also U2.TD-; no longer FX1.3
- net WAN_YLW: no longer U$6.Y+
Other:
- moved on the sheet: C13, C7, LED1, LED2, MCP1826, R22, R47, R48, R53, R54

Commit message: Normal Push, With Surge Protection on Host USB.
Parts:
- added C14, C22, C5, C6, C9: (no value), SparkFun:CAP0402-CAP
- added C23: 1uF, SparkFun:CAP0402-CAP
- added C24: 0.1uF, SparkFun-Capacitors:CAP0402-CAP
- added L3: (no value), SparkFun-Passives:INDUCTOR0402
- added R4, R5: 22, SparkFun:RESISTOR0402-RES
- added R9: 1k, SparkFun:RESISTOR0402-RES
- added U$3: PUSBMXX4-TL, schematic:PUSBMXX4-TL
- C2, C4: device schematic:CPOL-USE -> schematic:CPOL-USE5-10.5
- C3: device schematic:CPOL-USE -> schematic:CPOL-USE3.5-10
- C7: device adafruit:CPOL-USF -> adafruit:CPOL-USE5-10.5
Connections:
- removed net N$17: USB1.3
- removed net N$27: USB1.4
- removed net N$29: USB1.5
- removed net N$3: USB1.1
- removed net N$4: USB1.2
- removed net VOUT: C4.+, D7.A, IC1.FB, L1.2, Q1.G, R2.1
- new net N$19: U$2.!RESET
- new net N$32: U$3.3
- new net N$33: U$3.4
- new net N$34: U$3.5
- new net N$37: C23.2, U$2.UCAP
- new net N$38: R4.2, U$2.D+
- new net N$39: R5.2, U$2.D-
- new net N$41: L3.1, USB1.5
- new net N$43: R9.2, U$2.PE2/!HWB
- new net VCC: C14.1, C22.1, C24.1, C4.+, C5.1, C6.1, C9.1, D7.A, IC1.FB, L1.2, Q1.G, R2.1, U$2.AREF, U$2.AVCC@24, U$2.AVCC@44, U$2.VCC@14, U$2.VCC@34, U$3.6, USB1.1
- net GND: now also C14.2, C22.2, C23.1, C24.2, C5.2, C6.2, C9.2, L3.2, R9.1, U$2.GND@15, U$2.GND@23, U$2.GND@35, U$2.GND@43, U$2.UGND, U$3.7, USB1.4
- net USBUPD1_N: now also U$3.1, USB1.2
- net USBUPD1_P: now also U$3.2, USB1.3
- net USB_D_N: now also R5.1
- net USB_D_P: now also R4.1
- net VBUS: now also U$2.UVCC, U$2.VBUS
Other:
- moved on the sheet: C8, D7, Q1, R2, U$2, USB1

Commit message: Normal Push.
Parts:
- removed R59: (no value), BaseApp:RESISTOR
- removed SKW71_UART: (no value), SparkFun-Connectors:M03SMD_RA_MALE
- added C25: 1uF, SparkFun:CAP0402-CAP
- added J1: AVR_SPI_PRG_6NS, Sensor Mesh:AVR_SPI_PRG_6NS
- added JP1: (no value), SparkFun-Connectors:AUDIO-JACK1:1
- added R10: 1k, SparkFun:RESISTOR0402-RES
- added R14, R23, R24, R25: 22, SparkFun:RESISTOR0402-RES
- added U$5: MAX5556ESA+, schematic:MAX5556ESA+
- C2: value 200uF -> 1uF; device schematic:CPOL-USE5-10.5 -> SparkFun:CAP0402-CAP
Connections:
- removed net N$19: U$2.!RESET
- removed net SKW71_RX: SKW71_UART.1, U$19.UART_RX(SPI_CS1)
- removed net SKW71_TX: SKW71_UART.2, U$19.UART_TX(SPI_CS2)
- new net AT_RESET: J1.5, R10.1, U$2.!RESET
- new net GPIO_18: U$19.I2S_CK(GPIO_18), U$5.SCLK
- new net GPIO_20: U$19.I2S_SD(GPIO_20), U$5.SDATA
- new net N$27: R14.2, R23.2
- new net N$35: R24.2, R25.2
- new net N$49: C2.2, JP1.RIGHT, R14.1
- new net N$51: C25.2, JP1.LEFT, R24.1
- new net OUTL: C25.1, R25.1, U$5.OUTL
- new net OUTR: C2.1, R23.1, U$5.OUTR
- new net PB1/SCK: J1.3, U$2.PB1(SCK)
- new net PB2/MOSI: J1.4, U$2.PB2(MOSI)
- new net PB3/MISO: J1.1, U$2.PB3(MISO)
- new net PD2/RXD: U$19.UART_TX(SPI_CS2), U$2.PD2(RX)
- new net PD3/TXD: U$19.UART_RX(SPI_CS1), U$2.PD3(TX)
- net GND: now also J1.6, JP1.SLEEVE, U$5.GND; no longer C2.-, SKW71_UART.3
- net GPIO_19: now also U$5.LRCLK; no longer R59.2
- net GPIO_21: now also U$5.MCLK
- net VCC: now also J1.2, R10.2, U$5.VDD
- net VDD: no longer R59.1
- net VIN: no longer C2.+
Other:
- note added: "HOST USB"

Commit message: normal Push.
Parts:
- removed D7: BA340A, SparkFun-DiscreteSemi:B340A
- removed JP2: (no value), SparkFun-Connectors:M04POLAR
- removed Q1: BSS84, transistor-small-signal:BSS84
- removed R64: (no value), BaseApp:RESISTOR
- added JP3: (no value), pinhead:PINHD-2X20
- added R26: (no value), SparkFun-Passives:RESISTOR-ARRAY0603-ARV
- added R27: (no value), SparkFun-Passives:RESISTOR0402-RES
- added U$6: FDFMA2P857, BaseApp:FDFMA2P857
- added U$7: SE2580L, schematic:SE2580L
- R2: value (none) -> 10k
Connections:
- removed net GPIO_18: U$19.I2S_CK(GPIO_18), U$5.SCLK
- removed net GPIO_19: JP2.4, U$19.I2S_WS(GPIO_19), U$5.LRCLK
- removed net GPIO_20: U$19.I2S_SD(GPIO_20), U$5.SDATA
- removed net GPIO_21: U$19.I2S_MCK(GPIO_21), U$5.MCLK
- removed net GPIO_22: JP2.2, R64.2, U$19.I2S_MICIN(GPIO_22)
- removed net SHDN: MCP1826G$1.!SHDN
- new net A0: JP3.5, U$2.PF7(ADC7)
- new net A1: JP3.6, U$2.PF6(ADC6)
- new net A2: JP3.7, U$2.PF5(ADC5)
- new net A3: JP3.8, U$2.PF4(ADC4)
- new net A4: JP3.9, U$2.PF1(ADC1)
- new net A5: JP3.10, U$2.PF0(ADC0)
- new net GPIO_23: JP3.32, U$19.GPIO_23
- new net I2S_CK: JP3.37, U$19.I2S_CK(GPIO_18), U$5.SCLK
- new net I2S_MCK: JP3.35, U$19.I2S_MCK(GPIO_21), U$5.MCLK
- new net I2S_MICIN: JP3.34, U$19.I2S_MICIN(GPIO_22)
- new net I2S_SD: JP3.36, U$19.I2S_SD(GPIO_20), U$5.SDATA
- new net I2S_WS: JP3.33, U$19.I2S_WS(GPIO_19), U$5.LRCLK
- new net JMP_START_LED: U$19.LED8(GPIO_26)
- new net JUMPSTART: U$19.JUMPSTART
- new net N$19: U$7.GND4, U$7.GND5, U$7.GND6, U$7.GND7
- new net N$21: U$7.EN2
- new net N$29: U$7.VCC1
- new net N$30: U$7.GND2
- new net N$40: U$7.GND3
- new net N$45: LED6.A, R26A.1
- new net N$46: LED5.A, R26B.1
- new net N$50: LED2.A, R26C.1
- new net N$52: LED1.A, R26D.1
- new net N$53: U$7.RFO2
- new net N$54: U$7.RFIN2
- new net N$55: U$7.GND
- new net N$56: U$7.VCC
- new net N$57: U$7.GND1
- new net PB0/SS: JP3.23, U$2.PB0(SS)
- new net PB4: JP3.17, U$2.PB4(ADC11)
- new net PB5: JP3.18, U$2.PB5(ADC12)
- new net PB6: JP3.19, U$2.PB6(ADC13)
- new net PB7: JP3.20, MCP1826G$1.!SHDN, R27.2, U$2.PB7
- new net PC6: JP3.14, U$2.PC6
- new net PC7: JP3.22, U$2.PC7
- new net PD4: JP3.13, U$2.PD4(ADC8)
- new net PD5: JP3.38, U$2.PD5
- new net PD6: JP3.21, U$2.PD6(ADC9)
- new net PD7: JP3.15, U$2.PD7(ADC10)
- new net PE6: JP3.16, U$2.PE6
- new net RESET: JP3.27
- new net RESET_CONFIG: JP3.28, R65.2, U$19.RESET_CONFIG
- new net SCL: JP3.12, U$2.PD0(SCL)
- new net SDA: JP3.11, U$2.PD1(SDA)
- new net SKW_SPI_CLK: JP3.31, U$19.SPI_CLK
- new net SKW_SPI_MISO: JP3.29, U$19.SPI_MISO
- new net SKW_SPI_MOSI: JP3.30, U$19.SPI_MOSI
- new net SYSTEM_LED: R26B.2, U$19.LED7(GPIO_27)
- new net USB_LED: R26D.2, U$19.LED1(GPIO_1)
- new net WIRELESS_LED: R26C.2, U$19.LED0(GPIO_0)
- net GND: now also JP3.2, JP3.39, JP3.4, JP3.40, LED1.C, LED2.C, LED5.C, LED6.C; no longer JP2.1, JP2.3
- net N$1: now also U$7.VC2G2; no longer R65.2, U$19.RESET_CONFIG
- net PB1/SCK: now also JP3.24
- net PB2/MOSI: now also JP3.25
- net PB3/MISO: now also JP3.26
- net VBUS: now also U$6.D@1, U$6.D@2; no longer Q1.D
- net VCC: now also C18.1, C8.1, JP3.3, LED3.A, LED4.A, MCP1826G$1.VIN, R13.2, R27.1, U$1.ADP, U$1.EN, U$1.EN0, U$6.C@1, U$6.C@2, U$6.S; no longer C4.+, D7.A, L1.2, Q1.G, R2.1
- net VDD: now also JP3.1, R26A.2; no longer R64.1
- net VSOURCE: now also C4.+, L1.2, R2.1, U$6.A, U$6.G; no longer C18.1, C8.1, D7.C, LED3.A, LED4.A, MCP1826G$1.VIN, Q1.S, R13.2, U$1.ADP, U$1.EN, U$1.EN0
Other:
- note added: "Atmega32u4"
- note added: "Battery Charger"
- note added: "Extension"
- note added: "I2S to Audio Jack"
- moved on the sheet: B1, C1, C10, C11, C12, C13, C14, C15, C16, C17, C18, C19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

Commit message: normal Push.
Parts:
- removed C2, C25: 1uF, SparkFun:CAP0402-CAP
- removed JP1: (no value), SparkFun-Connectors:AUDIO-JACK1:1
- removed R23, R24, R25: 22, SparkFun:RESISTOR0402-RES
- removed R47, R48, R53, R54: 330R, BaseApp:RESISTOR
- added SW1: (no value), BaseApp:TACTILE-2PIN'
- added X1: (no value), adafruit:ANTENNA_U.FL
- R14: value 22 -> 330; device SparkFun:RESISTOR0402-RES -> SparkFun-Passives:RESISTOR-ARRAY0603-ARV
- R3: value (none) -> 1k
- R6, R7: value 57.6k -> 1.5k
- U$5: value MAX5556ESA+ -> RF-SMA; device schematic:MAX5556ESA+ -> BaseApp:RF-SMA
Connections:
- removed net N$1: U$7.VC2G2
- removed net N$14: C20.2, U$1.OUT
- removed net N$21: U$7.EN2
- removed net N$27: R14.2, R23.2
- removed net N$35: R24.2, R25.2
- removed net N$49: C2.2, JP1.RIGHT, R14.1
- removed net N$51: C25.2, JP1.LEFT, R24.1
- removed net N$53: U$7.RFO2
- removed net N$55: U$7.GND
- removed net N$56: U$7.VCC
- removed net N$57: U$7.GND1
- removed net OUTL: C25.1, R25.1, U$5.OUTL
- removed net OUTR: C2.1, R23.1, U$5.OUTR
- new net RF2_OUT: U$5.1, U$7.RFO2
- new net VLITHIUM: C20.2, MCP1826G$1.VIN, U$1.OUT
- net ETH0_GRN+: now also R14D.1; no longer R54.2
- net GND: now also R14B.1, R14C.1, U$5.GND@1, U$5.GND@2, U$5.GND@3, U$7.GND, U$7.GND1, X1.GND@0, X1.GND@1; no longer JP1.SLEEVE, R47.2, R53.2
- net I2S_CK: no longer U$5.SCLK
- net I2S_MCK: no longer U$5.MCLK
- net I2S_SD: no longer U$5.SDATA
- net I2S_WS: no longer U$5.LRCLK
- net JUMPSTART: now also SW1.2
- net N$24: now also R14C.2; no longer R53.1
- net N$25: now also R14A.1; no longer R48.1
- net N$31: now also R14B.2; no longer R47.1
- net N$54: now also X1.SIGNAL
- net N$95: now also R14D.2; no longer R54.1
- net VCC: no longer MCP1826G$1.VIN, U$5.VDD
- net VDD: now also R14A.2, SW1.1, U$7.EN2, U$7.VC2G2, U$7.VCC; no longer R48.2
Other:
- note added: "WPS Button"
- note removed: "I2S to Audio Jack"
