File: Boards/baseVariant/schematic.brd (EAGLE design)
At the start: 160 x 100 mm, 122 parts, among them IC1 BQ24120

Commit message: Schematic Reframed.
Parts:
- removed C2: 100u, rcl:PANASONIC_D
- removed D8: ss14, SparkFun:SMA-DIODE
- removed JP5: (no value), jumper:JP1
- removed L1: 22uH, SparkFun:CR54
- removed NCP1: (no value), SparkFun:SOT23-5
- removed R31: 10K, resistor:R0603
Connections:
- removed net N$1: D8.A, L1.P$1, NCP1.5
- removed net N$33: R20.2
- removed net RC6: NCP1.1
- removed net VUSB: C2.+, D8.C, NCP1.2
- new net N$31: MCP1826.2
- new net SHDN: MCP1826.1
- net !SHDN: no longer MCP1826.1, R31.2
- net +3V3: no longer C13.1, C7.+, MCP1826.4, R22.1, R31.1
- net GND: now also R20.2; no longer C2.-, NCP1.4
- net VDD: now also C13.1, C7.+, MCP1826.4, R22.1; no longer L1.P$2
Changed lines of the file:
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@@
 <element name="JP1" library="SparkFun-Passives" package="SJ_2S" value="" x="-90.17" y="105.41"/>
 <element name="C7" library="adafruit" package="E2,5-6" value="220uf" x="-39.37" y="76.2"/>
-<element name="JP5" library="jumper" package="JP1" value="" x="-44.45" y="82.55"/>
-<element name="R31" library="resistor" package="R0603" value="10K" x="-72.39" y="88.9"/>
 <element name="LED1" library="adafruit" package="CHIP-LED0603" value="" x="-59.69" y="74.93"/>
 <element name="LED2" library="adafruit" package="CHIP-LED0603" value="" x="-63.5" y="74.93"/>
@@
 <element name="R58" library="BaseApp" package="R0603" value="1K" x="-91.44" y="95.25"/>
 <element name="RST_BRD" library="SparkFun-Connectors" package="MOLEX-1X2" value="" x="-57.15" y="67.31"/>
-<element name="NCP1" library="SparkFun" package="SOT23-5" value="" x="-57.15" y="100.33"/>
-<element name="L1" library="SparkFun" package="CR54" value="22uH" x="-62.23" y="67.31"/>
-<element name="C2" library="rcl" package="PANASONIC_D" value="100u" x="-99.06" y="67.31"/>
-<element name="D8" library="SparkFun" package="SMA-DIODE" value="ss14" x="-100.33" y="100.33"/>
 <element name="IC1" library="texas" package="QFN20_3,5X4,5" value="BQ24120" x="-109.22" y="5.08">
 <attribute name="OC_NEWARK" value="12M9386" x="-109.22" y="5.08" size="1.778" layer="27" display="off"/>
@@
 <contactref element="R58" pad="1"/>
 <contactref element="RST_BRD" pad="1"/>
-<contactref element="NCP1" pad="4"/>
-<contactref element="C2" pad="-"/>
 <contactref element="C29" pad="2"/>
 <contactref element="IC1" pad="16"/>
@@
 <contactref element="C8" pad="2"/>
 <contactref element="BAT" pad="3"/>
+<contactref element="R20" pad="2"/>
 <wire x1="-132.7" y1="-33.02" x2="-128.27" y2="-43.18" width="0" layer="19" extent="1-1"/>
-<wire x1="-126.38" y1="-21.59" x2="-132.7" y2="-33.02" width="0" layer="19" extent="1-1"/>
+<wire x1="-125.08" y1="-29.21" x2="-132.7" y2="-33.02" width="0" layer="19" extent="1-1"/>
+<wire x1="-126.38" y1="-21.59" x2="-125.08" y2="-29.21" width="0" layer="19" extent="1-1"/>
 <wire x1="-126.38" y1="-17.78" x2="-126.38" y2="-21.59" width="0" layer="19" extent="1-1"/>
 <wire x1="-125.08" y1="-13.97" x2="-126.38" y2="-17.78" width="0" layer="19" extent="1-1"/>
@@
 <wire x1="-87.6" y1="69.96" x2="-84.9" y2="67.31" width="0" layer="19" extent="1-1"/>
 <wire x1="-92.9" y1="67.31" x2="-87.6" y2="69.96" width="0" layer="19" extent="1-1"/>
-<wire x1="-101.46" y1="67.31" x2="-92.9" y2="67.31" width="0" layer="19" extent="1-1"/>
 <wire x1="-84.8106" y1="55.9054" x2="-84.9" y2="67.31" width="0" layer="19" extent="1-1"/>
 <wire x1="-88.48" y1="82.55" x2="-87.6" y2="69.96" width="0" layer="19" extent="1-1"/>
@@
 <wire x1="-50.38" y1="105.41" x2="-47.41" y2="100.33" width="0" layer="19" extent="1-1"/>
 <wire x1="-53.76" y1="105.41" x2="-50.38" y2="105.41" width="0" layer="19" extent="1-1"/>
-<wire x1="-56.2" y1="101.6301" x2="-53.76" y2="105.41" width="0" layer="19" extent="1-1"/>
-<wire x1="-60.23" y1="99.06" x2="-56.2" y2="101.6301" width="0" layer="19" extent="1-1"/>
 <wire x1="-43.6" y1="105.41" x2="-47.41" y2="100.33" width="0" layer="19" extent="1-1"/>
 <wire x1="-38.72" y1="105.41" x2="-43.6" y2="105.41" width="0" layer="19" extent="1-1"/>
+<wire x1="-60.23" y1="99.06" x2="-53.76" y2="105.41" width="0" layer="19" extent="1-1"/>
 <wire x1="-56.73" y1="88.9" x2="-60.23" y2="99.06" width="0" layer="19" extent="1-1"/>
 <wire x1="-51.65" y1="88.9" x2="-56.73" y2="88.9" width="0" layer="19" extent="1-1"/>
@@
 </signal>
 <signal name="+3V3">
-<contactref element="C13" pad="1"/>
-<contactref element="R22" pad="1"/>
-<contactref element="MCP1826" pad="4"/>
-<contactref element="C7" pad="+"/>
 <contactref element="3V3" pad="TP"/>
 <contactref element="R14" pad="1"/>
-<contactref element="R31" pad="1"/>
 <contactref element="R4" pad="1"/>
 <contactref element="R5" pad="1"/>
@@
 <wire x1="-36.41" y1="100.33" x2="-30.06" y2="100.33" width="0" layer="19" extent="1-1"/>
 <wire x1="-42.76" y1="100.33" x2="-36.41" y2="100.33" width="0" layer="19" extent="1-1"/>
-<wire x1="-49.11" y1="100.33" x2="-42.76" y2="100.33" width="0" layer="19" extent="1-1"/>
-<wire x1="-60.54" y1="105.41" x2="-49.11" y2="100.33" width="0" layer="19" extent="1-1"/>
-<wire x1="-65.62" y1="105.41" x2="-60.54" y2="105.41" width="0" layer="19" extent="1-1"/>
 <wire x1="-24.27" y1="76.2" x2="-29.63" y2="88.9" width="0" layer="19" extent="1-1"/>
 <wire x1="-34.29" y1="69.51" x2="-24.27" y2="76.2" width="0" layer="19" extent="1-1"/>
-<wire x1="-40.64" y1="76.2" x2="-34.29" y2="69.51" width="0" layer="19" extent="1-1"/>
-<wire x1="-63.08" y1="88.9" x2="-60.54" y2="105.41" width="0" layer="19" extent="1-1"/>
-<wire x1="-73.24" y1="88.9" x2="-63.08" y2="88.9" width="0" layer="19" extent="1-1"/>
-<wire x1="-71.12" y1="82.55" x2="-73.24" y2="88.9" width="0" layer="19" extent="1-1"/>
-<wire x1="-96.94" y1="88.9" x2="-73.24" y2="88.9" width="0" layer="19" extent="1-1"/>
+<wire x1="-60.54" y1="105.41" x2="-42.76" y2="100.33" width="0" layer="19" extent="1-1"/>
+<wire x1="-65.62" y1="105.41" x2="-60.54" y2="105.41" width="0" layer="19" extent="1-1"/>
+<wire x1="-71.12" y1="82.55" x2="-65.62" y2="105.41" width="0" layer="19" extent="1-1"/>
+<wire x1="-96.94" y1="88.9" x2="-71.12" y2="82.55" width="0" layer="19" extent="1-1"/>
 <wire x1="-52.83" y1="33.02" x2="-34.29" y2="69.51" width="0" layer="19" extent="1-1"/>
 <wire x1="-68.58" y1="12.7" x2="-52.83" y2="33.02" width="0" layer="19" extent="1-1"/>
 <wire x1="-86.36" y1="12.7" x2="-68.58" y2="12.7" width="0" layer="19" extent="1-1"/>
 <wire x1="-87.63" y1="12.7" x2="-86.36" y2="12.7" width="0" layer="19" extent="1-1"/>
-<wire x1="-80.01" y1="28.75" x2="-86.36" y2="12.7" width="0" layer="19" extent="1-1"/>
 </signal>
 <signal name="P-TX">
@@
 <contactref element="VDD" pad="TP"/>
 <contactref element="R28" pad="2"/>
-<contactref element="L1" pad="P$2"/>
+<contactref element="C13" pad="1"/>
+<contactref element="R22" pad="1"/>
+<contactref element="MCP1826" pad="4"/>
+<contactref element="C7" pad="+"/>
 <wire x1="-45.3" y1="105.41" x2="-14.39" y2="100.33" width="0" layer="19" extent="1-1"/>
-<wire x1="-55.46" y1="105.41" x2="-45.3" y2="105.41" width="0" layer="19" extent="1-1"/>
+<wire x1="-49.11" y1="100.33" x2="-45.3" y2="105.41" width="0" layer="19" extent="1-1"/>
+<wire x1="-55.46" y1="105.41" x2="-49.11" y2="100.33" width="0" layer="19" extent="1-1"/>
 <wire x1="-60.11" y1="95.25" x2="-55.46" y2="105.41" width="0" layer="19" extent="1-1"/>
-<wire x1="-66.04" y1="82.55" x2="-60.11" y2="95.25" width="0" layer="19" extent="1-1"/>
-<wire x1="-62.23" y1="65.39" x2="-66.04" y2="82.55" width="0" layer="19" extent="1-1"/>
-<wire x1="-40.64" y1="58.42" x2="-62.23" y2="65.39" width="0" layer="19" extent="1-1"/>
+<wire x1="-63.08" y1="88.9" x2="-60.11" y2="95.25" width="0" layer="19" extent="1-1"/>
+<wire x1="-66.04" y1="82.55" x2="-63.08" y2="88.9" width="0" layer="19" extent="1-1"/>
+<wire x1="-40.64" y1="76.2" x2="-49.11" y2="100.33" width="0" layer="19" extent="1-1"/>
+<wire x1="-40.64" y1="58.42" x2="-40.64" y2="76.2" width="0" layer="19" extent="1-1"/>
 <wire x1="-20.955" y1="51.99" x2="-40.64" y2="58.42" width="0" layer="19" extent="1-1"/>
+<wire x1="-80.01" y1="28.75" x2="-40.64" y2="58.42" width="0" layer="19" extent="1-1"/>
 </signal>
 <signal name="USB_D_N">
@@
 </signal>
 <signal name="!SHDN">
-<contactref element="MCP1826" pad="1"/>
-<contactref element="R31" pad="2"/>
 <contactref element="PIC25K50" pad="26"/>
-<wire x1="-28.575" y1="51.99" x2="-83.82" y2="28.75" width="0" layer="19" extent="1-1"/>
-<wire x1="-71.54" y1="88.9" x2="-28.575" y2="51.99" width="0" layer="19" extent="1-1"/>
 </signal>
 <signal name="RA0">
@@
 <wire x1="-54.61" y1="67.31" x2="-77.05" y2="95.25" width="0" layer="19" extent="1-1"/>
 </signal>
-<signal name="VUSB">
-<contactref element="NCP1" pad="2"/>
-<contactref element="C2" pad="+"/>
-<contactref element="D8" pad="C"/>
-<wire x1="-98.18" y1="100.33" x2="-57.15" y2="99.0299" width="0" layer="19" extent="1-1"/>
-<wire x1="-96.66" y1="67.31" x2="-98.18" y2="100.33" width="0" layer="19" extent="1-1"/>
-</signal>
-<signal name="N$1">
-<contactref element="NCP1" pad="5"/>
-<contactref element="L1" pad="P$1"/>
-<contactref element="D8" pad="A"/>
-<wire x1="-62.23" y1="69.23" x2="-58.1" y2="101.6301" width="0" layer="19" extent="1-1"/>
-<wire x1="-102.48" y1="100.33" x2="-58.1" y2="101.6301" width="0" layer="19" extent="1-1"/>
-</signal>
-<signal name="RC6">
-<contactref element="NCP1" pad="1"/>
-</signal>
 <signal name="VBUS">
 <contactref element="C29" pad="1"/>
@@
 <wire x1="-107.97" y1="3.355" x2="-125.08" y2="-17.78" width="0" layer="19" extent="1-1"/>
 </signal>
-<signal name="N$33">
-<contactref element="R20" pad="2"/>
-</signal>
 <signal name="NTC">
 <contactref element="IC1" pad="12"/>
@@
 <wire x1="-61.38" y1="88.9" x2="-78.74" y2="28.75" width="0" layer="19" extent="1-1"/>
 </signal>
+<signal name="SHDN">
+<contactref element="MCP1826" pad="1"/>
+</signal>
+<signal name="N$31">
+<contactref element="MCP1826" pad="2"/>
+</signal>
 </signals>

Commit message: Normal Push
Parts:
- removed U$31: PINHEAD-1X3, BaseApp:PINHEAD-1X3-2MM
- added SKW71_UART: (no value), SparkFun-Connectors:1X03_SMD_RA_MALE
Connections:
- net +3V3: no longer C62.2, C89.2, R59.1, R64.1, U$19.1, U$19.29, U$19.31, V-.2
- net GND: now also SKW71_UART.3; no longer U$31.3
- net SKW71_RX: now also SKW71_UART.1; no longer U$31.1
- net SKW71_TX: now also SKW71_UART.2; no longer U$31.2
- net VDD: now also C62.2, C89.2, R59.1, R64.1, U$19.1, U$19.29, U$19.31, V-.2
Changed lines of the file:
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@@
 <element name="C62" library="BaseApp" package="C0603" value="0.1u" x="-15.24" y="88.9"/>
 <element name="C89" library="BaseApp" package="C0603" value="1uf" x="-30.48" y="88.9"/>
-<element name="U$31" library="BaseApp" package="PINHEAD-1X3-2MM" value="PINHEAD-1X3" x="-62.23" y="99.06"/>
+<element name="SKW71_UART" library="SparkFun-Connectors" package="1X03_SMD_RA_MALE" value="" x="-62.23" y="99.06">
+<attribute name="PROD_ID" value="CONN-10925" x="-62.23" y="99.06" size="1.778" layer="27" display="off"/>
+</element>
 <element name="JP2" library="SparkFun-Connectors" package="MOLEX-1X4" value="" x="-40.64" y="82.55"/>
 <element name="R59" library="BaseApp" package="R0603" value="" x="-59.69" y="105.41"/>
@@
 <contactref element="U$19" pad="27"/>
 <contactref element="C89" pad="1"/>
-<contactref element="U$31" pad="3"/>
 <contactref element="JP2" pad="1"/>
 <contactref element="JP2" pad="3"/>
@@
 <contactref element="BAT" pad="3"/>
 <contactref element="R20" pad="2"/>
+<contactref element="SKW71_UART" pad="3"/>
 <wire x1="-132.7" y1="-33.02" x2="-128.27" y2="-43.18" width="0" layer="19" extent="1-1"/>
 <wire x1="-125.08" y1="-29.21" x2="-132.7" y2="-33.02" width="0" layer="19" extent="1-1"/>
@@
 <wire x1="-39.79" y1="95.25" x2="-31.33" y2="88.9" width="0" layer="19" extent="1-1"/>
 <wire x1="-47.41" y1="100.33" x2="-39.79" y2="95.25" width="0" layer="19" extent="1-1"/>
+<wire x1="-59.69" y1="104.06" x2="-47.41" y2="100.33" width="0" layer="19" extent="1-1"/>
 <wire x1="-50.38" y1="105.41" x2="-47.41" y2="100.33" width="0" layer="19" extent="1-1"/>
 <wire x1="-53.76" y1="105.41" x2="-50.38" y2="105.41" width="0" layer="19" extent="1-1"/>
 <wire x1="-43.6" y1="105.41" x2="-47.41" y2="100.33" width="0" layer="19" extent="1-1"/>
 <wire x1="-38.72" y1="105.41" x2="-43.6" y2="105.41" width="0" layer="19" extent="1-1"/>
-<wire x1="-60.23" y1="99.06" x2="-53.76" y2="105.41" width="0" layer="19" extent="1-1"/>
-<wire x1="-56.73" y1="88.9" x2="-60.23" y2="99.06" width="0" layer="19" extent="1-1"/>
-<wire x1="-51.65" y1="88.9" x2="-56.73" y2="88.9" width="0" layer="19" extent="1-1"/>
+<wire x1="-51.65" y1="88.9" x2="-59.69" y2="104.06" width="0" layer="19" extent="1-1"/>
+<wire x1="-56.73" y1="88.9" x2="-51.65" y2="88.9" width="0" layer="19" extent="1-1"/>
 </signal>
 <signal name="N$37">
@@
 <contactref element="R5" pad="1"/>
 <contactref element="R48" pad="2"/>
-<contactref element="U$19" pad="1"/>
-<contactref element="C62" pad="2"/>
-<contactref element="R64" pad="1"/>
-<contactref element="R59" pad="1"/>
-<contactref element="U$19" pad="29"/>
-<contactref element="C89" pad="2"/>
-<contactref element="U$19" pad="31"/>
-<contactref element="V-" pad="2"/>
 <contactref element="R13" pad="2"/>
 <contactref element="L4" pad="P$1"/>
 <contactref element="C64" pad="+"/>
-<wire x1="-29.63" y1="88.9" x2="-14.39" y2="88.9" width="0" layer="19" extent="1-1"/>
-<wire x1="-29.63" y1="95.25" x2="-29.63" y2="88.9" width="0" layer="19" extent="1-1"/>
-<wire x1="-30.06" y1="100.33" x2="-29.63" y2="95.25" width="0" layer="19" extent="1-1"/>
+<wire x1="-29.63" y1="95.25" x2="-30.06" y2="100.33" width="0" layer="19" extent="1-1"/>
 <wire x1="-36.41" y1="100.33" x2="-30.06" y2="100.33" width="0" layer="19" extent="1-1"/>
 <wire x1="-42.76" y1="100.33" x2="-36.41" y2="100.33" width="0" layer="19" extent="1-1"/>
-<wire x1="-24.27" y1="76.2" x2="-29.63" y2="88.9" width="0" layer="19" extent="1-1"/>
-<wire x1="-34.29" y1="69.51" x2="-24.27" y2="76.2" width="0" layer="19" extent="1-1"/>
-<wire x1="-60.54" y1="105.41" x2="-42.76" y2="100.33" width="0" layer="19" extent="1-1"/>
-<wire x1="-65.62" y1="105.41" x2="-60.54" y2="105.41" width="0" layer="19" extent="1-1"/>
-<wire x1="-71.12" y1="82.55" x2="-65.62" y2="105.41" width="0" layer="19" extent="1-1"/>
+<wire x1="-24.27" y1="76.2" x2="-29.63" y2="95.25" width="0" layer="19" extent="1-1"/>
+<wire x1="-71.12" y1="82.55" x2="-42.76" y2="100.33" width="0" layer="19" extent="1-1"/>
 <wire x1="-96.94" y1="88.9" x2="-71.12" y2="82.55" width="0" layer="19" extent="1-1"/>
-<wire x1="-52.83" y1="33.02" x2="-34.29" y2="69.51" width="0" layer="19" extent="1-1"/>
-<wire x1="-68.58" y1="12.7" x2="-52.83" y2="33.02" width="0" layer="19" extent="1-1"/>
-<wire x1="-86.36" y1="12.7" x2="-68.58" y2="12.7" width="0" layer="19" extent="1-1"/>
-<wire x1="-87.63" y1="12.7" x2="-86.36" y2="12.7" width="0" layer="19" extent="1-1"/>
+<wire x1="-52.83" y1="33.02" x2="-24.27" y2="76.2" width="0" layer="19" extent="1-1"/>
 </signal>
 <signal name="P-TX">
@@
 <contactref element="MCP1826" pad="4"/>
 <contactref element="C7" pad="+"/>
-<wire x1="-45.3" y1="105.41" x2="-14.39" y2="100.33" width="0" layer="19" extent="1-1"/>
-<wire x1="-49.11" y1="100.33" x2="-45.3" y2="105.41" width="0" layer="19" extent="1-1"/>
+<contactref element="U$19" pad="1"/>
+<contactref element="C62" pad="2"/>
+<contactref element="R64" pad="1"/>
+<contactref element="R59" pad="1"/>
+<contactref element="U$19" pad="29"/>
+<contactref element="C89" pad="2"/>
+<contactref element="U$19" pad="31"/>
+<contactref element="V-" pad="2"/>
+<wire x1="-14.39" y1="88.9" x2="-14.39" y2="100.33" width="0" layer="19" extent="1-1"/>
+<wire x1="-29.63" y1="88.9" x2="-14.39" y2="88.9" width="0" layer="19" extent="1-1"/>
+<wire x1="-40.64" y1="76.2" x2="-29.63" y2="88.9" width="0" layer="19" extent="1-1"/>
+<wire x1="-34.29" y1="69.51" x2="-40.64" y2="76.2" width="0" layer="19" extent="1-1"/>
+<wire x1="-40.64" y1="58.42" x2="-34.29" y2="69.51" width="0" layer="19" extent="1-1"/>
+<wire x1="-20.955" y1="51.99" x2="-40.64" y2="58.42" width="0" layer="19" extent="1-1"/>
+<wire x1="-49.11" y1="100.33" x2="-29.63" y2="88.9" width="0" layer="19" extent="1-1"/>
+<wire x1="-45.3" y1="105.41" x2="-49.11" y2="100.33" width="0" layer="19" extent="1-1"/>
 <wire x1="-55.46" y1="105.41" x2="-49.11" y2="100.33" width="0" layer="19" extent="1-1"/>
-<wire x1="-60.11" y1="95.25" x2="-55.46" y2="105.41" width="0" layer="19" extent="1-1"/>
+<wire x1="-60.54" y1="105.41" x2="-55.46" y2="105.41" width="0" layer="19" extent="1-1"/>
+<wire x1="-65.62" y1="105.41" x2="-60.54" y2="105.41" width="0" layer="19" extent="1-1"/>
+<wire x1="-60.11" y1="95.25" x2="-60.54" y2="105.41" width="0" layer="19" extent="1-1"/>
 <wire x1="-63.08" y1="88.9" x2="-60.11" y2="95.25" width="0" layer="19" extent="1-1"/>
 <wire x1="-66.04" y1="82.55" x2="-63.08" y2="88.9" width="0" layer="19" extent="1-1"/>
-<wire x1="-40.64" y1="76.2" x2="-49.11" y2="100.33" width="0" layer="19" extent="1-1"/>
-<wire x1="-40.64" y1="58.42" x2="-40.64" y2="76.2" width="0" layer="19" extent="1-1"/>
-<wire x1="-20.955" y1="51.99" x2="-40.64" y2="58.42" width="0" layer="19" extent="1-1"/>
 <wire x1="-80.01" y1="28.75" x2="-40.64" y2="58.42" width="0" layer="19" extent="1-1"/>
+<wire x1="-86.36" y1="12.7" x2="-80.01" y2="28.75" width="0" layer="19" extent="1-1"/>
+<wire x1="-87.63" y1="12.7" x2="-86.36" y2="12.7" width="0" layer="19" extent="1-1"/>
+<wire x1="-68.58" y1="12.7" x2="-86.36" y2="12.7" width="0" layer="19" extent="1-1"/>
 </signal>
 <signal name="USB_D_N">
@@
 <signal name="SKW71_RX">
 <contactref element="U$19" pad="37"/>
-<contactref element="U$31" pad="1"/>
-<wire x1="-64.23" y1="99.06" x2="-91.44" y2="12.7" width="0" layer="19" extent="1-1"/>
+<contactref element="SKW71_UART" pad="1"/>
+<wire x1="-64.77" y1="104.06" x2="-91.44" y2="12.7" width="0" layer="19" extent="1-1"/>
 </signal>
 <signal name="SKW71_TX">
 <contactref element="U$19" pad="38"/>
-<contactref element="U$31" pad="2"/>
-<wire x1="-62.23" y1="99.06" x2="-91.44" y2="16.085" width="0" layer="19" extent="1-1"/>
+<contactref element="SKW71_UART" pad="2"/>
+<wire x1="-62.23" y1="104.06" x2="-91.44" y2="16.085" width="0" layer="19" extent="1-1"/>
 </signal>
 <signal name="GPIO_21">
@@
 <wire x1="-35.49" y1="69.51" x2="-33.09" y2="69.51" width="0" layer="19" extent="1-1"/>
 <wire x1="-70.7" y1="105.41" x2="-35.49" y2="69.51" width="0" layer="19" extent="1-1"/>
-</signal>
-<signal name="N$97">
-<contactref element="R65" pad="2"/>
-<contactref element="U$19" pad="23"/>
-<wire x1="-69" y1="105.41" x2="-82.55" y2="12.7" width="0" layer="19" extent="1-1"/>
 </signal>
 <signal name="N$44">
@@
 <contactref element="MCP1826" pad="2"/>
 </signal>
+<signal name="N$1">
+<contactref element="U$19" pad="23"/>
+<contactref element="R65" pad="2"/>
+<wire x1="-69" y1="105.41" x2="-82.55" y2="12.7" width="0" layer="19" extent="1-1"/>
+</signal>
 </signals>
