File: Boards/baseVariant/schematic.brd (EAGLE design)
At the start: 93 x 70 mm, 98 parts, among them IC1 LM2596S, J1 AVR_SPI_PRG_6NS, Q1 BSS84, U1 MAGJACK-POE, U2 MAGJACK-POE

Commit message: normal Push.
Parts:
- removed D7: BA340A, SparkFun-DiscreteSemi:SMA-DIODE
- removed JP2: (no value), SparkFun-Connectors:MOLEX-1X4
- removed Q1: BSS84, transistor-small-signal:SOT23
- removed R64: (no value), BaseApp:R0603
- added JP3: (no value), pinhead:2X20
- added R26: (no value), SparkFun-Passives:0603-ARV
- added R27: (no value), SparkFun-Passives:0402-RES
- added U$6: FDFMA2P857, BaseApp:6-WDFN-EXPOSED-PAD
- added U$7: SE2580L, schematic:SE2580L
- R2: value (none) -> 10k
- moved U$5 17.6 mm to (25.1, 33.2), turned to 90 degrees
- moved U$19 7.95 mm to (31.4, 39.6)
- moved L2 6.89 mm to (59.1, 54.5)
- moved R65 4.88 mm to (18.6, 36.3), flipped to the bottom
- moved C62 3.82 mm to (33.7, 44.2)
- moved C1 2.00 mm to (25.7, 22.0)
- moved C15 2.00 mm to (11.7, 31.0)
- moved C16 2.00 mm to (11.7, 34.0)
- moved C17 2.00 mm to (11.7, 25.0)
- moved C32 2.00 mm to (11.7, 28.0)
- moved D1 2.00 mm to (39.0, 26.2)
- moved R15 2.00 mm to (21.7, 22.0)
- moved R16 2.00 mm to (38.7, 38.0)
- moved R17 2.00 mm to (40.7, 38.0)
- moved R19 2.00 mm to (17.7, 22.0)
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Connections:
- removed net GPIO_18: U$19.13, U$5.2
- removed net GPIO_19: JP2.4, U$19.5, U$5.3
- removed net GPIO_20: U$19.11, U$5.1
- removed net GPIO_21: U$19.9, U$5.4
- removed net GPIO_22: JP2.2, R64.2, U$19.7
- removed net SHDN: MCP1826.1
- new net A0: JP3.5, U$2.36
- new net A1: JP3.6, U$2.37
- new net A2: JP3.7, U$2.38
- new net A3: JP3.8, U$2.39
- new net A4: JP3.9, U$2.40
- new net A5: JP3.10, U$2.41
- new net GPIO_23: JP3.32, U$19.3
- new net I2S_CK: JP3.37, U$19.13, U$5.2
- new net I2S_MCK: JP3.35, U$19.9, U$5.4
- new net I2S_MICIN: JP3.34, U$19.7
- new net I2S_SD: JP3.36, U$19.11, U$5.1
- new net I2S_WS: JP3.33, U$19.5, U$5.3
- new net JMP_START_LED: U$19.21
- new net JUMPSTART: U$19.25
- new net N$19: U$7.P$17, U$7.P$18, U$7.P$19, U$7.P$20
- new net N$21: U$7.P$8
- new net N$29: U$7.P$9
- new net N$30: U$7.P$12
- new net N$40: U$7.P$14
- new net N$45: LED6.A, R26.1
- new net N$46: LED5.A, R26.2
- new net N$50: LED2.A, R26.3
- new net N$52: LED1.A, R26.4
- new net N$53: U$7.P$15
- new net N$54: U$7.P$1
- new net N$55: U$7.P$2
- new net N$56: U$7.P$3
- new net N$57: U$7.P$4
- new net PB0/SS: JP3.23, U$2.8
- new net PB4: JP3.17, U$2.28
- new net PB5: JP3.18, U$2.29
- new net PB6: JP3.19, U$2.30
- new net PB7: JP3.20, MCP1826.1, R27.2, U$2.12
- new net PC6: JP3.14, U$2.31
- new net PC7: JP3.22, U$2.32
- new net PD4: JP3.13, U$2.25
- new net PD5: JP3.38, U$2.22
- new net PD6: JP3.21, U$2.26
- new net PD7: JP3.15, U$2.27
- new net PE6: JP3.16, U$2.1
- new net RESET: JP3.27
- new net RESET_CONFIG: JP3.28, R65.2, U$19.23
- new net SCL: JP3.12, U$2.18
- new net SDA: JP3.11, U$2.19
- new net SKW_SPI_CLK: JP3.31, U$19.30
- new net SKW_SPI_MISO: JP3.29, U$19.28
- new net SKW_SPI_MOSI: JP3.30, U$19.32
- new net SYSTEM_LED: R26.7, U$19.19
- new net USB_LED: R26.5, U$19.35
- new net WIRELESS_LED: R26.6, U$19.36
- net GND: now also JP3.2, JP3.39, JP3.4, JP3.40, LED1.K, LED2.K, LED5.K, LED6.K; no longer JP2.1, JP2.3
- net N$1: now also U$7.P$16; no longer R65.2, U$19.23
- net PB1/SCK: now also JP3.24
- net PB2/MOSI: now also JP3.25
- net PB3/MISO: now also JP3.26
- net VBUS: now also U$6.D@1, U$6.D@2; no longer Q1.3
- net VCC: now also C18.1, C8.1, JP3.3, LED3.A, LED4.A, MCP1826.2, R13.2, R27.1, U$1.P$3, U$1.P$7, U$1.P$8, U$6.C@1, U$6.C@2, U$6.S; no longer C4.+, D7.A, L1.P$2, Q1.1, R2.1
- net VDD: now also JP3.1, R26.8; no longer R64.1
- net VSOURCE: now also C4.+, L1.P$2, R2.1, U$6.A, U$6.G; no longer C18.1, C8.1, D7.C, LED3.A, LED4.A, MCP1826.2, Q1.2, R13.2, U$1.P$3, U$1.P$7, U$1.P$8
Other:
- outline, holes or cut-outs redrawn

Commit message: normal Push.
Parts:
- removed C2, C25: 1uF, SparkFun:0402-CAP
- removed JP1: (no value), SparkFun-Connectors:STEREOJACK2.5MM
- removed R23, R24, R25: 22, SparkFun:0402-RES
- removed R47, R48, R53, R54: 330R, BaseApp:R0603
- added SW1: (no value), BaseApp:TACTILE-2PIN-RTANGLE
- added X1: (no value), adafruit:U.FL
- R14: value 22 -> 330; device SparkFun:0402-RES -> SparkFun-Passives:0603-ARV
- R3: value (none) -> 1k
- R6, R7: value 57.6k -> 1.5k
- U$5: value MAX5556ESA+ -> RF-SMA; device schematic:SO-8 -> BaseApp:BU-SMA-H
- moved V- 59.9 mm to (62.4, 0.77), flipped to the bottom
- moved U$5 32.6 mm to (6.86, 6.25), flipped to the top, turned to 270 degrees
- moved R14 23.5 mm to (39.6, 8.84), flipped to the top
- moved C10 18.5 mm to (48.7, 32.0)
- moved C17 18.1 mm to (27.2, 34.3), flipped to the bottom, turned to 0 degrees
- moved C16 17.8 mm to (27.2, 25.3), flipped to the bottom, turned to 180 degrees
- moved R21 15.9 mm to (23.4, 28.0), flipped to the bottom, turned to 180 degrees
- moved C32 15.9 mm to (27.2, 31.3), flipped to the bottom, turned to 0 degrees
- moved C15 15.8 mm to (27.2, 28.3), flipped to the bottom, turned to 0 degrees
- moved U$4 15.3 mm to (33.8, 29.8)
- moved U2 15.1 mm to (30.0, 9.19)
- moved U1 14.9 mm to (49.4, 9.19)
- moved USB1 14.0 mm to (59.0, -2.61)
- moved R11 12.3 mm to (65.1, 19.5)
- moved U$7 9.21 mm to (11.1, 16.6)
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Connections:
- removed net N$1: U$7.P$16
- removed net N$14: C20.2, U$1.P$14
- removed net N$21: U$7.P$8
- removed net N$27: R14.2, R23.2
- removed net N$35: R24.2, R25.2
- removed net N$49: C2.2, JP1.4, R14.1
- removed net N$51: C25.2, JP1.1, R24.1
- removed net N$53: U$7.P$15
- removed net N$55: U$7.P$2
- removed net N$56: U$7.P$3
- removed net N$57: U$7.P$4
- removed net OUTL: C25.1, R25.1, U$5.8
- removed net OUTR: C2.1, R23.1, U$5.5
- new net RF2_OUT: U$5.1, U$7.P$15
- new net VLITHIUM: C20.2, MCP1826.2, U$1.P$14
- net ETH0_GRN+: now also R14.4; no longer R54.2
- net GND: now also R14.2, R14.3, U$5.2, U$5.3, U$5.4, U$5.5, U$7.P$2, U$7.P$4, X1.1, X1.2; no longer JP1.5, R47.2, R53.2, U$5.6
- net I2S_CK: no longer U$5.2
- net I2S_MCK: no longer U$5.4
- net I2S_SD: no longer U$5.1
- net I2S_WS: no longer U$5.3
- net JUMPSTART: now also SW1.2
- net N$24: now also R14.6; no longer R53.1
- net N$25: now also R14.1; no longer R48.1
- net N$31: now also R14.7; no longer R47.1
- net N$54: now also X1.3
- net N$95: now also R14.5; no longer R54.1
- net VCC: no longer MCP1826.2, U$5.7
- net VDD: now also R14.8, SW1.1, U$7.P$16, U$7.P$3, U$7.P$8; no longer R48.2
