File: Boards/bulkVariant/schematic.sch (EAGLE design)
At the start: 99 parts, among them IC1 LM2596S, J1 AVR_SPI_PRG_6NS, U1 MAGJACK-POE, U2 MAGJACK-POE

Commit message: normal Push.
Parts:
- added U$11: USB_FEMALE_A_STACKED_2, schematic:USB_FEMALE_A_STACKED_2
Changed lines of the file:
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@@
 <setting verticaltext="up"/>
 </settings>
-<grid distance="0.05" unitdist="inch" unit="inch" style="lines" multiple="1" display="yes" altdistance="0.025" altunitdist="inch" altunit="inch"/>
+<grid distance="0.1" unitdist="inch" unit="inch" style="lines" multiple="1" display="no" altdistance="0.01" altunitdist="inch" altunit="inch"/>
 <layers>
 <layer number="1" name="Top" color="4" fill="1" visible="no" active="no"/>
@@
 <part name="R28" library="SparkFun-Passives" deviceset="RESISTOR" device="0402-RES"/>
 <part name="C25" library="SparkFun-Capacitors" deviceset="CAP" device="0402-CAP"/>
+<part name="U$11" library="schematic" deviceset="USB_FEMALE_A_STACKED_2" device=""/>
 </parts>
 <sheets>
@@
 <instance part="R28" gate="G$1" x="330.2" y="238.76" rot="R90"/>
 <instance part="C25" gate="G$1" x="346.71" y="240.03" rot="R180"/>
+<instance part="U$11" gate="G$1" x="248.92" y="218.44"/>
 </instances>
 <busses>
