File: Boards/modularVariant/schematic.sch (EAGLE design)
At the start: 75 parts, among them IC1 LM2596S, U1 MAGJACK-POE, U2 MAGJACK-POE

Commit message: Normal Push.
Parts:
- added JP1: (no value), pinhead:PINHD-2X6
- added U3: PIC16F1503-X_MG, pic16f1503_qfn_mg:PIC16F1503-X_MG
Changed lines of the file:
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@@
 <part name="R14" library="SparkFun-Passives" deviceset="RESISTOR-ARRAY" device="0603-ARV" value="330"/>
 <part name="SW1" library="BaseApp" deviceset="TACTILE-2PIN" device="'"/>
+<part name="JP1" library="pinhead" deviceset="PINHD-2X6" device=""/>
+<part name="U3" library="pic16f1503_qfn_mg" deviceset="PIC16F1503-X_MG" device=""/>
 </parts>
 <sheets>
@@
 <instance part="R14" gate="D" x="502.92" y="86.36" rot="R90"/>
 <instance part="SW1" gate="G$1" x="34.29" y="317.5"/>
+<instance part="JP1" gate="A" x="492.76" y="313.69"/>
+<instance part="U3" gate="A" x="59.69" y="240.03"/>
 </instances>
 <busses>

Commit message: normal Push.
Parts:
- removed JP1: (no value), pinhead:PINHD-2X6
- removed LED1, LED2, LED5, LED6: (no value), led:LED3MM
- removed R26: (no value), SparkFun-Passives:RESISTOR-ARRAY0603-ARV
- removed R65: (no value), BaseApp:RESISTOR
- removed U3: PIC16F1503-X_MG, pic16f1503_qfn_mg:PIC16F1503-X_MG
- removed V-: SPST-3PIN-RTANGLEP02, BaseApp:SPST-3PIN-RTANGLEP02
- added $$U$1, $$U$2, $$U$3, $$U$4: LIGHT_PIPE, BaseApp:LIGHT_PIPE
- added C2: (no value), SparkFun-Passives:CAP0402-CAP
- added C5: (no value), SparkFun-Capacitors:CAP0402-CAP
- added DL1, DL2, DL3, DL4: (no value), BaseApp:DUOLED-1X2
- added EXT: (no value), pinhead:PINHD-2X8
- added J1: AVR_SPI_PRG_6OFFSET_PADS, SparkFun-Connectors:AVR_SPI_PRG_6OFFSET_PADS
- added R10, R5: (no value), SparkFun-Resistors:RESISTOR-ARRAY0603-ARV
- added R23: 3.2k, SparkFun-Passives:RESISTOR0402-RES
- added R4: (no value), SparkFun-Passives:RESISTOR0402-RES
- added R9: 1k, SparkFun-Passives:RESISTOR0402-RES
- added SJ1, SJ2: (no value), BaseApp:JUMPER
- added SKW_UART: (no value), SparkFun-Connectors:M03PTH
- added U$2: ATTINY84, SparkFun-DigitalIC:ATTINY84
- C13, C19, C20, C21, C8: device rcl:C-EUC0603 -> rcl:C-EUC0402
- R22: device resistor:R-EU_R0603 -> resistor:R-EU_R0402
Connections:
- removed net N$22: R6.1, U$1.STAT1N
- removed net N$28: R7.1, U$1.STAT2N
- removed net N$45: LED6.A, R26A.1
- removed net N$46: LED5.A, R26B.1
- removed net N$50: LED2.A, R26C.1
- removed net N$52: LED1.A, R26D.1
- removed net PB7: MCP1826G$1.!SHDN, R27.2
- new net ATTINY_RESET: J1.5, R4.1, U$2.(PCINT11/~RESET/DW)PB3
- new net LED_A: EXT.13, R5A.1
- new net LED_B: EXT.14, R5B.1
- new net N$1: DL2.A1, R10R.2
- new net N$14: SJ1.1, U$2.(PCINT9/XTAL2)PB1
- new net N$17: DL3.A2, R5B.2
- new net N$19: DL4.A1, R5R.2
- new net N$21: SJ2.1, U$2.(PCINT8/XTAL1/CLKI)PB0
- new net N$29: DL4.A2, R5D.2
- new net N$3: DL1.A1, R10A.2
- new net N$30: SW1.1, U$2.(PCINT10/INT0/OC0A/CKOUT)PB2
- new net N$35: DL3.A1, R5A.2
- new net N$4: DL2.A2, R10D.2
- new net N$40: DL1.A2, R10B.2
- new net PA0: R5R.1, U$2.(PCINT0/AREF/ADC0)PA0
- new net PA1: R5D.1, U$2.(PCINT1/AIN0/ADC1)PA1
- new net PA4: EXT.16, J1.3, U$2.(PCINT4/T1/SCL/USCK/ADC4)PA4
- new net PA5: J1.1, U$2.(PCINT5/OC1B/MISO/DO/ADC5)PA5
- new net PA6: EXT.15, J1.4, U$2.(PCINT6/OC1A/SDA/MOSI/ADC6)PA6
- new net POWER_CTRL: MCP1826G$1.!SHDN, R27.2, U$2.(PCINT7/ICP/OC0B/ADC7)PA7
- new net STAT1: R6.1, SJ1.2, U$1.STAT1N
- new net STAT2: R7.1, SJ2.2, U$1.STAT2N
- net GND: now also C2.2, DL1.C1, DL1.C2, DL2.C1, DL2.C2, DL3.C1, DL3.C2, DL4.C1, DL4.C2, EXT.10, EXT.2, EXT.4, J1.6, R23.2, SKW_UART.1, SW1.2, U$2.GND; no longer LED1.C, LED2.C, LED5.C, LED6.C
- net I2S_CK: now also EXT.9
- net I2S_MCK: now also EXT.7
- net I2S_MICIN: now also EXT.6
- net I2S_SD: now also EXT.8
- net I2S_WS: now also EXT.5
- net JMP_START_LED: now also R10A.1
- net JUMPSTART: now also U$2.(PCINT2/AIN1/ADC2)PA2; no longer SW1.2
- net N$26: now also C5.1, IC1.FB, R23.1, R9.1; no longer R65.1, V-.1, V-.3
- net PD2/RXD: now also EXT.12, SKW_UART.2
- net PD3/TXD: now also EXT.11, SKW_UART.3
- net RESET_CONFIG: now also U$2.(PCINT3/T0/ADC3)PA3; no longer R65.2
- net SYSTEM_LED: now also R10B.1; no longer R26B.2
- net USB_LED: now also R10D.1; no longer R26D.2
- net VCC: now also EXT.3; no longer IC1.FB, R27.1
- net VDD: now also EXT.1; no longer R26A.2, SW1.1, V-.2
- net VLITHIUM: now also C2.1, J1.2, R27.1, R4.2, U$2.VCC
- net VSOURCE: now also C5.2, R9.2
- net WIRELESS_LED: now also R10R.1; no longer R26C.2
Other:
- note removed: "WPS Button"
- moved on the sheet: D3, SW1

Commit message: normal Push.
Parts:
- J1: value AVR_SPI_PRG_6OFFSET_PADS -> AVR_SPI_PRG_6NS; device SparkFun-Connectors:AVR_SPI_PRG_6OFFSET_PADS -> SparkFun-Connectors:AVR_SPI_PRG_6NS
Changed lines of the file:
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@@
 <part name="C2" library="SparkFun-Passives" deviceset="CAP" device="0402-CAP"/>
 <part name="R4" library="SparkFun-Passives" deviceset="RESISTOR" device="0402-RES"/>
-<part name="J1" library="SparkFun-Connectors" deviceset="AVR_SPI_PRG_6" device="OFFSET_PADS"/>
+<part name="J1" library="SparkFun-Connectors" deviceset="AVR_SPI_PRG_6" device="NS" value="AVR_SPI_PRG_6NS"/>
 <part name="SKW_UART" library="SparkFun-Connectors" deviceset="M03" device="PTH"/>
 <part name="GND16" library="SparkFun-Aesthetics" deviceset="GND" device=""/>

Commit message: normal Push.
Parts:
- added C6, C9: 33pF, SparkFun-Capacitors:CAP0402-CAP
- added JP1: M05X2PTH, SparkFun-Connectors:M05X2PTH
- added Q1: FC-12M, crystal:FC-12M
- C18: device rcl:C-EUC0603 -> rcl:C-EUC0402
- C28: value 1000uf/35V -> 1000uf/10V
Connections:
- net GND: now also C6.2, C9.2, EXT.16, JP1.10, JP1.2, JP1.4, JP1.6, JP1.8
- net GPIO_23: now also EXT.15
- net N$14: now also C6.1, Q1.2; no longer SJ1.1
- net N$21: now also C9.1, Q1.1; no longer SJ2.1
- net PA4: now also SJ1.1; no longer EXT.16
- net PA6: now also SJ2.1; no longer EXT.15
- net VCC: now also JP1.3, JP1.7
- net VDD: now also JP1.1, JP1.9
- net VIN: now also JP1.5
Other:
- moved on the sheet: EXT, SJ1, SJ2
