File: Boards/modularVariant/schematic.sch (EAGLE design)
At the start: 93 parts, among them IC1 LM2596S, J1 AVR_SPI_PRG_6NS, Q1 FC-12M, U1 MAGJACK-POE, U2 MAGJACK-POE

Commit message: normal Push.
Parts:
- added R24, R25, R26: 330, SparkFun-Passives:RESISTOR0402-RES
- R14: device SparkFun-Passives:RESISTOR-ARRAY0603-ARV -> SparkFun-Passives:RESISTOR0402-RES
Connections:
- net ETH0_GRN+: now also R24.2; no longer R14D.1
- net GND: now also R14.2, R26.1; no longer R14B.1, R14C.1
- net N$24: now also R14.1; no longer R14C.2
- net N$25: now also R25.2; no longer R14A.1
- net N$31: now also R26.2; no longer R14B.2
- net N$95: now also R24.1; no longer R14D.2
- net VDD: now also R25.1; no longer R14A.2
Changed lines of the file:
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@@
 </variantdefs>
 <classes>
-<class number="0" name="default" width="0.2032" drill="0.3048">
+<class number="0" name="default" width="0.1524" drill="0.3048">
 <clearance class="0" value="0.1524"/>
 </class>
-<class number="1" name="power" width="0.2032" drill="0.3048">
+<class number="1" name="power" width="0.1524" drill="0.3048">
 <clearance class="1" value="0.1524"/>
 </class>
-<class number="2" name="gnd" width="0.2032" drill="0.3048">
+<class number="2" name="gnd" width="0.1524" drill="0.3048">
 <clearance class="2" value="0.1524"/>
 </class>
@@
 <part name="R27" library="SparkFun-Passives" deviceset="RESISTOR" device="0402-RES"/>
 <part name="U$6" library="BaseApp" deviceset="FDFMA2P857" device=""/>
-<part name="R14" library="SparkFun-Passives" deviceset="RESISTOR-ARRAY" device="0603-ARV" value="330"/>
 <part name="SW1" library="BaseApp" deviceset="TACTILE-2PIN" device="'"/>
 <part name="EXT" library="pinhead" deviceset="PINHD-2X8" device=""/>
@@
 <part name="C9" library="SparkFun-Capacitors" deviceset="CAP" device="0402-CAP" value="33pF"/>
 <part name="JP1" library="SparkFun-Connectors" deviceset="M05X2" device="PTH"/>
+<part name="R24" library="SparkFun-Passives" deviceset="RESISTOR" device="0402-RES" value="330"/>
+<part name="R14" library="SparkFun-Passives" deviceset="RESISTOR" device="0402-RES" value="330"/>
+<part name="R25" library="SparkFun-Passives" deviceset="RESISTOR" device="0402-RES" value="330"/>
+<part name="R26" library="SparkFun-Passives" deviceset="RESISTOR" device="0402-RES" value="330"/>
 </parts>
 <sheets>
@@
 <instance part="R27" gate="G$1" x="137.16" y="54.61" rot="R180"/>
 <instance part="U$6" gate="G$1" x="193.04" y="85.09"/>
-<instance part="R14" gate="A" x="497.84" y="149.86" rot="R180"/>
-<instance part="R14" gate="B" x="508" y="149.86" rot="R90"/>
-<instance part="R14" gate="C" x="496.57" y="104.14" rot="R180"/>
-<instance part="R14" gate="D" x="502.92" y="86.36" rot="R90"/>
 <instance part="SW1" gate="G$1" x="158.75" y="238.76"/>
 <instance part="EXT" gate="A" x="520.7" y="295.91"/>
@@
 <instance part="C9" gate="G$1" x="200.66" y="227.33" rot="R90"/>
 <instance part="JP1" gate="G$1" x="461.01" y="295.91"/>
+<instance part="R24" gate="G$1" x="509.27" y="86.36" rot="R270"/>
+<instance part="R14" gate="G$1" x="496.57" y="104.14"/>
+<instance part="R25" gate="G$1" x="497.84" y="149.86"/>
+<instance part="R26" gate="G$1" x="508" y="149.86" rot="R90"/>
 </instances>
 <busses>
@@
 <wire x1="504.19" y1="104.14" x2="501.65" y2="104.14" width="0.1524" layer="91"/>
 <junction x="504.19" y="104.14"/>
-<pinref part="R14" gate="C" pin="1"/>
+<pinref part="R14" gate="G$1" pin="2"/>
+<junction x="501.65" y="104.14"/>
 </segment>
 <segment>
@@
 <wire x1="508" y1="144.78" x2="508" y2="140.97" width="0.1524" layer="91"/>
 <label x="508" y="140.97" size="1.016" layer="95" rot="R180" xref="yes"/>
-<pinref part="R14" gate="B" pin="1"/>
+<pinref part="R26" gate="G$1" pin="1"/>
+<junction x="508" y="144.78"/>
 </segment>
 <segment>
@@
 <wire x1="492.76" y1="149.86" x2="490.22" y2="149.86" width="0.1524" layer="91"/>
 <label x="490.22" y="149.86" size="1.016" layer="95" rot="R180" xref="yes"/>
-<pinref part="R14" gate="A" pin="2"/>
+<pinref part="R25" gate="G$1" pin="1"/>
+<junction x="492.76" y="149.86"/>
 </segment>
 <segment>
@@
 <junction x="488.95" y="93.98"/>
 <wire x1="502.92" y1="93.98" x2="488.95" y2="93.98" width="0.1524" layer="91"/>
-<pinref part="R14" gate="D" pin="2"/>
+<pinref part="R24" gate="G$1" pin="1"/>
+<junction x="509.27" y="91.44"/>
+<wire x1="502.92" y1="91.44" x2="509.27" y2="91.44" width="0.1524" layer="91"/>
 </segment>
 </net>
@@
 <wire x1="502.92" y1="81.28" x2="502.92" y2="68.58" width="0.1524" layer="91"/>
 <label x="502.92" y="68.58" size="1.778" layer="95" rot="R90"/>
-<pinref part="R14" gate="D" pin="1"/>
+<pinref part="R24" gate="G$1" pin="2"/>
+<junction x="509.27" y="81.28"/>
+<wire x1="509.27" y1="81.28" x2="502.92" y2="81.28" width="0.1524" layer="91"/>
 </segment>
 <segment>
@@
 <junction x="488.95" y="154.94"/>
 <wire x1="508" y1="154.94" x2="488.95" y2="154.94" width="0.1524" layer="91"/>
-<pinref part="R14" gate="B" pin="2"/>
+<pinref part="R26" gate="G$1" pin="2"/>
+<junction x="508" y="154.94"/>
 </segment>
 </net>
@@
 <wire x1="488.95" y1="144.78" x2="502.92" y2="144.78" width="0.1524" layer="91"/>
 <wire x1="502.92" y1="144.78" x2="502.92" y2="149.86" width="0.1524" layer="91"/>
-<pinref part="R14" gate="A" pin="1"/>
+<pinref part="R25" gate="G$1" pin="2"/>
+<junction x="502.92" y="149.86"/>
 </segment>
 </net>
@@
 <junction x="488.95" y="104.14"/>
 <wire x1="491.49" y1="104.14" x2="488.95" y2="104.14" width="0.1524" layer="91"/>
-<pinref part="R14" gate="C" pin="2"/>
-</segment>
-</net>
+<pinref part="R14" gate="G$1" pin="1"/>
+<junction x="491.49" y="104.14"/>
+</segment>
+</net>

Commit message: normal Push.
Parts:
- removed IC1: LM2596S, national-semiconductor:LM2596S
- removed L1: 33uH 3A, schematic:INDUCTOR
- added C14: 56pF, SparkFun-Capacitors:CAP0402-CAP
- added C22: 10nF, SparkFun-Capacitors:CAP0402-CAP
- added L4: 6.8uH, WE-PD:WE-PD-7447715006_1260/1245/1280/1210
- added R28: 100k, SparkFun-Passives:RESISTOR0402-RES
- added R29: 3k, SparkFun-Passives:RESISTOR0402-RES
- added U$5: SKY87608, schematic:SKY87608
- C5: value (none) -> 0.1uF
- R23: value 3.2k -> 20k
- R9: value 1k -> 91k
Connections:
- new net CMP: C14.2, C22.2, U$5.CMP
- new net N$22: R28.1, U$5.EN
- new net N$27: R23.1, R9.1, U$5.FB
- new net N$37: C22.1, R29.2
- net GND: now also C14.1, R29.1, U$5.GND; no longer EXT.10, EXT.16, IC1.!ON!/OFF, IC1.GND
- net GPIO_23: now also EXT.11; no longer EXT.15
- net N$2: now also C5.2, L4.1, U$5.LX; no longer IC1.OUT, L1.1
- net N$26: now also U$5.BST; no longer IC1.FB, R23.1, R9.1
- net PA0: now also SJ2.1; no longer R5R.1
- net PA1: now also SJ1.1; no longer R5D.1
- net PA4: no longer SJ1.1
- net PA5: now also R5R.1
- net PA6: now also R5D.1; no longer SJ2.1
- net PD3/TXD: now also EXT.10; no longer EXT.11
- net USB_D_N: now also EXT.16
- net USB_D_P: now also EXT.15
- net VIN: now also R28.2, U$5.IN; no longer IC1.VIN
- net VSOURCE: now also L4.2; no longer C5.2, L1.2
Other:
- moved on the sheet: C5

Commit message: normal Push.
Parts:
- removed L4: 6.8uH, WE-PD:WE-PD-7447715006_1260/1245/1280/1210
- added U$7: 6.8uH 0302, schematic:INDUCTOR_0302
Connections:
- net N$2: now also U$7.1; no longer L4.1
- net VSOURCE: now also U$7.2; no longer L4.2
Changed lines of the file:
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@@
 <part name="C22" library="SparkFun-Capacitors" deviceset="CAP" device="0402-CAP" value="10nF"/>
 <part name="R29" library="SparkFun-Passives" deviceset="RESISTOR" device="0402-RES" value="3k"/>
-<part name="L4" library="WE-PD" deviceset="WE-PD" device="_1260/1245/1280/1210" technology="-7447715006" value="6.8uH"/>
+<part name="U$7" library="schematic" deviceset="INDUCTOR_0302" device="" value="6.8uH 0302"/>
 </parts>
 <sheets>
@@
 <instance part="C22" gate="G$1" x="187.96" y="129.54" rot="R180"/>
 <instance part="R29" gate="G$1" x="182.88" y="120.65"/>
-<instance part="L4" gate="G$1" x="119.38" y="134.62"/>
+<instance part="U$7" gate="G$1" x="119.38" y="134.62" rot="R90"/>
 </instances>
 <busses>
@@
 <wire x1="129.54" y1="134.62" x2="134.62" y2="134.62" width="0.1524" layer="91"/>
 <label x="134.62" y="134.62" size="1.27" layer="95" xref="yes"/>
-<pinref part="L4" gate="G$1" pin="2"/>
-<junction x="124.46" y="134.62"/>
-<wire x1="124.46" y1="134.62" x2="129.54" y2="134.62" width="0.1524" layer="91"/>
+<wire x1="127" y1="134.62" x2="129.54" y2="134.62" width="0.1524" layer="91"/>
+<pinref part="U$7" gate="G$1" pin="2"/>
+<junction x="127" y="134.62"/>
 </segment>
 <segment>
@@
 <wire x1="102.87" y1="133.35" x2="102.87" y2="134.62" width="0.1524" layer="91"/>
 <wire x1="106.68" y1="137.16" x2="109.22" y2="137.16" width="0.1524" layer="91"/>
-<pinref part="L4" gate="G$1" pin="1"/>
-<junction x="114.3" y="134.62"/>
-<wire x1="109.22" y1="134.62" x2="114.3" y2="134.62" width="0.1524" layer="91"/>
-</segment>
-</net>
+<wire x1="109.22" y1="134.62" x2="111.76" y2="134.62" width="0.1524" layer="91"/>
+<pinref part="U$7" gate="G$1" pin="1"/>
+<junction x="111.76" y="134.62"/>
+</segment>
+</net>

Commit message: normal Push.
Parts:
- removed L2: 33uh, BaseApp:INDUCTOR
- removed SKW_UART: (no value), SparkFun-Connectors:M03PTH
- added U$11, U$12, U$13, U$14, U$15, U$16, U$17, U$9: FIDUCIAL, adafruit:FIDUCIAL
- added U$18: SRR0735A-330M, schematic:SRR0735A-330M
Connections:
- removed net N$10: D1.A, L2.1, U$4.SWO
- new net N$38: D1.A, U$18.1, U$4.SWO
- net GND: now also U$18.2; no longer L2.2, SKW_UART.1
- net PD2/RXD: no longer SKW_UART.2
- net PD3/TXD: no longer SKW_UART.3
Other:
- note added: "32.768kHz"
- note added: "FIDUCIAL"
Changed lines of the file:
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@@
 <part name="D1" library="SparkFun-DiscreteSemi" deviceset="DIODE" device="SMC/DO-214AB"/>
 <part name="C12" library="adafruit2" deviceset="CPOL-US" device="E5-10.5" value="470uf/50V"/>
-<part name="L2" library="BaseApp" deviceset="INDUCTOR" device="" value="33uh"/>
 <part name="R16" library="BaseApp" deviceset="RESISTOR" device="" value="R1"/>
 <part name="R17" library="BaseApp" deviceset="RESISTOR" device="" value="R2"/>
@@
 <part name="R4" library="SparkFun-Passives" deviceset="RESISTOR" device="0402-RES"/>
 <part name="J1" library="SparkFun-Connectors" deviceset="AVR_SPI_PRG_6" device="NS" value="AVR_SPI_PRG_6NS"/>
-<part name="SKW_UART" library="SparkFun-Connectors" deviceset="M03" device="PTH"/>
 <part name="GND16" library="SparkFun-Aesthetics" deviceset="GND" device=""/>
 <part name="DL1" library="BaseApp" deviceset="DUOLED-1X2" device=""/>
@@
 <part name="R29" library="SparkFun-Passives" deviceset="RESISTOR" device="0402-RES" value="3k"/>
 <part name="U$7" library="schematic" deviceset="INDUCTOR_0302" device="" value="6.8uH 0302"/>
+<part name="U$9" library="adafruit" deviceset="FIDUCIAL" device=""/>
+<part name="U$11" library="adafruit" deviceset="FIDUCIAL" device=""/>
+<part name="U$12" library="adafruit" deviceset="FIDUCIAL" device=""/>
+<part name="U$13" library="adafruit" deviceset="FIDUCIAL" device=""/>
+<part name="U$14" library="adafruit" deviceset="FIDUCIAL" device=""/>
+<part name="U$15" library="adafruit" deviceset="FIDUCIAL" device=""/>
+<part name="U$16" library="adafruit" deviceset="FIDUCIAL" device=""/>
+<part name="U$17" library="adafruit" deviceset="FIDUCIAL" device=""/>
+<part name="U$18" library="schematic" deviceset="SRR0735A-330M" device=""/>
 </parts>
 <sheets>
@@
 <wire x1="115.57" y1="59.69" x2="115.57" y2="3.81" width="1.9304" layer="94" style="shortdash"/>
 <text x="45.72" y="64.77" size="5.08" layer="94">Battery Charger</text>
+<text x="441.96" y="334.01" size="5.08" layer="94" font="vector" ratio="15">FIDUCIAL</text>
+<text x="181.61" y="227.33" size="1.778" layer="94">32.768kHz</text>
 </plain>
 <instances>
@@
 <attribute name="VALUE" x="376.301" y="145.796" size="1.778" layer="96" rot="R90"/>
 </instance>
-<instance part="L2" gate="G$1" x="356.87" y="142.24" rot="R90"/>
 <instance part="R16" gate="G$1" x="392.43" y="154.94" rot="R270"/>
 <instance part="R17" gate="G$1" x="392.43" y="170.18" rot="R270"/>
@@
 <instance part="R4" gate="G$1" x="139.7" y="243.84" rot="R90"/>
 <instance part="J1" gate="G$1" x="106.68" y="180.34"/>
-<instance part="SKW_UART" gate="G$1" x="21.59" y="300.99"/>
 <instance part="GND16" gate="1" x="276.86" y="237.49"/>
 <instance part="DL1" gate="G$1" x="266.7" y="245.11"/>
@@
 <instance part="R29" gate="G$1" x="182.88" y="120.65"/>
 <instance part="U$7" gate="G$1" x="119.38" y="134.62" rot="R90"/>
+<instance part="U$9" gate="G$1" x="444.5" y="358.14"/>
+<instance part="U$11" gate="G$1" x="454.66" y="358.14"/>
+<instance part="U$12" gate="G$1" x="464.82" y="358.14"/>
+<instance part="U$13" gate="G$1" x="474.98" y="358.14"/>
+<instance part="U$14" gate="G$1" x="444.5" y="347.98"/>
+<instance part="U$15" gate="G$1" x="454.66" y="347.98"/>
+<instance part="U$16" gate="G$1" x="464.82" y="347.98"/>
+<instance part="U$17" gate="G$1" x="474.98" y="347.98"/>
+<instance part="U$18" gate="G$1" x="358.14" y="142.24"/>
 </instances>
 <busses>
@@
 </segment>
 <segment>
-<pinref part="L2" gate="G$1" pin="2"/>
 <pinref part="C12" gate="G$1" pin="-"/>
 <wire x1="364.49" y1="142.24" x2="372.11" y2="142.24" width="0.1524" layer="91"/>
@@
 <pinref part="GND2" gate="1" pin="GND"/>
 <junction x="416.56" y="142.24"/>
+<junction x="364.49" y="142.24"/>
+<pinref part="U$18" gate="G$1" pin="2"/>
+<junction x="360.68" y="142.24"/>
+<wire x1="360.68" y1="142.24" x2="364.49" y2="142.24" width="0.1524" layer="91"/>
 </segment>
 <segment>
@@
 <wire x1="116.84" y1="177.8" x2="124.46" y2="177.8" width="0.1524" layer="91"/>
 <label x="124.46" y="177.8" size="1.016" layer="95" xref="yes"/>
-</segment>
-<segment>
-<pinref part="SKW_UART" gate="G$1" pin="1"/>
-<junction x="29.21" y="298.45"/>
-<wire x1="29.21" y1="298.45" x2="31.75" y2="298.45" width="0.1524" layer="91"/>
-<label x="31.75" y="298.45" size="1.016" layer="95" xref="yes"/>
 </segment>
 <segment>
@@
 <wire x1="328.93" y1="55.88" x2="328.93" y2="43.18" width="0.1524" layer="91"/>
 <pinref part="R15" gate="G$1" pin="1"/>
-</segment>
-</net>
-<net name="N$10" class="0">
-<segment>
-<pinref part="U$4" gate="G$1" pin="SWO"/>
-<pinref part="D1" gate="G$1" pin="A"/>
-<wire x1="341.63" y1="101.6" x2="341.63" y2="142.24" width="0.1524" layer="91"/>
-<pinref part="L2" gate="G$1" pin="1"/>
-<wire x1="341.63" y1="142.24" x2="341.63" y2="149.86" width="0.1524" layer="91"/>
-<wire x1="341.63" y1="142.24" x2="349.25" y2="142.24" width="0.1524" layer="91"/>
-<junction x="341.63" y="142.24"/>
 </segment>
 </net>
@@
 </segment>
 <segment>
-<pinref part="SKW_UART" gate="G$1" pin="2"/>
-<junction x="29.21" y="300.99"/>
-<wire x1="29.21" y1="300.99" x2="31.75" y2="300.99" width="0.1524" layer="91"/>
-<label x="31.75" y="300.99" size="1.016" layer="95" xref="yes"/>
-</segment>
-<segment>
 <pinref part="EXT" gate="A" pin="12"/>
 <junction x="525.78" y="290.83"/>
@@
 <wire x1="86.36" y1="314.96" x2="69.85" y2="314.96" width="0.1524" layer="91"/>
 <label x="69.85" y="314.96" size="1.27" layer="95" rot="R180" xref="yes"/>
-</segment>
-<segment>
-<pinref part="SKW_UART" gate="G$1" pin="3"/>
-<junction x="29.21" y="303.53"/>
-<wire x1="29.21" y1="303.53" x2="31.75" y2="303.53" width="0.1524" layer="91"/>
-<label x="31.75" y="303.53" size="1.016" layer="95" xref="yes"/>
 </segment>
 <segment>
@@
 </segment>
 </net>
+<net name="N$38" class="0">
+<segment>
+<pinref part="U$18" gate="G$1" pin="1"/>
+<junction x="353.06" y="142.24"/>
+<pinref part="U$4" gate="G$1" pin="SWO"/>
+<pinref part="D1" gate="G$1" pin="A"/>
+<wire x1="341.63" y1="101.6" x2="341.63" y2="142.24" width="0.1524" layer="91"/>
+<wire x1="341.63" y1="142.24" x2="341.63" y2="149.86" width="0.1524" layer="91"/>
+<wire x1="341.63" y1="142.24" x2="349.25" y2="142.24" width="0.1524" layer="91"/>
+<junction x="341.63" y="142.24"/>
+<junction x="349.25" y="142.24"/>
+<wire x1="353.06" y1="142.24" x2="349.25" y2="142.24" width="0.1524" layer="91"/>
+</segment>
+</net>
