File: Boards/modularVariant/schematic.brd (EAGLE design)
At the start: 93 x 70 mm, 100 parts, among them IC1 LM2596S, J1 AVR_SPI_PRG_6NS, U1 MAGJACK-POE, U2 MAGJACK-POE

Commit message: normal Push.
Parts:
- removed C14, C22, C5, C6, C9: (no value), SparkFun:0402-CAP
- removed C2, C25: (no value), SparkFun-Capacitors:0402-CAP
- removed C23: 1uF, SparkFun:0402-CAP
- removed J1: AVR_SPI_PRG_6NS, Sensor Mesh:2X3-NS
- removed JP1: (no value), SparkFun-Connectors:AUDIO-JACK-3.5MM-SMD
- removed JP3: (no value), pinhead:2X20
- removed R10, R9: 1k, SparkFun:0402-RES
- removed R23, R24, R25, R28: (no value), SparkFun-Passives:0402-RES
- removed R4, R5: 22, SparkFun:0402-RES
- removed U$11: USB_FEMALE_A_STACKED_2, schematic:USB_A_FEMALE_STACKED_2
- removed U$2: ATMEGA32U4QFN, SparkFun-DigitalIC:QFN-44
- removed U$5: RF-SMA, BaseApp:BU-SMA-H
- removed U$7: SE2580L, schematic:SE2580L
- removed U$9: MAX5556ESA+, schematic:SO-8
- removed X1: (no value), adafruit:U.FL
- moved USB1 43.2 mm to (56.3, -2.46)
- moved V- 41.9 mm to (59.7, 0.92)
- moved JP4 30.7 mm to (69.8, 2.39)
- moved C29 26.1 mm to (69.8, 2.64)
- moved SW1 15.7 mm to (10.2, 1.22)
- moved U2 11.0 mm to (25.0, 9.19)
- moved R14 11.0 mm to (34.6, 8.84)
- moved U$3 11.0 mm to (46.0, 13.8)
- moved U1 11.0 mm to (44.4, 9.19)
- moved R22 9.99 mm to (75.3, 52.4)
- moved C62 9.15 mm to (33.8, 53.3)
- moved C1 9.15 mm to (31.3, 31.3)
- moved C11 9.15 mm to (36.4, 32.0)
- moved R15 9.15 mm to (27.3, 31.3)
- moved R19 9.15 mm to (23.3, 31.3)
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Connections:
- removed net A0: JP3.5, U$2.36
- removed net A1: JP3.6, U$2.37
- removed net A2: JP3.7, U$2.38
- removed net A3: JP3.8, U$2.39
- removed net A4: JP3.9, U$2.40
- removed net A5: JP3.10, U$2.41
- removed net AT_RESET: J1.5, R10.1, U$2.13
- removed net N$14: R23.1, R24.2, U$9.8
- removed net N$19: U$7.P$17, U$7.P$18, U$7.P$19, U$7.P$20
- removed net N$27: R25.1, R28.2, U$9.5
- removed net N$29: U$7.P$9
- removed net N$30: U$7.P$12
- removed net N$37: C23.2, U$2.6
- removed net N$38: R4.2, U$2.4
- removed net N$39: R5.2, U$2.3
- removed net N$40: U$7.P$14
- removed net N$43: R9.2, U$2.33
- removed net N$54: U$7.P$1, X1.3
- removed net N$58: C2.2, JP1.RING, R23.2
- removed net N$62: C25.2, JP1.TIP, R25.2
- removed net PB0/SS: JP3.23, U$2.8
- removed net PB1/SCK: J1.3, JP3.24, U$2.9
- removed net PB2/MOSI: J1.4, JP3.25, U$2.10
- removed net PB3/MISO: J1.1, JP3.26, U$2.11
- removed net PB4: JP3.17, U$2.28
- removed net PB5: JP3.18, U$2.29
- removed net PB6: JP3.19, U$2.30
- removed net PC6: JP3.14, U$2.31
- removed net PC7: JP3.22, U$2.32
- removed net PD4: JP3.13, U$2.25
- removed net PD5: JP3.38, U$2.22
- removed net PD6: JP3.21, U$2.26
- removed net PD7: JP3.15, U$2.27
- removed net PE6: JP3.16, U$2.1
- removed net RESET: JP3.27
- removed net RF2_OUT: U$5.1, U$7.P$15
- removed net SCL: JP3.12, U$2.18
- removed net SDA: JP3.11, U$2.19
- net GND: no longer C14.2, C2.1, C22.2, C23.1, C25.1, C5.2, C6.2, C9.2, J1.6, JP1.SLEEVE, JP3.2, JP3.39, JP3.4, JP3.40, R24.1, R28.1, R9.1, U$2.15, U$2.23, U$2.35, U$2.43, U$2.5, U$5.2, U$5.3, U$5.4, U$5.5, U$7.P$2, U$7.P$4, U$9.6, X1.1, X1.2
- net GPIO_23: no longer JP3.32
- net I2S_CK: no longer JP3.37, U$9.2
- net I2S_MCK: no longer JP3.35, U$9.4
- net I2S_MICIN: no longer JP3.34
- net I2S_SD: no longer JP3.36, U$9.1
- net I2S_WS: no longer JP3.33, U$9.3
- net PB7: no longer JP3.20, U$2.12
- net PD2/RXD: no longer U$2.20
- net PD3/TXD: no longer U$2.21
- net RESET_CONFIG: no longer JP3.28
- net SKW_SPI_CLK: no longer JP3.31
- net SKW_SPI_MISO: no longer JP3.29
- net SKW_SPI_MOSI: no longer JP3.30
- net USB_D_N: no longer R5.1
- net USB_D_P: no longer R4.1
- net VBUS: no longer U$2.2, U$2.7
- net VCC: no longer C14.1, C22.1, C5.1, C6.1, C9.1, J1.2, JP3.3, R10.2, U$2.14, U$2.24, U$2.34, U$2.42, U$2.44
- net VDD: no longer JP3.1, U$7.P$16, U$7.P$3, U$7.P$8, U$9.7

Commit message: Normal Push.
Parts:
- added JP1: (no value), pinhead:2X06
- added U3: PIC16F1503-X_MG, pic16f1503_qfn_mg:QFN16_3X3MC
- moved U$10 8.61 mm to (29.2, 32.6), turned to 90 degrees
- moved C24 5.18 mm to (40.3, 25.8)
- moved C1 3.66 mm to (31.2, 27.7)
- moved C11 3.66 mm to (36.2, 28.3)
- moved C15 3.66 mm to (27.2, 33.8)
- moved C17 3.66 mm to (27.2, 39.8)
- moved C32 3.66 mm to (27.2, 36.8)
- moved C62 3.66 mm to (33.7, 49.7)
- moved R15 3.66 mm to (27.2, 27.7)
- moved R19 3.66 mm to (23.2, 27.7)
- moved R21 3.66 mm to (23.4, 33.5)
- moved R8 3.66 mm to (25.2, 27.7)
- moved U$4 3.66 mm to (33.8, 35.3)
- moved C16 3.66 mm to (27.2, 30.8)
- moved D1 3.66 mm to (42.1, 31.7)
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Connections:
- new net VSS: U3.13
- net VDD: now also U3.16

Commit message: normal Push.
Parts:
- removed JP1: (no value), pinhead:2X06
- removed LED1, LED2, LED5, LED6: (no value), led:LED3MM
- removed R26: (no value), SparkFun-Passives:0603-ARV
- removed R65: (no value), BaseApp:R0603
- removed U3: PIC16F1503-X_MG, pic16f1503_qfn_mg:QFN16_3X3MC
- removed V-: SPST-3PIN-RTANGLEP02, BaseApp:TL3340AF160QG
- added $$U$1, $$U$2, $$U$3, $$U$4: LIGHT_PIPE, BaseApp:LIGHT-PIPE
- added C2: (no value), SparkFun-Passives:0402-CAP
- added C5: (no value), SparkFun-Capacitors:0402-CAP
- added DL1, DL2, DL3, DL4: (no value), BaseApp:DUOLED-C-0603
- added EXT: (no value), pinhead:2X08
- added J1: AVR_SPI_PRG_6OFFSET_PADS, SparkFun-Connectors:2X3_OFFSET
- added R10, R5: (no value), SparkFun-Resistors:0603-ARV
- added R23: 3.2k, SparkFun-Passives:0402-RES
- added R4: (no value), SparkFun-Passives:0402-RES
- added R9: 1k, SparkFun-Passives:0402-RES
- added SJ1, SJ2: (no value), BaseApp:SJW
- added SKW_UART: (no value), SparkFun-Connectors:1X03
- added U$2: ATTINY84, SparkFun-DigitalIC:SO14
- C13, C19, C20, C21, C8: device rcl:C0603 -> rcl:C0402
- R22: device resistor:R0603 -> resistor:R0402
- moved LED3 66.6 mm to (64.0, 5.15), turned to 0 degrees
- moved LED4 65.5 mm to (65.2, 5.15), turned to 0 degrees
- moved R6 60.9 mm to (64.0, 7.62), turned to 270 degrees
- moved R7 59.7 mm to (65.1, 7.62), turned to 270 degrees
- moved R13 46.2 mm to (67.5, 12.0)
- moved R2 32.9 mm to (67.9, 19.5), turned to 0 degrees
- moved C8 32.1 mm to (68.9, 17.8), turned to 90 degrees
- moved R3 24.7 mm to (76.4, 12.8), turned to 180 degrees
- moved C13 24.0 mm to (59.2, 49.9), turned to 0 degrees
- moved D5 22.1 mm to (73.6, 14.8), turned to 0 degrees
- moved L2 22.0 mm to (42.6, 47.8)
- moved MCP1826 21.1 mm to (54.0, 48.8), turned to 90 degrees
- moved D6 20.8 mm to (78.3, 16.3)
- moved R22 20.3 mm to (55.0, 52.7)
- moved D4 19.8 mm to (73.6, 18.5), turned to 0 degrees
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Connections:
- removed net N$22: R6.1, U$1.P$4
- removed net N$28: R7.1, U$1.P$6
- removed net N$45: LED6.A, R26.1
- removed net N$46: LED5.A, R26.2
- removed net N$50: LED2.A, R26.3
- removed net N$52: LED1.A, R26.4
- removed net PB7: MCP1826.1, R27.2
- removed net VSS: U3.13
- new net ATTINY_RESET: J1.5, R4.1, U$2.4
- new net LED_A: EXT.13, R5.1
- new net LED_B: EXT.14, R5.2
- new net N$1: DL2.A1, R10.6
- new net N$14: SJ1.1, U$2.3
- new net N$17: DL3.A2, R5.7
- new net N$19: DL4.A1, R5.6
- new net N$21: SJ2.1, U$2.2
- new net N$29: DL4.A2, R5.5
- new net N$3: DL1.A1, R10.8
- new net N$30: SW1.1, U$2.5
- new net N$35: DL3.A1, R5.8
- new net N$4: DL2.A2, R10.5
- new net N$40: DL1.A2, R10.7
- new net PA0: R5.3, U$2.13
- new net PA1: R5.4, U$2.12
- new net PA4: EXT.16, J1.3, U$2.9
- new net PA5: J1.1, U$2.8
- new net PA6: EXT.15, J1.4, U$2.7
- new net POWER_CTRL: MCP1826.1, R27.2, U$2.6
- new net STAT1: R6.1, SJ1.2, U$1.P$4
- new net STAT2: R7.1, SJ2.2, U$1.P$6
- net GND: now also C2.2, DL1.C1, DL1.C2, DL2.C1, DL2.C2, DL3.C1, DL3.C2, DL4.C1, DL4.C2, EXT.10, EXT.2, EXT.4, J1.6, R23.2, SKW_UART.1, SW1.2, U$2.14; no longer LED1.K, LED2.K, LED5.K, LED6.K
- net I2S_CK: now also EXT.9
- net I2S_MCK: now also EXT.7
- net I2S_MICIN: now also EXT.6
- net I2S_SD: now also EXT.8
- net I2S_WS: now also EXT.5
- net JMP_START_LED: now also R10.1
- net JUMPSTART: now also U$2.11; no longer SW1.2
- net N$26: now also C5.1, IC1.4, R23.1, R9.1; no longer R65.1, V-.1, V-.3
- net PD2/RXD: now also EXT.12, SKW_UART.2
- net PD3/TXD: now also EXT.11, SKW_UART.3
- net RESET_CONFIG: now also U$2.10; no longer R65.2
- net SYSTEM_LED: now also R10.2; no longer R26.7
- net USB_LED: now also R10.4; no longer R26.5
- net VCC: now also EXT.3; no longer IC1.4, R27.1
- net VDD: now also EXT.1; no longer R26.8, SW1.1, U3.16, V-.2
- net VLITHIUM: now also C2.1, J1.2, R27.1, R4.2, U$2.1
- net VSOURCE: now also C5.2, R9.2
- net WIRELESS_LED: now also R10.3; no longer R26.6

Commit message: normal Push.
Parts:
- J1: value AVR_SPI_PRG_6OFFSET_PADS -> AVR_SPI_PRG_6NS; device SparkFun-Connectors:2X3_OFFSET -> SparkFun-Connectors:2X3-NS
Changed lines of the file:
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@@
 <element name="C2" library="SparkFun-Passives" package="0402-CAP" value="" x="56.388" y="26.67" rot="R180"/>
 <element name="R4" library="SparkFun-Passives" package="0402-RES" value="" x="64.3128" y="24.8412" rot="R270"/>
-<element name="J1" library="SparkFun-Connectors" package="2X3_OFFSET" value="AVR_SPI_PRG_6OFFSET_PADS" x="75.438" y="29.2608" rot="R270"/>
+<element name="J1" library="SparkFun-Connectors" package="2X3-NS" value="AVR_SPI_PRG_6NS" x="75.438" y="29.2608" rot="R270"/>
 <element name="SKW_UART" library="SparkFun-Connectors" package="1X03" value="" x="8.9916" y="58.8264" rot="R270"/>
 <element name="DL1" library="BaseApp" package="DUOLED-C-0603" value="" x="24" y="66.5" rot="R90"/>

Commit message: normal Push.
Parts:
- added C6, C9: 33pF, SparkFun-Capacitors:0402-CAP
- added JP1: M05X2PTH, SparkFun-Connectors:AVR_ICSP
- added Q1: FC-12M, crystal:FC-12M
- C18: device rcl:C0603 -> rcl:C0402
- C28: value 1000uf/35V -> 1000uf/10V
- moved EXT 33.9 mm to (32.9, 56.1)
- moved D1 16.5 mm to (25.9, 35.1)
- moved C12 16.4 mm to (16.9, 57.1), turned to 90 degrees
- moved C24 15.5 mm to (25.2, 26.9)
- moved R15 15.5 mm to (12.1, 28.7)
- moved R19 15.5 mm to (8.09, 28.7)
- moved R21 15.5 mm to (8.27, 34.6)
- moved R8 15.5 mm to (10.1, 28.7)
- moved C1 15.5 mm to (16.1, 28.7)
- moved C11 15.5 mm to (21.1, 29.4)
- moved C15 15.5 mm to (12.2, 34.8)
- moved C16 15.5 mm to (12.2, 31.8)
- moved R16 15.5 mm to (16.3, 41.1)
- moved R17 15.5 mm to (22.7, 41.2)
- moved U$10 15.5 mm to (14.1, 33.7)
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Connections:
- net GND: now also C6.2, C9.2, EXT.16, JP1.10, JP1.2, JP1.4, JP1.6, JP1.8
- net GPIO_23: now also EXT.15
- net N$14: now also C6.1, Q1.2; no longer SJ1.1
- net N$21: now also C9.1, Q1.1; no longer SJ2.1
- net PA4: now also SJ1.1; no longer EXT.16
- net PA6: now also SJ2.1; no longer EXT.15
- net VCC: now also JP1.3, JP1.7
- net VDD: now also JP1.1, JP1.9
- net VIN: now also JP1.5

Commit message: normal Push.
Parts:
- added R24, R25, R26: 330, SparkFun-Passives:0402-RES
- R14: device SparkFun-Passives:0603-ARV -> SparkFun-Passives:0402-RES
- moved SW1 72.4 mm to (82.6, 1.07)
- moved C10 16.8 mm to (33.5, 26.0), turned to 270 degrees
- moved D5 16.6 mm to (87.8, 24.4)
- moved R21 16.6 mm to (24.8, 33.7), flipped to the top
- moved U$3 16.3 mm to (45.4, 12.8), flipped to the top
- moved R27 13.9 mm to (79.4, 33.8), turned to 90 degrees
- moved C17 13.8 mm to (24.8, 35.4), flipped to the top, turned to 180 degrees
- moved JP1 13.0 mm to (48.8, 29.9)
- moved C19 12.8 mm to (68.7, 20.4), flipped to the top
- moved C32 12.7 mm to (24.8, 37.2), flipped to the top, turned to 180 degrees
- moved D6 11.9 mm to (90.1, 19.2)
- moved CN2 10.8 mm to (72.3, 20.5)
- moved LED3 10.1 mm to (54.0, 5.30)
- moved R6 9.77 mm to (54.2, 7.93)
- moved R7 9.47 mm to (55.7, 7.93)
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Connections:
- net ETH0_GRN+: now also R24.2; no longer R14.4
- net GND: now also R26.1; no longer R14.3
- net N$24: now also R14.1; no longer R14.6
- net N$25: now also R25.2; no longer R14.1
- net N$31: now also R26.2; no longer R14.7
- net N$95: now also R24.1; no longer R14.5
- net VDD: now also R25.1; no longer R14.8
Routing:
- net GND: track 0.00 -> 1490.6 mm, vias 0 -> 18
- net VCC: track 0.00 -> 784.4 mm, vias 0 -> 7
- net VDD: track 0.00 -> 614.0 mm, vias 0 -> 16
- net PD_VDC: track 0.00 -> 536.7 mm, vias 0 -> 15
- net ETH0_GRN-: track 0.00 -> 496.4 mm, vias 0 -> 17
- net +57: track 0.00 -> 370.0 mm, vias 0 -> 4
- net N$6: track 0.00 -> 330.6 mm, vias 0 -> 10
- net VIN: track 0.00 -> 329.4 mm, vias 0 -> 3
- net PA6: track 0.00 -> 250.7 mm, vias 0 -> 1
- net PA4: track 0.00 -> 220.2 mm, vias 0 -> 1
- net VSOURCE: track 0.00 -> 217.5 mm, vias 0 -> 8
- net VLITHIUM: track 0.00 -> 203.3 mm, vias 0 -> 4
- net PD3/TXD: track 0.00 -> 187.7 mm, vias 0 -> 6
- net N$15: track 0.00 -> 175.3 mm, vias 0 -> 4
- net +2V: track 0.00 -> 169.7 mm, vias 0 -> 2
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
Commit message: normal Push.
Parts:
- removed IC1: LM2596S, national-semiconductor:TO263-5
- removed L1: 33uH 3A, schematic:INDUCTOR-10X9.8X6
- added C14: 56pF, SparkFun-Capacitors:0402-CAP
- added C22: 10nF, SparkFun-Capacitors:0402-CAP
- added L4: 6.8uH, WE-PD:WE-PD_1260/1245/1280/1210
- added R28: 100k, SparkFun-Passives:0402-RES
- added R29: 3k, SparkFun-Passives:0402-RES
- added U$5: SKY87608, schematic:8PIN-SOP-8L-EP
- C5: value (none) -> 0.1uF
- R23: value 3.2k -> 20k
- R9: value 1k -> 91k
- moved L2 52.3 mm to (6.12, 27.7), turned to 180 degrees
- moved C28 43.2 mm to (13.7, 59.0), turned to 180 degrees
- moved LED4 29.7 mm to (52.9, 34.8), turned to 180 degrees
- moved LED3 29.5 mm to (55.6, 34.8), turned to 180 degrees
- moved D6 26.8 mm to (65.1, 28.8), turned to 0 degrees
- moved JP1 26.6 mm to (43.3, 55.9)
- moved EXT 25.8 mm to (38.6, 30.9), turned to 0 degrees
- moved C6 25.6 mm to (71.8, 49.1)
- moved C9 25.6 mm to (70.0, 49.1)
- moved R4 25.5 mm to (72.8, 50.7)
- moved J1 25.2 mm to (82.0, 55.3)
- moved R7 24.7 mm to (53.0, 32.5), turned to 90 degrees
- moved R6 24.6 mm to (55.6, 32.5), turned to 90 degrees
- moved Q1 24.5 mm to (70.9, 50.9)
- moved C2 24.4 mm to (68.9, 50.7), turned to 270 degrees
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Connections:
- new net CMP: C14.2, C22.2, U$5.P$6
- new net N$22: R28.1, U$5.P$7
- new net N$27: R23.1, R9.1, U$5.P$5
- new net N$37: C22.1, R29.2
- net GND: now also C14.1, R29.1, U$5.P$4; no longer EXT.10, EXT.16, IC1.3, IC1.5
- net GPIO_23: now also EXT.11; no longer EXT.15
- net N$2: now also C5.2, L4.1, U$5.P$2; no longer IC1.2, L1.P$1
- net N$26: now also U$5.P$8; no longer IC1.4, R23.1, R9.1
- net PA0: now also SJ2.1; no longer R5.3
- net PA1: now also SJ1.1; no longer R5.4
- net PA4: no longer SJ1.1
- net PA5: now also R5.3
- net PA6: now also R5.4; no longer SJ2.1
- net PD3/TXD: now also EXT.10; no longer EXT.11
- net USB_D_N: now also EXT.16
- net USB_D_P: now also EXT.15
- net VIN: now also R28.2, U$5.P$1; no longer IC1.1
- net VSOURCE: now also L4.2; no longer C5.2, L1.P$2
Routing:
- net GND: track 1490.6 -> 0.00 mm, vias 18 -> 0
- net VCC: track 784.4 -> 0.00 mm, vias 7 -> 0
- net VDD: track 614.0 -> 0.00 mm, vias 16 -> 0
- net PD_VDC: track 536.7 -> 0.00 mm, vias 15 -> 0
- net ETH0_GRN-: track 496.4 -> 0.00 mm, vias 17 -> 0
- net +57: track 370.0 -> 0.00 mm, vias 4 -> 0
- net N$6: track 330.6 -> 0.00 mm, vias 10 -> 0
- net VIN: track 329.4 -> 0.00 mm, vias 3 -> 0
- net PA6: track 250.7 -> 0.00 mm, vias 1 -> 0
- net PA4: track 220.2 -> 0.00 mm, vias 1 -> 0
- net VSOURCE: track 217.5 -> 0.00 mm, vias 8 -> 0
- net VLITHIUM: track 203.3 -> 0.00 mm, vias 4 -> 0
- net PD3/TXD: track 187.7 -> 0.00 mm, vias 6 -> 0
- net N$15: track 175.3 -> 0.00 mm, vias 4 -> 0
- net +2V: track 169.7 -> 0.00 mm, vias 2 -> 0
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
Commit message: normal Push.
Parts:
- removed L4: 6.8uH, WE-PD:WE-PD_1260/1245/1280/1210
- added U$7: 6.8uH 0302, schematic:0302
- moved C18 4.27 mm to (62.6, 22.7)
- moved CN2 4.27 mm to (62.7, 18.5)
- moved R1 4.27 mm to (62.6, 21.5)
- moved B1 3.66 mm to (73.0, 20.3)
- moved C8 3.66 mm to (81.2, 23.8)
- moved R2 3.66 mm to (79.4, 18.1)
- moved U$6 3.66 mm to (80.3, 21.2)
- moved C5 0.68 mm to (78.5, 36.9), turned to 90 degrees
Connections:
- net N$2: now also U$7.P$1; no longer L4.1
- net VSOURCE: now also U$7.P$2; no longer L4.2
