File: Boards/modularVariant/schematic.brd (EAGLE design)
At the start: 93 x 70 mm, 100 parts, among them J1 AVR_SPI_PRG_6NS, Q1 FC-12M, U1 MAGJACK-POE, U2 MAGJACK-POE

Commit message: normal Push.
Parts:
- moved C16 5.26 mm to (23.4, 41.0)
- moved U$4 2.66 mm to (20.0, 36.8)
- moved C32 1.56 mm to (26.0, 34.8), turned to 90 degrees
- moved USB1 0.46 mm to (46.7, -2.30)

Commit message: normal Push.
Parts:
- removed L2: 33uh, BaseApp:INDUCTOR-10X9.8X6
- removed SKW_UART: (no value), SparkFun-Connectors:1X03
- added U$11, U$12, U$13, U$14, U$15, U$16, U$17, U$9: FIDUCIAL, adafruit:FIDUCIAL_1MM
- added U$18: SRR0735A-330M, schematic:SRR0735A-330M
- moved U$1 9.72 mm to (63.8, 21.4)
- moved R13 9.61 mm to (53.9, 22.2), turned to 180 degrees
- moved C18 8.58 mm to (64.5, 14.3)
- moved R1 8.58 mm to (64.5, 13.1)
- moved CN2 8.58 mm to (64.5, 10.1)
- moved R16 8.52 mm to (7.94, 34.1), turned to 270 degrees
- moved R21 8.25 mm to (5.61, 27.8)
- moved C21 8.15 mm to (56.5, 19.1)
- moved C1 8.12 mm to (25.1, 28.7), turned to 180 degrees
- moved C20 8.11 mm to (56.5, 20.7)
- moved R12 8.10 mm to (56.5, 26.9)
- moved R11 8.09 mm to (56.5, 25.7)
- moved R20 8.08 mm to (56.5, 24.3)
- moved C19 8.08 mm to (56.5, 23.0)
- moved R17 8.03 mm to (5.34, 33.9)
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Connections:
- removed net N$10: D1.A, L2.P$1, U$4.18
- new net N$38: D1.A, U$18.P$1, U$4.18
- net GND: now also U$18.P$2; no longer L2.P$2, SKW_UART.1
- net PD2/RXD: no longer SKW_UART.2
- net PD3/TXD: no longer SKW_UART.3
