File: Boards/poe_base/schematic.brd (EAGLE design)
At the start: 93 x 70 mm, 107 parts, among them J1 AVR_SPI_PRG_6NS, Q1 FC-12M, U1 MAGJACK-POE, U2 MAGJACK-POE

Commit message: normal Push.
Parts:
- removed C1: 100nf/100V, rcl:C0805
- removed C10: 10uf/100V, adafruit2:E2,5-6E
- removed C11: 2.2uf/100V, adafruit:E2-5
- removed C12: 470uf/50V, adafruit2:E5-10,5
- removed C15: 3.3nF, rcl:C0805
- removed C16: 150pF, rcl:C0805
- removed C17: 100nf/100v, rcl:C0805
- removed C18, C20, C21: 0.1uf, rcl:C0402
- removed C19: 4.7uF, rcl:C0402
- removed C2: (no value), SparkFun-Passives:0402-CAP
- removed C28: 1000uf/10V, adafruit:E5-13
- removed C32: 330nf/50v, rcl:C0805
- removed C6, C9: 33pF, SparkFun-Capacitors:0402-CAP
- removed CN2: (no value), adafruit:JST-PH-2-THM
- removed D1: (no value), SparkFun-DiscreteSemi:SMC
- removed D4: BA340A, SparkFun-DiscreteSemi:SMA-DIODE
- removed J1: AVR_SPI_PRG_6NS, SparkFun-Connectors:2X3-NS
- removed LED3, LED4: (no value), led:CHIP-LED0603
- removed Q1: FC-12M, crystal:FC-12M
- removed R11, R12: 57.6k, resistor:R0402
- removed R13: 10k, resistor:R0402
- removed R15: 45.3, BaseApp:R0603
- removed R16: R1, BaseApp:R0603
- removed R17: R2, BaseApp:R0603
- removed R18: 220R/2W, adafruit:R2512
- removed R19: 49.9k, BaseApp:R0603
- removed R20: 71.5, resistor:R0402
- removed R21: 30K, BaseApp:R0603
- removed SJ1, SJ2: (no value), BaseApp:SJW
- removed SW1: (no value), BaseApp:TACTILE-2PIN-RTANGLE
- removed U$1: AAT3672-1/-2, schematic:AAT3672-1/-2
- removed U$10, U$28: SOL-PAD-OPEN, BaseApp:SOL-PAD-OPEN
- removed U$18: SRR0735A-330M, schematic:SRR0735A-330M
- removed U$2: ATTINY84, SparkFun-DigitalIC:SO14
- removed U$4: SI3402, BaseApp:SI3402
- added JP2: (no value), pinhead:2X04
- added JP3: (no value), pinhead:2X08
- added S1: (no value), switch-omron:B3F-31XX
- added S2: (no value), switch-omron:B3F-10XX
- JP1: value M05X2PTH -> (none); device SparkFun-Connectors:AVR_ICSP -> pinhead:2X04
- R1: value 57.6k -> 1k; device resistor:R0402 -> SparkFun-Passives:0402-RES
- R10: value (none) -> 1k; device SparkFun-Resistors:0603-ARV -> SparkFun-Passives:0402-RES
- R4: device SparkFun-Passives:0402-RES -> SparkFun:0402-RES
- R6, R7: value 1.5k -> (none); device resistor:R0402 -> SparkFun:0402-RES
- R8: value 25.5K -> (none); device BaseApp:R0603 -> SparkFun:0402-RES
- moved R10 61.1 mm to (82.8, 53.0), turned to 180 degrees
- moved R4 49.5 mm to (24.7, 62.0), turned to 90 degrees
- moved R6 43.2 mm to (23.2, 62.0)
- moved R8 39.0 mm to (38.1, 62.2), turned to 90 degrees
- moved R7 30.5 mm to (39.8, 62.2)
- moved EXT 28.9 mm to (50.8, 57.1)
- moved C24 28.6 mm to (45.2, 10.7), turned to 90 degrees
- moved R1 19.0 mm to (82.4, 6.86), turned to 270 degrees
- moved C89 14.4 mm to (20.6, 54.7), turned to 90 degrees
- moved JP1 8.81 mm to (35.6, 57.1), turned to 0 degrees
- moved R9 8.55 mm to (86.1, 26.5)
- moved C7 6.35 mm to (67.9, 56.2)
- moved U$5 3.20 mm to (73.9, 31.1)
- moved R23 2.14 mm to (77.0, 27.6)
- moved C8 2.13 mm to (87.3, 26.5)
Connections:
- removed net +57: C1.2, C10.+, C11.+, C12.+, C32.2, D1.C, R8.2, U$28.P$1, U$4.12, U$4.16
- removed net ATTINY_RESET: J1.5, R4.1, U$2.4
- removed net CHRADP: R11.2, R12.1, U$1.P$10
- removed net N$11: U$10.P$1, U$4.4
- removed net N$12: C17.1, U$10.P$2, U$4.3
- removed net N$13: C15.1, U$4.1
- removed net N$14: C6.1, Q1.2, U$2.3
- removed net N$15: C32.1, U$4.2
- removed net N$16: R16.1, R17.2, U$4.20
- removed net N$18: R19.1, U$4.5
- removed net N$21: C9.1, Q1.1, U$2.2
- removed net N$30: SW1.1, U$2.5
- removed net N$36: R20.2, U$1.P$11
- removed net N$38: D1.A, U$18.P$1, U$4.18
- removed net N$42: C21.2, U$1.P$15
- removed net N$47: LED4.C, R7.2
- removed net N$48: LED3.C, R6.2
- removed net N$5: R1.2, U$1.P$2
- removed net N$7: C15.2, C16.1, R21.2
- removed net N$9: R15.1, U$4.8
- removed net PA0: SJ2.1, U$2.13
- removed net PA1: SJ1.1, U$2.12
- removed net PA4: J1.3, U$2.9
- removed net PA5: J1.1, R5.3, U$2.8
- removed net PA6: J1.4, R5.4, U$2.7
- removed net PD2/RXD: EXT.12, U$19.38
- removed net PD3/TXD: EXT.10, U$19.37
- removed net PD_VDC: C28.+, D4.A, R17.1, R18.2, U$28.P$2
- removed net STAT1: R6.1, SJ1.2, U$1.P$4
- removed net STAT2: R7.1, SJ2.2, U$1.P$6
- removed net TS: R13.1, U$1.P$12
- removed net VBAT: C19.1, CN2.1, U$1.P$13, U$1.P$9
- removed net VLITHIUM: C2.1, C20.2, J1.2, MCP1826.2, R27.1, R4.2, U$1.P$14, U$2.1
- new net HOSTD_N: JP3.9, U$3.P$1, USB1.2
- new net HOSTD_P: JP3.7, U$3.P$2, USB1.3
- new net JUMP_START_LED: R4.1
- new net LED_C: EXT.5, R5.3
- new net LED_D: EXT.4, R5.4
- new net SKW_UART_RXD: EXT.14, JP2.3, U$19.37
- new net SKW_UART_TXD: EXT.16, JP2.5, U$19.38
- new net SYS_LED: R6.1
- new net U_LED: R8.1
- new net VVCC: C8.1, JP1.1, JP3.1, U$6.C@1, U$6.C@2, U$6.S
- new net WRLS_LED: R7.1
- net ETH0_GRN+: no longer R19.2
- net ETH0_GRN-: no longer C10.-, C11.-, U$4.17, U$4.19, U$4.7
- net GND: now also JP2.1, JP2.8, JP3.16, JP3.4, JP3.6, R10.1; no longer C1.1, C12.-, C18.2, C19.2, C2.2, C20.1, C21.1, C28.-, C6.2, C9.2, CN2.2, EXT.2, EXT.4, J1.6, JP1.10, JP1.2, R12.2, R15.2, R16.2, R18.1, R20.1, SW1.2, U$1.P$1, U$1.P$5, U$18.P$2, U$2.14, U$4.9, U$4.PAD
- net GPIO_23: now also EXT.15; no longer EXT.11
- net I2S_CK: now also EXT.13; no longer EXT.9
- net I2S_MCK: now also EXT.11
- net I2S_MICIN: now also EXT.10
- net I2S_SD: now also EXT.12
- net I2S_WS: now also EXT.9; no longer EXT.5
- net JMP_START_LED: no longer R10.1
- net JUMPSTART: now also JP2.4, S1.2; no longer U$2.11
- net LED_A: now also EXT.1; no longer EXT.13
- net LED_B: now also EXT.3; no longer EXT.14
- net N$1: now also R7.2; no longer R10.6
- net N$3: now also R4.2; no longer R10.8
- net N$4: now also R8.2; no longer R10.5
- net N$40: now also R6.2; no longer R10.7
- net N$6: now also R10.2, S2.3, S2.4; no longer C16.2, C17.2, R21.1, U$4.15
- net N$8: now also R1.2, S1.1; no longer R8.1, U$4.6
- net PAS_VDC: now also JP3.14
- net POWER_CTRL: now also JP2.6; no longer U$2.6
- net RESET_CONFIG: now also JP2.2, S2.1, S2.2; no longer U$2.10
- net SP1: now also JP3.15; no longer U$4.11
- net SP2: now also JP3.13; no longer U$4.10
- net SYSTEM_LED: no longer R10.2
- net USBUPD1_N: now also JP3.10; no longer U$3.P$1, USB1.2
- net USBUPD1_P: now also JP3.8; no longer U$3.P$2, USB1.3
- net USB_D_N: now also JP3.12; no longer EXT.16
- net USB_D_P: now also JP3.11; no longer EXT.15
- net USB_LED: no longer R10.4
- net VCC: now also JP1.2, JP1.5, JP3.2, MCP1826.2, R27.1; no longer C18.1, C8.1, EXT.3, JP1.3, JP1.7, LED3.A, LED4.A, R13.2, U$1.P$3, U$1.P$7, U$1.P$8, U$6.C@1, U$6.C@2, U$6.S
- net VDD: now also EXT.2, JP1.7, JP2.7, JP3.5; no longer EXT.1, JP1.1, JP1.9
- net VIN: now also JP1.3, JP3.3; no longer D4.C, JP1.5
- net VSOURCE: no longer R11.1
- net WIRELESS_LED: no longer R10.3
