File: Boards/poe_base/schematic.sch (EAGLE design)
At the start: 107 parts, among them J1 AVR_SPI_PRG_6NS, Q1 FC-12M, U1 MAGJACK-POE, U2 MAGJACK-POE

Commit message: normal Push.
Parts:
- removed L2: 33uh, BaseApp:INDUCTOR
- added U$18: SRR0735A-330M, schematic:SRR0735A-330M
Connections:
- removed net N$10: D1.A, L2.1, U$4.SWO
- new net N$38: D1.A, U$18.1, U$4.SWO
- net GND: now also U$18.2; no longer L2.2
Other:
- note added: "#1"
- note added: "32.768kHz"
- note added: "FIDUCIAL"
Changed lines of the file:
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@@
 <part name="D1" library="SparkFun-DiscreteSemi" deviceset="DIODE" device="SMC/DO-214AB"/>
 <part name="C12" library="adafruit2" deviceset="CPOL-US" device="E5-10.5" value="470uf/50V"/>
-<part name="L2" library="BaseApp" deviceset="INDUCTOR" device="" value="33uh"/>
 <part name="R16" library="BaseApp" deviceset="RESISTOR" device="" value="R1"/>
 <part name="R17" library="BaseApp" deviceset="RESISTOR" device="" value="R2"/>
@@
 <part name="U$16" library="adafruit" deviceset="FIDUCIAL" device=""/>
 <part name="U$17" library="adafruit" deviceset="FIDUCIAL" device=""/>
+<part name="U$18" library="schematic" deviceset="SRR0735A-330M" device=""/>
 </parts>
 <sheets>
@@
 <wire x1="115.57" y1="59.69" x2="115.57" y2="3.81" width="1.9304" layer="94" style="shortdash"/>
 <text x="45.72" y="64.77" size="5.08" layer="94">Battery Charger</text>
+<text x="441.96" y="334.01" size="5.08" layer="94" font="vector" ratio="15">FIDUCIAL</text>
+<text x="181.61" y="227.33" size="1.778" layer="94">32.768kHz</text>
+<text x="544.83" y="7.62" size="1.778" layer="94">POE</text>
+<text x="488.95" y="6.35" size="1.778" layer="94">#1</text>
 </plain>
 <instances>
@@
 <attribute name="VALUE" x="376.301" y="145.796" size="1.778" layer="96" rot="R90"/>
 </instance>
-<instance part="L2" gate="G$1" x="356.87" y="142.24" rot="R90"/>
 <instance part="R16" gate="G$1" x="392.43" y="154.94" rot="R270"/>
 <instance part="R17" gate="G$1" x="392.43" y="170.18" rot="R270"/>
@@
 <instance part="R29" gate="G$1" x="182.88" y="120.65"/>
 <instance part="U$7" gate="G$1" x="119.38" y="134.62" rot="R90"/>
-<instance part="U$9" gate="G$1" x="453.39" y="398.78"/>
-<instance part="U$11" gate="G$1" x="463.55" y="398.78"/>
-<instance part="U$12" gate="G$1" x="473.71" y="398.78"/>
-<instance part="U$13" gate="G$1" x="483.87" y="398.78"/>
-<instance part="U$14" gate="G$1" x="453.39" y="388.62"/>
-<instance part="U$15" gate="G$1" x="463.55" y="388.62"/>
-<instance part="U$16" gate="G$1" x="473.71" y="388.62"/>
-<instance part="U$17" gate="G$1" x="483.87" y="388.62"/>
+<instance part="U$9" gate="G$1" x="444.5" y="358.14"/>
+<instance part="U$11" gate="G$1" x="454.66" y="358.14"/>
+<instance part="U$12" gate="G$1" x="464.82" y="358.14"/>
+<instance part="U$13" gate="G$1" x="474.98" y="358.14"/>
+<instance part="U$14" gate="G$1" x="444.5" y="347.98"/>
+<instance part="U$15" gate="G$1" x="454.66" y="347.98"/>
+<instance part="U$16" gate="G$1" x="464.82" y="347.98"/>
+<instance part="U$17" gate="G$1" x="474.98" y="347.98"/>
+<instance part="U$18" gate="G$1" x="358.14" y="142.24"/>
 </instances>
 <busses>
@@
 </segment>
 <segment>
-<pinref part="L2" gate="G$1" pin="2"/>
 <pinref part="C12" gate="G$1" pin="-"/>
 <wire x1="364.49" y1="142.24" x2="372.11" y2="142.24" width="0.1524" layer="91"/>
@@
 <pinref part="GND2" gate="1" pin="GND"/>
 <junction x="416.56" y="142.24"/>
+<junction x="364.49" y="142.24"/>
+<pinref part="U$18" gate="G$1" pin="2"/>
+<junction x="360.68" y="142.24"/>
+<wire x1="360.68" y1="142.24" x2="364.49" y2="142.24" width="0.1524" layer="91"/>
 </segment>
 <segment>
@@
 <wire x1="328.93" y1="55.88" x2="328.93" y2="43.18" width="0.1524" layer="91"/>
 <pinref part="R15" gate="G$1" pin="1"/>
-</segment>
-</net>
-<net name="N$10" class="0">
-<segment>
-<pinref part="U$4" gate="G$1" pin="SWO"/>
-<pinref part="D1" gate="G$1" pin="A"/>
-<wire x1="341.63" y1="101.6" x2="341.63" y2="142.24" width="0.1524" layer="91"/>
-<pinref part="L2" gate="G$1" pin="1"/>
-<wire x1="341.63" y1="142.24" x2="341.63" y2="149.86" width="0.1524" layer="91"/>
-<wire x1="341.63" y1="142.24" x2="349.25" y2="142.24" width="0.1524" layer="91"/>
-<junction x="341.63" y="142.24"/>
 </segment>
 </net>
@@
 </segment>
 </net>
+<net name="N$38" class="0">
+<segment>
+<pinref part="U$18" gate="G$1" pin="1"/>
+<junction x="353.06" y="142.24"/>
+<pinref part="U$4" gate="G$1" pin="SWO"/>
+<pinref part="D1" gate="G$1" pin="A"/>
+<wire x1="341.63" y1="101.6" x2="341.63" y2="142.24" width="0.1524" layer="91"/>
+<wire x1="341.63" y1="142.24" x2="341.63" y2="149.86" width="0.1524" layer="91"/>
+<wire x1="341.63" y1="142.24" x2="349.25" y2="142.24" width="0.1524" layer="91"/>
+<junction x="341.63" y="142.24"/>
+<junction x="349.25" y="142.24"/>
+<wire x1="353.06" y1="142.24" x2="349.25" y2="142.24" width="0.1524" layer="91"/>
+</segment>
+</net>

Commit message: normal Push.
Parts:
- removed C1: 100nf/100V, rcl:C-EUC0805
- removed C10: 10uf/100V, adafruit2:CPOL-USE2,5-6E
- removed C11: 2.2uf/100V, adafruit:CPOL-USE2-5
- removed C12: 470uf/50V, adafruit2:CPOL-USE5-10.5
- removed C15: 3.3nF, rcl:C-EUC0805
- removed C16: 150pF, rcl:C-EUC0805
- removed C17: 100nf/100v, rcl:C-EUC0805
- removed C18, C20, C21: 0.1uf, rcl:C-EUC0402
- removed C19: 4.7uF, rcl:C-EUC0402
- removed C2: (no value), SparkFun-Passives:CAP0402-CAP
- removed C28: 1000uf/10V, adafruit:CPOL-USE5-13
- removed C32: 330nf/50v, rcl:C-EUC0805
- removed C6, C9: 33pF, SparkFun-Capacitors:CAP0402-CAP
- removed CN2: (no value), adafruit:JST_2PIN-THM
- removed D1: (no value), SparkFun-DiscreteSemi:DIODESMC/DO-214AB
- removed D4: BA340A, SparkFun-DiscreteSemi:B340A
- removed J1: AVR_SPI_PRG_6NS, SparkFun-Connectors:AVR_SPI_PRG_6NS
- removed LED3, LED4: (no value), led:LEDCHIP-LED0603
- removed Q1: FC-12M, crystal:FC-12M
- removed R11, R12: 57.6k, resistor:R-EU_R0402
- removed R13: 10k, resistor:R-EU_R0402
- removed R15: 45.3, BaseApp:RESISTOR
- removed R16: R1, BaseApp:RESISTOR
- removed R17: R2, BaseApp:RESISTOR
- removed R18: 220R/2W, adafruit:R-US_R2512
- removed R19: 49.9k, BaseApp:RESISTOR
- removed R20: 71.5, resistor:R-EU_R0402
- removed R21: 30K, BaseApp:RESISTOR
- removed SJ1, SJ2: (no value), BaseApp:JUMPER
- removed SW1: (no value), BaseApp:TACTILE-2PIN'
- removed U$1: AAT3672-1/-2, schematic:AAT3672-1/-2
- removed U$10, U$28: SOL-PAD-OPEN, BaseApp:SOL-PAD-OPEN
- removed U$18: SRR0735A-330M, schematic:SRR0735A-330M
- removed U$2: ATTINY84, SparkFun-DigitalIC:ATTINY84
- removed U$4: SI3402, BaseApp:SI3402
- added JP2: (no value), pinhead:PINHD-2X4
- added JP3: (no value), pinhead:PINHD-2X8
- added S1: (no value), switch-omron:31-XX
- added S2: (no value), switch-omron:10-XX
- JP1: value M05X2PTH -> (none); device SparkFun-Connectors:M05X2PTH -> pinhead:PINHD-2X4
- R1: value 57.6k -> 1k; device resistor:R-EU_R0402 -> SparkFun-Passives:RESISTOR0402-RES
- R10: value (none) -> 1k; device SparkFun-Resistors:RESISTOR-ARRAY0603-ARV -> SparkFun-Passives:RESISTOR0402-RES
- R4: device SparkFun-Passives:RESISTOR0402-RES -> SparkFun:RESISTOR0402-RES
- R6, R7: value 1.5k -> (none); device resistor:R-EU_R0402 -> SparkFun:RESISTOR0402-RES
- R8: value 25.5K -> (none); device BaseApp:RESISTOR -> SparkFun:RESISTOR0402-RES
Connections:
- removed net +57: C1.2, C10.+, C11.+, C12.+, C32.2, D1.C, R8.2, U$28.1, U$4.VPOSF, U$4.VPOSS
- removed net ATTINY_RESET: J1.5, R4.1, U$2.(PCINT11/~RESET/DW)PB3
- removed net CHRADP: R11.2, R12.1, U$1.CHRADP
- removed net N$11: U$10.1, U$4.ISOSSFT
- removed net N$12: C17.1, U$10.2, U$4.VDD
- removed net N$13: C15.1, U$4.EROUT
- removed net N$14: C6.1, Q1.2, U$2.(PCINT9/XTAL2)PB1
- removed net N$15: C32.1, U$4.SSFT
- removed net N$16: R16.1, R17.2, U$4.FB
- removed net N$18: R19.1, U$4.!PLOSS
- removed net N$21: C9.1, Q1.1, U$2.(PCINT8/XTAL1/CLKI)PB0
- removed net N$30: SW1.1, U$2.(PCINT10/INT0/OC0A/CKOUT)PB2
- removed net N$36: R20.2, U$1.TERM
- removed net N$38: D1.A, U$18.1, U$4.SWO
- removed net N$42: C21.2, U$1.CT
- removed net N$47: LED4.C, R7.2
- removed net N$48: LED3.C, R6.2
- removed net N$5: R1.2, U$1.ADPSET
- removed net N$7: C15.2, C16.1, R21.2
- removed net N$9: R15.1, U$4.RCL
- removed net PA0: SJ2.1, U$2.(PCINT0/AREF/ADC0)PA0
- removed net PA1: SJ1.1, U$2.(PCINT1/AIN0/ADC1)PA1
- removed net PA4: J1.3, U$2.(PCINT4/T1/SCL/USCK/ADC4)PA4
- removed net PA5: J1.1, R5R.1, U$2.(PCINT5/OC1B/MISO/DO/ADC5)PA5
- removed net PA6: J1.4, R5D.1, U$2.(PCINT6/OC1A/SDA/MOSI/ADC6)PA6
- removed net PD2/RXD: EXT.12, U$19.UART_TX(SPI_CS2)
- removed net PD3/TXD: EXT.10, U$19.UART_RX(SPI_CS1)
- removed net PD_VDC: C28.+, D4.A, R17.1, R18.2, U$28.2
- removed net STAT1: R6.1, SJ1.2, U$1.STAT1N
- removed net STAT2: R7.1, SJ2.2, U$1.STAT2N
- removed net TS: R13.1, U$1.TS
- removed net VBAT: C19.1, CN2.2, U$1.BAT, U$1.ENBAT
- removed net VLITHIUM: C2.1, C20.2, J1.2, MCP1826G$1.VIN, R27.1, R4.2, U$1.OUT, U$2.VCC
- new net HOSTD_N: JP3.9, U$3.1, USB1.2
- new net HOSTD_P: JP3.7, U$3.2, USB1.3
- new net JUMP_START_LED: R4.1
- new net LED_C: EXT.5, R5R.1
- new net LED_D: EXT.4, R5D.1
- new net SKW_UART_RXD: EXT.14, JP2.3, U$19.UART_RX(SPI_CS1)
- new net SKW_UART_TXD: EXT.16, JP2.5, U$19.UART_TX(SPI_CS2)
- new net SYS_LED: R6.1
- new net U_LED: R8.1
- new net VVCC: C8.1, JP1.1, JP3.1, U$6.C@1, U$6.C@2, U$6.S
- new net WRLS_LED: R7.1
- net ETH0_GRN+: no longer R19.2
- net ETH0_GRN-: no longer C10.-, C11.-, U$4.HSO, U$4.VSS1, U$4.VSS2
- net GND: now also JP2.1, JP2.8, JP3.16, JP3.4, JP3.6, R10.1; no longer C1.1, C12.-, C18.2, C19.2, C2.2, C20.1, C21.1, C28.-, C6.2, C9.2, CN2.1, EXT.2, EXT.4, J1.6, JP1.10, JP1.2, R12.2, R15.2, R16.2, R18.1, R20.1, SW1.2, U$1.EP, U$1.GND, U$18.2, U$2.GND, U$4.PAD, U$4.VNEG
- net GPIO_23: now also EXT.15; no longer EXT.11
- net I2S_CK: now also EXT.13; no longer EXT.9
- net I2S_MCK: now also EXT.11
- net I2S_MICIN: now also EXT.10
- net I2S_SD: now also EXT.12
- net I2S_WS: now also EXT.9; no longer EXT.5
- net JMP_START_LED: no longer R10A.1
- net JUMPSTART: now also JP2.4, S1.S; no longer U$2.(PCINT2/AIN1/ADC2)PA2
- net LED_A: now also EXT.1; no longer EXT.13
- net LED_B: now also EXT.3; no longer EXT.14
- net N$1: now also R7.2; no longer R10R.2
- net N$3: now also R4.2; no longer R10A.2
- net N$4: now also R8.2; no longer R10D.2
- net N$40: now also R6.2; no longer R10B.2
- net N$6: now also R10.2, S2.P, S2.P1; no longer C16.2, C17.2, R21.1, U$4.VSSA
- net N$8: now also R1.2, S1.P; no longer R8.1, U$4.RDET
- net PAS_VDC: now also JP3.14
- net POWER_CTRL: now also JP2.6; no longer U$2.(PCINT7/ICP/OC0B/ADC7)PA7
- net RESET_CONFIG: now also JP2.2, S2.S, S2.S1; no longer U$2.(PCINT3/T0/ADC3)PA3
- net SP1: now also JP3.15; no longer U$4.SP1
- net SP2: now also JP3.13; no longer U$4.SP2
- net SYSTEM_LED: no longer R10B.1
- net USBUPD1_N: now also JP3.10; no longer U$3.1, USB1.2
- net USBUPD1_P: now also JP3.8; no longer U$3.2, USB1.3
- net USB_D_N: now also JP3.12; no longer EXT.16
- net USB_D_P: now also JP3.11; no longer EXT.15
- net USB_LED: no longer R10D.1
- net VCC: now also JP1.2, JP1.5, JP3.2, MCP1826G$1.VIN, R27.1; no longer C18.1, C8.1, EXT.3, JP1.3, JP1.7, LED3.A, LED4.A, R13.2, U$1.ADP, U$1.EN, U$1.EN0, U$6.C@1, U$6.C@2, U$6.S
- net VDD: now also EXT.2, JP1.7, JP2.7, JP3.5; no longer EXT.1, JP1.1, JP1.9
- net VIN: now also JP1.3, JP3.3; no longer D4.C, JP1.5
- net VSOURCE: no longer R11.1
- net WIRELESS_LED: no longer R10R.1
Other:
- note added: "DC 5V"
- note added: "ETHERNET PORT"
- note removed: "32.768kHz"
- note removed: "Battery Charger"
- note removed: "Battery JST"
- note removed: "DC 5V-6V"
- moved on the sheet: C29, EXT, R14, R24, R25, R26, R4, U1, U2
