File: Boards/washer/schematic.brd (EAGLE design)
At the start: 93 x 70 mm, 93 parts, among them U1 MAGJACK-POE, U2 MAGJACK-POE

Commit message: normal Push.
Parts:
- U$18: value SRR0735A-330M -> 33uH; device schematic:SRR0735A-330M -> BaseApp:INDUCTOR-10X9.8X6
- U$7: device schematic:0302 -> SparkFun-Passives:SRN6045
- moved R17 53.6 mm to (61.1, 37.5), turned to 315 degrees
- moved R21 47.5 mm to (50.2, 23.1), turned to 225 degrees
- moved R19 47.3 mm to (62.2, 24.3), turned to 315 degrees
- moved R16 46.7 mm to (50.5, 33.1), turned to 135 degrees
- moved U$18 46.5 mm to (51.8, 42.0)
- moved U$10 45.8 mm to (55.6, 24.0), turned to 225 degrees
- moved R8 45.8 mm to (64.0, 26.1), turned to 315 degrees
- moved C17 45.3 mm to (52.8, 25.7), turned to 225 degrees
- moved C15 45.2 mm to (49.1, 29.3), turned to 225 degrees
- moved R15 44.2 mm to (65.6, 27.8), turned to 315 degrees
- moved C16 42.0 mm to (62.8, 39.1), turned to 315 degrees
- moved C1 39.0 mm to (67.3, 34.1), turned to 135 degrees
- moved U$28 38.0 mm to (66.0, 23.8), turned to 225 degrees
- moved C28 38.0 mm to (74.4, 21.6)
- moved C24 37.8 mm to (66.3, 29.3), turned to 135 degrees
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Connections:
- net N$2: now also U$7.1; no longer U$7.P$1
- net VSOURCE: now also U$7.2; no longer U$7.P$2
