File: Boards/washer/schematic.sch (EAGLE design)
At the start: 93 parts, among them U1 MAGJACK-POE, U2 MAGJACK-POE

Commit message: normal Push.
Parts:
- U$18: value SRR0735A-330M -> 33uH; device schematic:SRR0735A-330M -> BaseApp:INDUCTOR
- U$7: device schematic:INDUCTOR_0302 -> SparkFun-Passives:INDUCTORBOURNS_SRN6045
Changed lines of the file:
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@@
 <part name="C22" library="SparkFun-Capacitors" deviceset="CAP" device="0402-CAP" value="10nF"/>
 <part name="R29" library="SparkFun-Passives" deviceset="RESISTOR" device="0402-RES" value="3k"/>
-<part name="U$7" library="schematic" deviceset="INDUCTOR_0302" device="" value="6.8uH 0302"/>
+<part name="U$7" library="SparkFun-Passives" deviceset="INDUCTOR" device="BOURNS_SRN6045" value="6.8uH 0302"/>
 <part name="U$9" library="adafruit" deviceset="FIDUCIAL" device=""/>
 <part name="U$11" library="adafruit" deviceset="FIDUCIAL" device=""/>
@@
 <part name="U$16" library="adafruit" deviceset="FIDUCIAL" device=""/>
 <part name="U$17" library="adafruit" deviceset="FIDUCIAL" device=""/>
-<part name="U$18" library="schematic" deviceset="SRR0735A-330M" device=""/>
+<part name="U$18" library="BaseApp" deviceset="INDUCTOR" device="" value="33uH"/>
 <part name="JP2" library="pinhead" deviceset="PINHD-2X6" device=""/>
 <part name="JP1" library="pinhead" deviceset="PINHD-1X4" device=""/>
@@
 <instance part="U$16" gate="G$1" x="464.82" y="347.98"/>
 <instance part="U$17" gate="G$1" x="474.98" y="347.98"/>
-<instance part="U$18" gate="G$1" x="358.14" y="142.24"/>
+<instance part="U$18" gate="G$1" x="356.87" y="142.24" rot="R90"/>
 <instance part="JP2" gate="A" x="462.28" y="295.91"/>
 <instance part="JP1" gate="A" x="210.82" y="312.42"/>
@@
 <junction x="364.49" y="142.24"/>
 <pinref part="U$18" gate="G$1" pin="2"/>
-<junction x="360.68" y="142.24"/>
-<wire x1="360.68" y1="142.24" x2="364.49" y2="142.24" width="0.1524" layer="91"/>
+<junction x="364.49" y="142.24"/>
 </segment>
 <segment>
@@
 <segment>
 <pinref part="U$18" gate="G$1" pin="1"/>
-<junction x="353.06" y="142.24"/>
+<junction x="349.25" y="142.24"/>
 <pinref part="U$4" gate="G$1" pin="SWO"/>
 <pinref part="D1" gate="G$1" pin="A"/>
@@
 <junction x="341.63" y="142.24"/>
 <junction x="349.25" y="142.24"/>
-<wire x1="353.06" y1="142.24" x2="349.25" y2="142.24" width="0.1524" layer="91"/>
-</segment>
-</net>
+</segment>
+</net>
