File: Boards/washer/revB/schematic.brd (EAGLE design)
At the start: 93 x 70 mm, 93 parts, among them U1 MAGJACK-POE, U2 MAGJACK-POE

Commit message: normal Push.
Parts:
- removed C12: 470uf/50V, adafruit2:E5-10,5
- removed R14, R24, R25, R26: 330, SparkFun-Passives:0402-RES
- removed R19: 49.9k, BaseApp:R0603
- removed U$6: FDFMA2P857, BaseApp:6-WDFN-EXPOSED-PAD
- removed U1, U2: MAGJACK-POE, SparkFun-Connectors:MAGJACK-POE
- added C2, C6, C65, C66: 0.1uf, BaseApp:C0603
- added R32, R33, R42, R43: 75R, BaseApp:R0603
- added U$1: ISOLATION_DIODE-TT8U1CT, BaseApp:8-TSST
- added U$22, U$23: HR601680, schematic:SOIC-16
- added U$24, U$25: RJ45-8, schematic:RJHSE-5080-ND
- C10: value 10uf/100V -> 12uF/100V
- C11: value 2.2uf/100V -> 0.1uf/100V
- C7: value 220uf -> 10uF; device adafruit:E5-10,5 -> adafruit:E1,8-4
- JP2: device pinhead:2X06 -> pinhead:2X05
- moved C8 61.0 mm to (20.3, 26.7), turned to 90 degrees
- moved R2 56.6 mm to (24.8, 26.9), turned to 90 degrees
- moved C24 55.3 mm to (14.7, 7.79), turned to 90 degrees
- moved L3 39.6 mm to (12.2, 19.7), turned to 90 degrees
- moved USB1 39.2 mm to (7.51, -1.39)
- moved R21 38.9 mm to (72.5, 54.7), turned to 45 degrees
- moved C29 38.7 mm to (20.2, 6.24)
- moved JP4 37.8 mm to (22.6, 1.63)
- moved C17 34.1 mm to (76.1, 50.8)
- moved C11 33.0 mm to (54.0, 45.2), turned to 315 degrees
- moved C13 30.8 mm to (40.5, 59.5)
- moved C7 30.5 mm to (44.2, 60.3), turned to 270 degrees
- moved R22 30.3 mm to (40.4, 61.1), turned to 180 degrees
- moved U$3 30.2 mm to (15.3, 14.2), turned to 90 degrees
- moved MCP1826 29.7 mm to (35.3, 58.2)
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Connections:
- removed net ETH0_GRN+: R19.2, R24.2
- removed net LED_A: EXT.5, R11.1
- removed net LED_B: EXT.3, R12.1
- removed net N$18: R19.1, U$4.5
- removed net N$23: U2.11
- removed net N$24: R14.1, U1.12
- removed net N$25: R25.2, U2.13
- removed net N$31: R26.2, U2.12
- removed net N$32: U$3.P$3
- removed net N$33: U$3.P$4
- removed net N$34: U$3.P$5
- removed net N$95: R24.1, U1.13
- new net N$43: C2.2, R32.2
- new net N$45: C6.2, R33.2
- new net N$48: U$23.P$16, U$25.P$3
- new net N$49: U$23.P$14, U$25.P$6
- new net N$50: R33.1, U$23.P$15
- new net N$51: U$23.P$11, U$25.P$1
- new net N$52: U$23.P$9, U$25.P$2
- new net N$53: R32.1, U$23.P$10
- new net N$54: R42.1, U$22.P$10
- new net N$55: U$22.P$9, U$24.P$2
- new net N$56: U$22.P$11, U$24.P$1
- new net N$57: R43.1, U$22.P$15
- new net N$58: U$22.P$14, U$24.P$6
- new net N$59: U$22.P$16, U$24.P$3
- new net N$69: C65.2, R42.2
- new net N$70: C66.2, R43.2
- net +2V: now also U$22.P$2, U$22.P$7, U$23.P$2, U$23.P$7; no longer U1.3, U1.4, U2.3, U2.4
- net +57: no longer C12.+
- net ETH0_GRN-: no longer U1.14
- net GND: now also C2.1, C6.1, C65.1, C66.1, JP2.10, U$24.P$7, U$24.P$8; no longer C12.-, EXT.16, JP2.12, R14.2, R26.1, U1.GND0, U1.GND1, U2.10, U2.14, U2.GND0, U2.GND1
- net GPIO_23: now also EXT.9; no longer EXT.2
- net I2S_CK: now also EXT.7; no longer EXT.10
- net I2S_MCK: now also EXT.6; no longer EXT.7
- net I2S_MICIN: now also EXT.3; no longer EXT.6
- net I2S_SD: now also EXT.5; no longer EXT.8
- net I2S_WS: now also EXT.8; no longer EXT.9
- net JUMPSTART: now also EXT.16; no longer JP2.10
- net LAN_RX+: now also U$22.P$1; no longer U2.1
- net LAN_RX-: now also U$22.P$3; no longer U2.2
- net LAN_TX+: now also U$22.P$6; no longer U2.5
- net LAN_TX-: now also U$22.P$8; no longer U2.6
- net LAN_YLW: now also R12.1; no longer U1.11
- net PAS_VDC: now also U$24.P$4, U$24.P$5; no longer U2.9
- net POWER_CTRL: now also JP2.9; no longer JP2.11
- net RESET_CONFIG: now also EXT.14; no longer JP2.9
- net SKW_SPI_CLK: now also EXT.15; no longer EXT.13
- net SKW_SPI_MISO: now also EXT.11; no longer EXT.14
- net SKW_SPI_MOSI: now also EXT.13; no longer EXT.15
- net SKW_UART_RXD: now also EXT.10; no longer EXT.11
- net SP1: now also U$25.P$7, U$25.P$8; no longer U1.10
- net SP2: now also U$25.P$4, U$25.P$5; no longer U1.9
- net VBUS: now also U$1.P$5, U$1.P$6; no longer U$6.D@1, U$6.D@2
- net VCC: now also JP2.1; no longer JP2.2
- net VDD: now also EXT.2; no longer R25.1
- net VSOURCE: now also U$1.P$1, U$1.P$4; no longer U$6.A, U$6.G
- net VVCC: now also JP2.2, U$1.P$3, U$1.P$7, U$1.P$8; no longer JP2.1, U$6.C@1, U$6.C@2, U$6.S
- net WAN_RX+: now also U$23.P$1; no longer U1.1
- net WAN_RX-: now also U$23.P$3; no longer U1.2
- net WAN_TX+: now also U$23.P$6; no longer U1.5
- net WAN_TX-: now also U$23.P$8; no longer U1.6
- net WAN_YLW: now also R11.1
Routing:
- net GND: track 0.00 -> 593.5 mm, vias 0 -> 9
- net JUMPSTART: track 0.00 -> 133.1 mm, vias 0 -> 5
- net VSOURCE: track 0.00 -> 128.1 mm, vias 0 -> 6
- net +2V: track 0.00 -> 122.6 mm, vias 0 -> 2
- net VDD: track 0.00 -> 114.5 mm, vias 0 -> 2
- net RESET_CONFIG: track 0.00 -> 110.3 mm, vias 0 -> 4
- net LED_D: track 0.00 -> 103.8 mm, vias 0 -> 3
- net VCC: track 0.00 -> 95.3 mm, vias 0 -> 3
- net LAN_RX+: track 0.00 -> 87.9 mm, vias 0 -> 2
- net LAN_YLW: track 0.00 -> 85.8 mm, vias 0 -> 2
- net SP1: track 0.00 -> 83.4 mm, vias 0 -> 2
- net SP2: track 0.00 -> 80.0 mm, vias 0 -> 2
- net POWER_CTRL: track 0.00 -> 72.0 mm, vias 0 -> 3
- net +57: track 0.00 -> 70.4 mm, vias 0 -> 2
- net WAN_YLW: track 0.00 -> 66.1 mm, vias 0 -> 4
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
Commit message: normal Push.
Parts:
- C7: value 10uF -> 220uF; device adafruit:E1,8-4 -> adafruit:E5-10,5
- moved R17 5.27 mm to (56.9, 44.7), turned to 315 degrees
- moved C10 4.31 mm to (55.3, 38.4)
- moved C11 4.22 mm to (50.8, 42.4)
- moved C7 3.05 mm to (47.3, 60.4)
- moved JP2 2.89 mm to (14.0, 30.5)
- moved D1 2.83 mm to (53.5, 51.8)
- moved EXT 1.16 mm to (17.8, 58.4)
Routing:
- net GND: track 593.5 -> 0.00 mm, vias 9 -> 0
- net JUMPSTART: track 133.1 -> 0.00 mm, vias 5 -> 0
- net VSOURCE: track 128.1 -> 0.00 mm, vias 6 -> 0
- net +2V: track 122.6 -> 0.00 mm, vias 2 -> 0
- net VDD: track 114.5 -> 0.00 mm, vias 2 -> 0
- net RESET_CONFIG: track 110.3 -> 0.00 mm, vias 4 -> 0
- net LED_D: track 103.8 -> 0.00 mm, vias 3 -> 0
- net VCC: track 95.3 -> 0.00 mm, vias 3 -> 0
- net LAN_RX+: track 87.9 -> 0.00 mm, vias 2 -> 0
- net LAN_YLW: track 85.8 -> 0.00 mm, vias 2 -> 0
- net SP1: track 83.4 -> 0.00 mm, vias 2 -> 0
- net SP2: track 80.0 -> 0.00 mm, vias 2 -> 0
- net POWER_CTRL: track 72.0 -> 0.00 mm, vias 3 -> 0
- net +57: track 70.4 -> 0.00 mm, vias 2 -> 0
- net WAN_YLW: track 66.1 -> 0.00 mm, vias 4 -> 0
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