File: Boards/washer/revB/schematic.sch (EAGLE design)
At the start: 97 parts

Commit message: normal Push.
Parts:
- C7: value 10uF -> 220uF; device adafruit:CPOL-USE1.8-4 -> adafruit:CPOL-USE5-10.5
Changed lines of the file:
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@@
 <part name="C13" library="rcl" deviceset="C-EU" device="C0402" value="0.1uf"/>
 <part name="JP4" library="SparkFun-Connectors" deviceset="USB" device="-MICROB"/>
-<part name="C7" library="adafruit" deviceset="CPOL-US" device="E1.8-4" value="10uF"/>
+<part name="C7" library="adafruit" deviceset="CPOL-US" device="E5-10.5" value="220uF"/>
 <part name="U$4" library="BaseApp" deviceset="SI3402" device=""/>
 <part name="R8" library="BaseApp" deviceset="RESISTOR" device="" value="25.5K"/>
