File: Boards/socketable/schematic.brd (EAGLE design)
At the start: 93 x 70 mm, 97 parts

Commit message: normal Push.
Parts:
- removed C15: 3.3nF, rcl:C0805
- removed C16: 150pF, rcl:C0805
- removed C17: 100nf/100v, rcl:C0805
- removed C28: 1000uf/10V, adafruit:E5-13
- removed C32: 330nf/50v, rcl:C0805
- removed C6: 0.1uf, BaseApp:C0603
- removed D1: (no value), SparkFun-DiscreteSemi:SMC
- removed R17: R2, BaseApp:R0603
- removed R18: 220R/2W, adafruit:R2512
- removed R21: 30K, BaseApp:R0603
- removed R32, R33: 75R, BaseApp:R0603
- removed U$10, U$28: SOL-PAD-OPEN, BaseApp:SOL-PAD-OPEN
- removed U$18: 33uH, BaseApp:INDUCTOR-10X9.8X6
- added C12: 1nF,2kV, BaseApp:C0603
- added C9: 0.1uF, 50V, BaseApp:C0603
- added R14: 75R, BaseApp:R0603
- added U$6: RF-SMA, BaseApp:BU-SMA-H
- added U$8: 21000MPOE, schematic:21000MPOE
- C1: value 100nf/100V -> 0.1uF, 50V; device rcl:C0805 -> BaseApp:C0603
- C10: value 12uF/100V -> 0.1uF, 50V; device adafruit2:E2,5-6E -> BaseApp:C0603
- C11: value 0.1uf/100V -> 0.1uF, 50V; device adafruit:E2-5 -> BaseApp:C0603
- C2: value 0.1uf -> 470uF, 25V; device BaseApp:C0603 -> resistor:E3,5-10
- C7: value 10uF -> 220uF; device adafruit:E1,8-4 -> adafruit:E5-10,5
- R15: value 45.3 -> 75R
- R16: value R1 -> 75R
- R8: value 25.5K -> 75R
- S1: value (none) -> 31-XX-SMD; device switch-omron:B3F-31XX -> schematic:BF3-31XX_SMD_PAD
- U$4: value SI3402 -> UFL; device BaseApp:SI3402 -> BaseApp:UFL
- moved U$4 67.1 mm to (11.0, 14.0), turned to 0 degrees
- moved R1 52.9 mm to (29.0, 6.40), turned to 0 degrees
- moved S1 50.7 mm to (32.0, 9.45)
- moved C1 44.7 mm to (46.0, 17.4), turned to 90 degrees
- moved C2 43.6 mm to (58.8, 58.2), turned to 90 degrees
- moved C11 36.2 mm to (73.2, 14.5), turned to 180 degrees
- moved R8 35.5 mm to (48.0, 17.4), turned to 90 degrees
- moved R16 34.6 mm to (69.3, 14.5), turned to 0 degrees
- moved C10 28.6 mm to (73.2, 16.9), turned to 180 degrees
- moved R15 28.6 mm to (69.3, 16.9), turned to 0 degrees
- moved C89 25.3 mm to (48.8, 46.6), turned to 90 degrees
- moved C3 22.1 mm to (59.1, 47.4)
- moved D3 21.5 mm to (70.0, 43.5)
- moved U$7 21.3 mm to (70.0, 48.8)
- moved R3 21.0 mm to (62.6, 32.5), turned to 90 degrees
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Connections:
- removed net +57: C1.2, C10.+, C11.+, C32.2, D1.C, R8.2, U$28.P$1, U$4.12, U$4.16
- removed net ETH0_GRN-: C10.-, C11.-, U$4.17, U$4.19, U$4.7
- removed net N$11: U$10.P$1, U$4.4
- removed net N$12: C17.1, U$10.P$2, U$4.3
- removed net N$15: C32.1, U$4.2
- removed net N$38: D1.A, U$18.P$1, U$4.18
- removed net N$43: C2.2, R32.2
- removed net N$45: C6.2, R33.2
- removed net N$50: R33.1, U$23.P$15
- removed net N$53: R32.1, U$23.P$10
- removed net N$6: C16.2, C17.2, R21.1, U$4.15
- removed net N$8: R8.1, U$4.6
- removed net N$9: R15.1, U$4.8
- new net N$18: C10.2, R15.2
- new net N$21: C12.1, R14.1, R15.1, R16.1, R8.1
- new net N$24: C11.2, R16.2
- new net PAIR12: C11.1, U$23.P$15, U$8.P$1
- new net PAIR36: C10.1, U$23.P$10, U$8.P$2
- net GND: now also C12.2, C2.-, U$4.GND@1, U$4.GND@2, U$6.2, U$6.3, U$6.4, U$6.5, U$8.P$5, U$8.P$8; no longer C1.1, C2.1, C28.-, C6.1, R15.2, R16.2, R18.1, U$18.P$2, U$4.9, U$4.PAD
- net JUMPSTART: now also S1.P$2; no longer S1.2
- net N$13: now also C9.2, R14.2; no longer C15.1, U$4.1
- net N$16: now also U$4.SIG, U$6.1; no longer R16.1, R17.2, U$4.20
- net N$5: now also S1.P$1; no longer S1.1
- net N$7: now also C1.2, R8.2; no longer C15.2, C16.1, R21.2
- net PD_VDC: now also C2.+, U$8.P$6, U$8.P$7; no longer C28.+, R17.1, R18.2, U$28.P$2
- net SP1: now also C1.1, U$8.P$4; no longer U$4.11
- net SP2: now also C9.1, U$8.P$3; no longer U$4.10

Commit message: normal Push.
Parts:
- moved C89 35.6 mm to (13.3, 44.4)
- moved C2 11.3 mm to (70.1, 58.1)
- moved C4 11.3 mm to (58.8, 58.0)
- moved USB1 0.76 mm to (17.7, -3.83)

Commit message: normal Push.
Parts:
- moved R42 14.2 mm to (58.4, 17.8)
- moved C12 10.6 mm to (55.6, 17.8)
- moved C8 7.73 mm to (27.9, 25.4)
- moved U$1 7.73 mm to (30.2, 23.4)
- moved R2 7.73 mm to (32.4, 25.6)
- moved C1 7.17 mm to (38.9, 17.7)
- moved R8 6.56 mm to (41.5, 17.7)
- moved U$4 6.35 mm to (11.0, 20.4)
- moved C65 6.26 mm to (36.0, 17.7)
- moved U$7 6.17 mm to (72.1, 43.0)
- moved R14 5.65 mm to (44.2, 17.7), turned to 90 degrees
- moved C9 4.73 mm to (47.1, 17.7), turned to 90 degrees
- moved R43 3.82 mm to (49.8, 17.7)
- moved D3 3.54 mm to (66.7, 42.5), turned to 270 degrees
- moved C66 2.93 mm to (52.7, 17.8)
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
Commit message: normal Push.
Parts:
- added R17, R18: 22, BaseApp:R0603
- C13, C8: device rcl:C0402 -> rcl:C0603
- C14, C22, C24, C29, C5: device SparkFun-Capacitors:0402-CAP -> SparkFun-Capacitors:0603-CAP
- L3: device SparkFun-Passives:C0402 -> SparkFun-Passives:0603
- R10, R11, R12, R13, R20, R5, R6, R7: device SparkFun:0402-RES -> SparkFun:0603-RES
- R2, R23, R27, R29, R3, R9: device SparkFun-Passives:0402-RES -> SparkFun-Passives:0603-RES
- R22: device resistor:R0402 -> resistor:R0603
- moved C4 39.8 mm to (35.1, 26.0), turned to 90 degrees
- moved C1 36.7 mm to (74.8, 24.8)
- moved R8 32.2 mm to (72.8, 24.8)
- moved C10 30.0 mm to (43.1, 17.2), turned to 270 degrees
- moved R14 28.1 mm to (72.1, 21.0), turned to 180 degrees
- moved C9 25.0 mm to (72.1, 19.1), turned to 180 degrees
- moved R15 23.9 mm to (45.4, 17.2), turned to 90 degrees
- moved C11 23.8 mm to (49.5, 17.1), turned to 270 degrees
- moved C65 19.8 mm to (55.8, 17.2)
- moved R16 18.0 mm to (51.5, 17.1), turned to 270 degrees
- moved C12 16.8 mm to (70.9, 24.8)
- moved U$3 14.8 mm to (30.7, 14.5)
- moved R43 14.5 mm to (64.3, 17.4)
- moved C24 14.3 mm to (30.2, 12.6)
- moved USB1 14.0 mm to (31.6, -1.85)
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Connections:
- new net N$8: JP4.D-, R18.1
- new net N$9: JP4.D+, R17.1
- net GND: now also U$5.P$10, U$5.P$9
- net USBUPD1_N: now also U$3.P$2; no longer U$3.P$1
- net USBUPD1_P: now also U$3.P$1; no longer U$3.P$2
- net USB_D_N: now also R18.2; no longer JP4.D-
- net USB_D_P: now also R17.2; no longer JP4.D+

Commit message: normal Push.
Parts:
- added TP1, TP10, TP11, TP12, TP13, TP14, TP2, TP3, TP4, TP5, TP6, TP7, TP8, TP9: TPB2,54, testpad:B2,54
- C13, C8: device rcl:C0603 -> BaseApp:C0603
- C14, C22, C24, C29, C5: device SparkFun-Capacitors:0603-CAP -> BaseApp:C0603
- R1, R28, R4: device SparkFun-Passives:0402-RES -> BaseApp:R0603
- R10, R11, R12, R13, R20, R5, R6, R7: device SparkFun:0603-RES -> BaseApp:R0603
- R2, R23, R27, R29, R3, R9: device SparkFun-Passives:0603-RES -> BaseApp:R0603
- R22: device resistor:R0603 -> BaseApp:R0603
- moved R18 18.6 mm to (12.6, 23.5)
- moved R17 18.2 mm to (15.2, 23.5)
- moved U$11 13.6 mm to (8.08, 14.0)
- moved U$13 13.6 mm to (8.08, 14.0)
- moved R4 9.80 mm to (74.5, 66.1), turned to 270 degrees
- moved L3 8.93 mm to (35.0, 19.0), turned to 180 degrees
- moved R23 3.36 mm to (73.6, 27.6)
- moved C22 2.60 mm to (73.6, 41.3)
- moved R9 2.29 mm to (73.6, 30.3)
- moved C7 2.13 mm to (49.7, 58.1)
- moved D3 1.93 mm to (67.1, 48.7)
- moved R2 1.70 mm to (26.3, 30.3)
- moved C12 1.68 mm to (69.2, 24.8)
- moved R1 1.64 mm to (16.9, 6.86)
- moved U$22 1.37 mm to (60.7, 25.0)
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Connections:
- net N$8 renamed US_N
- net N$9 renamed US_P
- net GND: now also TP14.TP, TP2.TP, TP4.TP
- net PAS_VDC: now also TP11.TP
- net PD_VDC: now also TP10.TP
- net SP1: now also TP13.TP
- net SP2: now also TP12.TP
- net USBUPD1_N: now also U$3.P$1; no longer U$3.P$2
- net USBUPD1_P: now also U$3.P$2; no longer U$3.P$1
- net VBUS: now also TP7.TP
- net VDD: now also TP1.TP, TP3.TP, TP9.TP
- net VIN: now also TP6.TP
- net VSOURCE: now also TP5.TP
- net VVCC: now also TP8.TP
Routing:
- net GND: track 0.00 -> 653.5 mm, vias 0 -> 46
- net RESET_CONFIG: track 0.00 -> 126.2 mm, vias 0 -> 6
- net VDD: track 0.00 -> 120.2 mm, vias 0 -> 2
- net VSOURCE: track 0.00 -> 116.4 mm, vias 0 -> 2
- net LED_D: track 0.00 -> 80.2 mm, vias 0 -> 4
- net +2V: track 0.00 -> 79.3 mm, vias 0 -> 2
- net VCC: track 0.00 -> 79.1 mm, vias 0 -> 2
- net LAN_YLW: track 0.00 -> 78.1 mm, vias 0 -> 6
- net VJACK: track 0.00 -> 77.0 mm, vias 0 -> 2
- net WAN_YLW: track 0.00 -> 73.3 mm, vias 0 -> 6
- net LED_C: track 0.00 -> 67.8 mm, vias 0 -> 2
- net SP2: track 0.00 -> 66.7 mm, vias 0 -> 1
- net USB_LED: track 0.00 -> 65.8 mm, vias 0 -> 2
- net JUMPSTART: track 0.00 -> 64.4 mm, vias 0 -> 1
- net SP1: track 0.00 -> 64.3 mm, vias 0 -> 2
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- added copper zone on layer 1, net GND
- added copper zone on layer 16, net GND

Commit message: normal Push.
Parts:
- renumbered S1 to WPS, U$3 to PTCTN, U$6 to SMA

Commit message: normal Push.
Parts:
- removed EXT: (no value), pinhead:2X08
- added +2V: TPB2,54, testpad:B2,54
- added SERIAL: (no value), pinhead:1X04
- JP1: device pinhead:1X04 -> pinhead:2X08
- moved JP1 10.3 mm to (19.1, 58.4), turned to 180 degrees
- moved TP4 9.40 mm to (45.3, 53.9)
- moved TP1 1.68 mm to (55.8, 60.8)
- moved TP2 1.52 mm to (59.0, 60.8)
- moved TP3 0.15 mm to (11.0, 44.3), flipped to the bottom
- renumbered TP10 to PD_VDC, TP11 to PAS_VDC, TP12 to SP2, TP13 to SP1, TP14 to GND, TP5 to VSOURCE, TP6 to VIN, TP7 to VBUS, TP8 to VVCC, TP9 to VDD, U$19 to SKW, U$24 to LAN, U$25 to WAN, U$4 to UFL, U$7 to L
Connections:
- net +2V: now also +2V.TP
- net GND: now also SERIAL.1; no longer JP1.1
- net GPIO_23: now also JP1.9; no longer EXT.9
- net I2S_CK: now also JP1.7; no longer EXT.7
- net I2S_MCK: now also JP1.6; no longer EXT.6
- net I2S_MICIN: now also JP1.3; no longer EXT.3
- net I2S_SD: now also JP1.5; no longer EXT.5
- net I2S_WS: now also JP1.8; no longer EXT.8
- net JUMPSTART: now also JP1.16; no longer EXT.16
- net LED_C: now also JP1.1; no longer EXT.1
- net LED_D: now also JP1.4; no longer EXT.4
- net RESET_CONFIG: now also JP1.14; no longer EXT.14
- net SKW_SPI_CLK: now also JP1.15; no longer EXT.15
- net SKW_SPI_MISO: now also JP1.11; no longer EXT.11
- net SKW_SPI_MOSI: now also JP1.13; no longer EXT.13
- net SKW_UART_RXD: now also JP1.10, SERIAL.2; no longer EXT.10, JP1.2
- net SKW_UART_TXD: now also JP1.12, SERIAL.3; no longer EXT.12, JP1.3
- net VDD: now also JP1.2, SERIAL.4; no longer EXT.2, JP1.4
Routing:
- net GND: track 653.5 -> 665.4 mm
- net +2V: track 79.3 -> 83.3 mm
- net VDD: track 120.2 -> 123.2 mm, vias 2 -> 3
- net JUMPSTART: track 64.4 -> 65.3 mm
Other:
- board text added: "GND"
- board text added: "VDD"
