File: Boards/socketable/schematic.brd (EAGLE design)
At the start: 93 x 70 mm, 104 parts

Commit message: normal Push.
Routing:
- net GND1: track 0.00 -> 1.83 mm, vias 0 -> 2
- net GND: track 665.4 -> 667.3 mm, vias 46 -> 50
Other:
- board text added: "PUSBM"

Commit message: normal Push.
Parts:
- C13, C65, C66, C8: value 0.1uf -> 0.1uF
- C29: value (none) -> 0.1uF
- C62: value 0.1u -> 0.1uF
- C89: value 1uf -> 1uF
- moved U$12 41.7 mm to (45.0, 50.0)
- moved U$9 41.7 mm to (45.0, 50.0)
- moved U$11 9.17 mm to (16.9, 16.5)
- moved U$13 9.17 mm to (16.9, 16.5)
- moved USB1 5.08 mm to (31.6, -6.93)
- moved WPS 1.99 mm to (22.9, 9.91)
- moved U$15 1.64 mm to (89.8, 65.2)
- moved U$16 1.64 mm to (89.8, 65.2)
- moved CN1 1.53 mm to (80.2, -3.30)
- moved U$14 1.50 mm to (89.3, 4.27)
- moved U$17 1.50 mm to (89.3, 4.27)
- moved WAN 0.91 mm to (47.7, 2.29)
- moved LAN 0.91 mm to (65.4, 2.44)
Routing:
- net USBUPD1_P: track 27.7 -> 47.8 mm, vias 0 -> 3
- net GND: track 667.3 -> 684.2 mm, vias 50 -> 56
- net USBUPD1_N: track 30.7 -> 45.7 mm, vias 0 -> 1
- net VCC: track 79.1 -> 85.9 mm, vias 2 -> 4
- net N$41: track 3.43 -> 8.48 mm
- net N$5: track 13.2 -> 10.2 mm
- net N$24: track 36.7 -> 39.0 mm
- net N$70: track 39.9 -> 42.0 mm
- net JUMPSTART: track 65.3 -> 67.1 mm
- net SP2: track 66.7 -> 68.4 mm
- net N$44: track 7.25 -> 8.78 mm
- net SP1: track 64.3 -> 65.2 mm
- net PAS_VDC: track 43.2 -> 44.1 mm
- net N$58: track 13.9 -> 14.8 mm
- net N$55: track 24.1 -> 25.0 mm
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Other:
- board text added: "2014"
- board text added: "Base Router Ver 1.0"
- board text added: "Baseapp System"
- board text added: "Hardware Tested"
- board text added: "RXD"
- board text added: "Socketable"
- board text added: "TXD"
