File: Boards/socketable/schematic.sch (EAGLE design)
At the start: 98 parts

Commit message: normal Push.
Parts:
- removed C15: 3.3nF, rcl:C-EUC0805
- removed C16: 150pF, rcl:C-EUC0805
- removed C17: 100nf/100v, rcl:C-EUC0805
- removed C28: 1000uf/10V, adafruit:CPOL-USE5-13
- removed C32: 330nf/50v, rcl:C-EUC0805
- removed C6: 0.1uf, BaseApp:CAPACITOR
- removed D1: (no value), SparkFun-DiscreteSemi:DIODESMC/DO-214AB
- removed R17: R2, BaseApp:RESISTOR
- removed R18: 220R/2W, adafruit:R-US_R2512
- removed R21: 30K, BaseApp:RESISTOR
- removed R32, R33: 75R, BaseApp:RESISTOR
- removed U$10, U$28: SOL-PAD-OPEN, BaseApp:SOL-PAD-OPEN
- removed U$18: 33uH, BaseApp:INDUCTOR
- added C9: 0.1uF, 50V, BaseApp:CAPACITOR
- added R14: 75R, BaseApp:RESISTOR
- added U$6: RF-SMA, BaseApp:RF-SMA
- added U$8: 21000MPOE, schematic:21000MPOE
- C1: value 100nf/100V -> 0.1uF, 50V; device rcl:C-EUC0805 -> BaseApp:CAPACITOR
- C10: value 10uf/100V -> 0.1uF, 50V; device adafruit2:CPOL-USE2,5-6E -> BaseApp:CAPACITOR
- C11: value 2.2uf/100V -> 0.1uF, 50V; device adafruit:CPOL-USE2-5 -> BaseApp:CAPACITOR
- C12: value 470uf/50V -> 1nF,2kV; device adafruit2:CPOL-USE5-10.5 -> BaseApp:CAPACITOR
- C2: value 0.1uf -> 470uF, 25V; device BaseApp:CAPACITOR -> resistor:CPOL-EUE3.5-10
- C7: value 220uf -> 220uF
- R15: value 45.3 -> 75R
- R16: value R1 -> 75R
- R8: value 25.5K -> 75R
- S1: value (none) -> 31-XX-SMD; device switch-omron:31-XX -> schematic:31-XX-SMD
- U$4: value SI3402 -> UFL; device BaseApp:SI3402 -> BaseApp:UFL
Connections:
- removed net +57: C1.2, C10.+, C11.+, C12.+, C32.2, D1.C, R8.2, U$28.1, U$4.VPOSF, U$4.VPOSS
- removed net ETH0_GRN-: C10.-, C11.-, U$4.HSO, U$4.VSS1, U$4.VSS2
- removed net N$11: U$10.1, U$4.ISOSSFT
- removed net N$12: C17.1, U$10.2, U$4.VDD
- removed net N$15: C32.1, U$4.SSFT
- removed net N$32: U$3.3
- removed net N$33: U$3.4
- removed net N$34: U$3.5
- removed net N$38: D1.A, U$18.1, U$4.SWO
- removed net N$43: C2.2, R32.2
- removed net N$45: C6.2, R33.2
- removed net N$50: R33.1, U$23.15
- removed net N$53: R32.1, U$23.10
- removed net N$6: C16.2, C17.2, R21.1, U$4.VSSA
- removed net N$8: R8.1, U$4.RDET
- removed net N$9: R15.1, U$4.RCL
- removed net SWK_SPI_MISO: EXT.11
- new net N$18: C10.2, R15.2
- new net N$21: C12.1, R14.1, R15.1, R16.1, R8.1
- new net N$24: C11.2, R16.2
- new net PAIR12: C11.1, U$23.15, U$8.PAIR12
- new net PAIR36: C10.1, U$23.10, U$8.PAIR36
- net GND: now also C12.2, C2.-, U$4.GND@1, U$4.GND@2, U$6.GND, U$6.GND@1, U$6.GND@2, U$6.GND@3, U$8.-VDC0, U$8.-VDC1; no longer C1.1, C12.-, C2.1, C28.-, C6.1, R15.2, R16.2, R18.1, U$18.2, U$4.PAD, U$4.VNEG
- net N$13: now also C9.2, R14.2; no longer C15.1, U$4.EROUT
- net N$16: now also U$4.SIG, U$6.1; no longer R16.1, R17.2, U$4.FB
- net N$7: now also C1.2, R8.2; no longer C15.2, C16.1, R21.2
- net PD_VDC: now also C2.+, U$8.+VDC0, U$8.+VDC1; no longer C28.+, R17.1, R18.2, U$28.2
- net SKW_SPI_MISO: now also EXT.11
- net SP1: now also C1.1, U$8.PAIR78; no longer U$4.SP1
- net SP2: now also C9.1, U$8.PAIR45; no longer U$4.SP2
Other:
- note removed: "POE Active"
- moved on the sheet: C1, R15, R16, R8

Commit message: normal Push.
Parts:
- added R17, R18: 22, BaseApp:RESISTOR
- C13, C8: device rcl:C-EUC0402 -> rcl:C-EUC0603
- C14, C22, C24, C29, C5: device SparkFun-Capacitors:CAP0402-CAP -> SparkFun-Capacitors:CAP0603-CAP
- L3: device SparkFun-Passives:INDUCTOR0402 -> SparkFun-Passives:INDUCTOR0603
- R10, R11, R12, R13, R20, R5, R6, R7: device SparkFun:RESISTOR0402-RES -> SparkFun:RESISTOR0603-RES
- R2, R23, R27, R29, R3, R9: device SparkFun-Passives:RESISTOR0402-RES -> SparkFun-Passives:RESISTOR0603-RES
- R22: device resistor:R-EU_R0402 -> resistor:R-EU_R0603
Connections:
- new net N$8: JP4.D-, R18.1
- new net N$9: JP4.D+, R17.1
- net GND: now also U$5.EXPAD, U$5.E_H
- net USBUPD1_N: now also U$3.2; no longer U$3.1
- net USBUPD1_P: now also U$3.1; no longer U$3.2
- net USB_D_N: now also R18.2; no longer JP4.D-
- net USB_D_P: now also R17.2; no longer JP4.D+
Other:
- note added: "DC 6V - 36V"
- note removed: "DC 6V - 40V"

Commit message: normal Push.
Parts:
- added TP1, TP10, TP11, TP12, TP13, TP14, TP2, TP3, TP4, TP5, TP6, TP7, TP8, TP9: TPB2,54, testpad:TPB2,54
- C13, C8: device rcl:C-EUC0603 -> BaseApp:CAPACITOR
- C14, C22, C24, C29, C5: device SparkFun-Capacitors:CAP0603-CAP -> BaseApp:CAPACITOR
- R1, R28, R4: device SparkFun-Passives:RESISTOR0402-RES -> BaseApp:RESISTOR
- R10, R11, R12, R13, R20, R5, R6, R7: device SparkFun:RESISTOR0603-RES -> BaseApp:RESISTOR
- R2, R23, R27, R29, R3, R9: device SparkFun-Passives:RESISTOR0603-RES -> BaseApp:RESISTOR
- R22: device resistor:R-EU_R0603 -> BaseApp:RESISTOR
Connections:
- net N$8 renamed US_N
- net N$9 renamed US_P
- net GND: now also TP14.TP, TP2.TP, TP4.TP
- net PAS_VDC: now also TP11.TP
- net PD_VDC: now also TP10.TP
- net SP1: now also TP13.TP
- net SP2: now also TP12.TP
- net USBUPD1_N: now also U$3.1; no longer U$3.2
- net USBUPD1_P: now also U$3.2; no longer U$3.1
- net VBUS: now also TP7.TP
- net VDD: now also TP1.TP, TP3.TP, TP9.TP
- net VIN: now also TP6.TP
- net VSOURCE: now also TP5.TP
- net VVCC: now also TP8.TP
Other:
- moved on the sheet: C13, C8

Commit message: normal Push.
Parts:
- renumbered S1 to WPS, U$3 to PTCTN, U$6 to SMA
Changed lines of the file:
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@@
 <part name="C8" library="BaseApp" deviceset="CAPACITOR" device="" value="0.1uf"/>
 <part name="USB1" library="schematic" deviceset="USB_SHIELD" device="USB_A_VERTICAL"/>
-<part name="U$3" library="schematic" deviceset="PUSBMXX4-TL" device=""/>
+<part name="PTCTN" library="schematic" deviceset="PUSBMXX4-TL" device=""/>
 <part name="L3" library="SparkFun-Passives" deviceset="INDUCTOR" device="0603"/>
 <part name="C24" library="BaseApp" deviceset="CAPACITOR" device="" value="0.1uF"/>
@@
 <part name="JP1" library="pinhead" deviceset="PINHD-1X4" device=""/>
 <part name="EXT" library="pinhead" deviceset="PINHD-2X8" device=""/>
-<part name="S1" library="schematic" deviceset="31-XX-SMD" device=""/>
+<part name="WPS" library="schematic" deviceset="31-XX-SMD" device=""/>
 <part name="R1" library="BaseApp" deviceset="RESISTOR" device="" value="1k"/>
 <part name="S2" library="switch-omron" deviceset="10-XX" device=""/>
@@
 <part name="U$25" library="schematic" deviceset="RJ45-8" device="" value="RJ45-8"/>
 <part name="U$1" library="BaseApp" deviceset="ISOLATION_DIODE" device="-TT8U1CT"/>
-<part name="U$6" library="BaseApp" deviceset="RF-SMA" device=""/>
+<part name="SMA" library="BaseApp" deviceset="RF-SMA" device=""/>
 <part name="U$8" library="schematic" deviceset="21000MPOE" device=""/>
 <part name="C1" library="BaseApp" deviceset="CAPACITOR" device="" value="0.1uF, 50V"/>
@@
 <instance part="C8" gate="G$1" x="207.01" y="73.66"/>
 <instance part="USB1" gate="G$1" x="480.06" y="233.68" rot="R180"/>
-<instance part="U$3" gate="G$1" x="508" y="217.17"/>
+<instance part="PTCTN" gate="G$1" x="508" y="217.17"/>
 <instance part="L3" gate="G$1" x="501.65" y="238.76" rot="R90"/>
 <instance part="C24" gate="G$1" x="487.68" y="220.98"/>
@@
 <instance part="JP1" gate="A" x="210.82" y="312.42"/>
 <instance part="EXT" gate="A" x="520.7" y="293.37"/>
-<instance part="S1" gate="G$1" x="33.02" y="359.41" rot="R270"/>
+<instance part="WPS" gate="G$1" x="33.02" y="359.41" rot="R270"/>
 <instance part="R1" gate="G$1" x="24.13" y="354.33" rot="R90"/>
 <instance part="S2" gate="1" x="30.48" y="377.19" rot="R270"/>
@@
 <instance part="U$25" gate="G$1" x="529.59" y="172.72"/>
 <instance part="U$1" gate="G$1" x="193.04" y="85.09"/>
-<instance part="U$6" gate="G$1" x="502.92" y="356.87"/>
+<instance part="SMA" gate="G$1" x="502.92" y="356.87"/>
 <instance part="U$8" gate="G$1" x="347.98" y="130.81" rot="R90"/>
 <instance part="C1" gate="G$1" x="280.67" y="109.22"/>
@@
 </segment>
 <segment>
-<pinref part="U$3" gate="G$1" pin="7"/>
+<pinref part="PTCTN" gate="G$1" pin="7"/>
 <junction x="508" y="207.01"/>
 <wire x1="508" y1="207.01" x2="511.81" y2="207.01" width="0.1524" layer="91"/>
@@
 <wire x1="528.32" y1="354.33" x2="528.32" y2="351.79" width="0.1524" layer="91"/>
 <wire x1="528.32" y1="351.79" x2="528.32" y2="341.63" width="0.1524" layer="91"/>
-<pinref part="U$6" gate="G$1" pin="GND"/>
+<pinref part="SMA" gate="G$1" pin="GND"/>
 <junction x="505.46" y="354.33"/>
-<pinref part="U$6" gate="G$1" pin="GND@1"/>
+<pinref part="SMA" gate="G$1" pin="GND@1"/>
 <junction x="505.46" y="351.79"/>
 <wire x1="505.46" y1="354.33" x2="505.46" y2="351.79" width="0.1524" layer="91"/>
-<pinref part="U$6" gate="G$1" pin="GND@2"/>
+<pinref part="SMA" gate="G$1" pin="GND@2"/>
 <junction x="505.46" y="349.25"/>
 <wire x1="505.46" y1="351.79" x2="505.46" y2="349.25" width="0.1524" layer="91"/>
-<pinref part="U$6" gate="G$1" pin="GND@3"/>
+<pinref part="SMA" gate="G$1" pin="GND@3"/>
 <junction x="505.46" y="346.71"/>
 <wire x1="505.46" y1="349.25" x2="505.46" y2="346.71" width="0.1524" layer="91"/>
@@
 <label x="538.48" y="233.68" size="1.016" layer="95" xref="yes"/>
 <wire x1="485.14" y1="233.68" x2="495.3" y2="233.68" width="0.1524" layer="91"/>
-<pinref part="U$3" gate="G$1" pin="2"/>
+<pinref part="PTCTN" gate="G$1" pin="2"/>
 <junction x="497.84" y="217.17"/>
 <wire x1="495.3" y1="233.68" x2="538.48" y2="233.68" width="0.1524" layer="91"/>
@@
 <label x="538.48" y="231.14" size="1.016" layer="95" xref="yes"/>
 <wire x1="485.14" y1="231.14" x2="497.84" y2="231.14" width="0.1524" layer="91"/>
-<pinref part="U$3" gate="G$1" pin="1"/>
+<pinref part="PTCTN" gate="G$1" pin="1"/>
 <junction x="497.84" y="219.71"/>
 <wire x1="497.84" y1="231.14" x2="538.48" y2="231.14" width="0.1524" layer="91"/>
@@
 <wire x1="487.68" y1="226.06" x2="487.68" y2="228.6" width="0.1524" layer="91"/>
 <junction x="487.68" y="228.6"/>
-<pinref part="U$3" gate="G$1" pin="6"/>
+<pinref part="PTCTN" gate="G$1" pin="6"/>
 <junction x="518.16" y="219.71"/>
 <wire x1="518.16" y1="219.71" x2="523.24" y2="219.71" width="0.1524" layer="91"/>
@@
 </segment>
 <segment>
-<pinref part="S1" gate="G$1" pin="S"/>
+<pinref part="WPS" gate="G$1" pin="S"/>
 <junction x="38.1" y="359.41"/>
 <wire x1="38.1" y1="359.41" x2="41.91" y2="359.41" width="0.1524" layer="91"/>
@@
 <pinref part="R1" gate="G$1" pin="2"/>
 <junction x="24.13" y="359.41"/>
-<pinref part="S1" gate="G$1" pin="P"/>
+<pinref part="WPS" gate="G$1" pin="P"/>
 <junction x="27.94" y="359.41"/>
 <wire x1="24.13" y1="359.41" x2="27.94" y2="359.41" width="0.1524" layer="91"/>
@@
 <junction x="528.32" y="356.87"/>
 <wire x1="528.32" y1="356.87" x2="528.32" y2="361.95" width="0.1524" layer="91"/>
-<pinref part="U$6" gate="G$1" pin="1"/>
+<pinref part="SMA" gate="G$1" pin="1"/>
 <junction x="505.46" y="356.87"/>
 <wire x1="528.32" y1="361.95" x2="505.46" y2="361.95" width="0.1524" layer="91"/>

Commit message: normal Push.
Parts:
- removed EXT: (no value), pinhead:PINHD-2X8
- removed TP10, TP14, TP7: TPB2,54, testpad:TPB2,54
- added +2V, GND, PD_VDC, VBUS: TPB2,54, testpad:TPB2,54
- added SERIAL: (no value), pinhead:PINHD-1X4
- JP1: device pinhead:PINHD-1X4 -> pinhead:PINHD-2X8
- renumbered TP11 to PAS_VDC, TP12 to SP2, TP13 to SP1, TP5 to VSOURCE, TP6 to VIN, TP8 to VVCC, TP9 to VDD, U$19 to SKW, U$24 to LAN, U$25 to WAN, U$4 to UFL, U$7 to L
Connections:
- net +2V: now also +2V.TP
- net GND: now also GND.TP, SERIAL.1; no longer JP1.1, TP14.TP
- net GPIO_23: now also JP1.9; no longer EXT.9
- net I2S_CK: now also JP1.7; no longer EXT.7
- net I2S_MCK: now also JP1.6; no longer EXT.6
- net I2S_MICIN: now also JP1.3; no longer EXT.3
- net I2S_SD: now also JP1.5; no longer EXT.5
- net I2S_WS: now also JP1.8; no longer EXT.8
- net JUMPSTART: now also JP1.16; no longer EXT.16
- net LED_C: now also JP1.1; no longer EXT.1
- net LED_D: now also JP1.4; no longer EXT.4
- net PD_VDC: now also PD_VDC.TP; no longer TP10.TP
- net RESET_CONFIG: now also JP1.14; no longer EXT.14
- net SKW_SPI_CLK: now also JP1.15; no longer EXT.15
- net SKW_SPI_MISO: now also JP1.11; no longer EXT.11
- net SKW_SPI_MOSI: now also JP1.13; no longer EXT.13
- net SKW_UART_RXD: now also JP1.10, SERIAL.2; no longer EXT.10, JP1.2
- net SKW_UART_TXD: now also JP1.12, SERIAL.3; no longer EXT.12, JP1.3
- net VBUS: now also VBUS.TP; no longer TP7.TP
- net VDD: now also JP1.2, SERIAL.4; no longer EXT.2, JP1.4

Commit message: normal Push.
Parts:
- C13, C65, C66, C8: value 0.1uf -> 0.1uF
- C29: value (none) -> 0.1uF
- C62: value 0.1u -> 0.1uF
- C89: value 1uf -> 1uF
Changed lines of the file:
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@@
 <parts>
 <part name="GND19" library="SparkFun-Aesthetics" deviceset="GND" device=""/>
-<part name="C29" library="BaseApp" deviceset="CAPACITOR" device=""/>
+<part name="C29" library="BaseApp" deviceset="CAPACITOR" device="" value="0.1uF"/>
 <part name="MCP1826" library="BaseApp" deviceset="MCP1825T" device="" value="mcp1826"/>
 <part name="GND26" library="SparkFun" deviceset="GND" device=""/>
 <part name="R22" library="BaseApp" deviceset="RESISTOR" device="" value="10K"/>
-<part name="C13" library="BaseApp" deviceset="CAPACITOR" device="" value="0.1uf"/>
+<part name="C13" library="BaseApp" deviceset="CAPACITOR" device="" value="0.1uF"/>
 <part name="JP4" library="SparkFun-Connectors" deviceset="USB" device="-MICROB"/>
 <part name="C7" library="adafruit" deviceset="CPOL-US" device="E5-10.5" value="220uF"/>
 <part name="SKW" library="BaseApp" deviceset="SKW71" device="-" value="SKW71-"/>
-<part name="C62" library="BaseApp" deviceset="CAPACITOR" device="" value="0.1u"/>
+<part name="C62" library="BaseApp" deviceset="CAPACITOR" device="" value="0.1uF"/>
 <part name="GND1" library="BaseApp" deviceset="GND" device=""/>
 <part name="GND4" library="BaseApp" deviceset="GND" device=""/>
@@
 <part name="GND47" library="BaseApp" deviceset="GND" device=""/>
 <part name="GND48" library="BaseApp" deviceset="GND" device=""/>
-<part name="C89" library="BaseApp" deviceset="CAPACITOR" device="" value="1uf"/>
+<part name="C89" library="BaseApp" deviceset="CAPACITOR" device="" value="1uF"/>
 <part name="U$27" library="BaseApp" deviceset="VCC" device="" value="+2v"/>
 <part name="VDD1" library="supply1" deviceset="VDD" device=""/>
@@
 <part name="R3" library="BaseApp" deviceset="RESISTOR" device="" value="1k"/>
 <part name="R2" library="BaseApp" deviceset="RESISTOR" device="" value="10k"/>
-<part name="C8" library="BaseApp" deviceset="CAPACITOR" device="" value="0.1uf"/>
+<part name="C8" library="BaseApp" deviceset="CAPACITOR" device="" value="0.1uF"/>
 <part name="USB1" library="schematic" deviceset="USB_SHIELD" device="USB_A_VERTICAL"/>
 <part name="PTCTN" library="schematic" deviceset="PUSBMXX4-TL" device=""/>
@@
 <part name="R42" library="BaseApp" deviceset="RESISTOR" device="" value="75R"/>
 <part name="R43" library="BaseApp" deviceset="RESISTOR" device="" value="75R"/>
-<part name="C65" library="BaseApp" deviceset="CAPACITOR" device="" value="0.1uf"/>
-<part name="C66" library="BaseApp" deviceset="CAPACITOR" device="" value="0.1uf"/>
+<part name="C65" library="BaseApp" deviceset="CAPACITOR" device="" value="0.1uF"/>
+<part name="C66" library="BaseApp" deviceset="CAPACITOR" device="" value="0.1uF"/>
 <part name="GND52" library="BaseApp" deviceset="GND" device=""/>
 <part name="U$21" library="BaseApp" deviceset="VCC" device="" value="+2v"/>
